File: Power8GDI/hardware/design/motor/dbw_driver.kicad_sch (KiCad schematic)
At the start: 25 parts, among them U901 DRV8871DDAR, U910 SN74LVC1G08QDBVRQ1, U911 SN74LVC1G08QDBVRQ1, U912 SN74LVC1G08QDBVRQ1, U913 SN74LVC1G08QDBVRQ1, U914 SN74LVC1G04QDBVRQ1, U915 SN74LVC1G04QDBVRQ1

Commit message: Add 24 direct protected low-side output circuits with hardware inhibit
Parts:
- U901: footprint Package_SO:HSOP-8-1EP_3.9x4.9mm_P1.27mm_EP2.41x3.1mm_ThermalVias -> Power8GDI_Board:HSOP8_EP_ThermalVia0p3
Changed lines of the file:
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@@
 (wire (pts (xy 355.6 80.01) (xy 355.6 87.63)) (stroke (width 0) (type default)))
 (global_label "GND" (shape bidirectional) (at 355.6 87.63 90) (effects (font (size 1.016 1.016)) (justify right bottom)))
-(symbol (lib_id "Power8GDI_Core:Motor_DRV8871DDA") (at 482.6 88.9 0) (unit 1) (in_bom yes) (on_board yes) (dnp no) (property "Reference" "U901" (at 482.6 68.58 0) (effects (font (size 1.27 1.27)))) (property "Value" "DRV8871DDAR" (at 482.6 109.22 0) (effects (font (size 1.27 1.27)))) (property "Footprint" "Package_SO:HSOP-8-1EP_3.9x4.9mm_P1.27mm_EP2.41x3.1mm_ThermalVias" (at 482.6 88.9 0) (effects (font (size 1.27 1.27)) (hide yes))) (property "Design note" "Industrial driver candidate, not AEC-Q100. Bothinputs0=>coast/sleep. Automaticfaultretry; nofaultoutput/currenttelemetry." (at 482.6 88.9 0) (effects (font (size 1.27 1.27)) (hide yes))) (pin "1") (pin "7") (pin "9") (pin "5") (pin "3") (pin "2") (pin "4") (pin "6") (pin "8") (instances (project "Power8GDI_Core" (path "/f4d21065-0a5b-5086-a08e-1af9469f04bd/a94361be-a999-5467-91e7-db9050858e28" (reference "U901") (unit 1)))))
+(symbol (lib_id "Power8GDI_Core:Motor_DRV8871DDA") (at 482.6 88.9 0) (unit 1) (in_bom yes) (on_board yes) (dnp no) (property "Reference" "U901" (at 482.6 68.58 0) (effects (font (size 1.27 1.27)))) (property "Value" "DRV8871DDAR" (at 482.6 109.22 0) (effects (font (size 1.27 1.27)))) (property "Footprint" "Power8GDI_Board:HSOP8_EP_ThermalVia0p3" (at 482.6 88.9 0) (effects (font (size 1.27 1.27)) (hide yes))) (property "Design note" "Industrial driver candidate, not AEC-Q100. Bothinputs0=>coast/sleep. Automaticfaultretry; nofaultoutput/currenttelemetry." (at 482.6 88.9 0) (effects (font (size 1.27 1.27)) (hide yes))) (pin "1") (pin "7") (pin "9") (pin "5") (pin "3") (pin "2") (pin "4") (pin "6") (pin "8") (instances (project "Power8GDI_Core" (path "/f4d21065-0a5b-5086-a08e-1af9469f04bd/a94361be-a999-5467-91e7-db9050858e28" (reference "U901") (unit 1)))))
 (wire (pts (xy 477.52 106.68) (xy 477.52 114.3)) (stroke (width 0) (type default)))
 (global_label "GND" (shape bidirectional) (at 477.52 114.3 90) (effects (font (size 1.016 1.016)) (justify right bottom)))
