File: Power8GDI/hardware/design/power_input/power_input.kicad_sch (KiCad schematic)
At the start: 19 parts, among them U501 LM5164QDDARQ1

Commit message: Add 24 direct protected low-side output circuits with hardware inhibit
Parts:
- U501: footprint Package_SO:HSOP-8-1EP_3.9x4.9mm_P1.27mm_EP2.41x3.1mm_ThermalVias -> Power8GDI_Board:HSOP8_EP_ThermalVia0p3
Changed lines of the file:
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@@
 (wire (pts (xy 152.4 105.41) (xy 152.4 113.03)) (stroke (width 0) (type default)))
 (global_label "GND" (shape bidirectional) (at 152.4 113.03 90) (effects (font (size 1.016 1.016)) (justify right bottom)))
-(symbol (lib_id "Power8GDI_Core:LM5164DDA") (at 254 76.2 0) (unit 1) (in_bom yes) (on_board yes) (dnp no) (property "Reference" "U501" (at 254 60.96 0) (effects (font (size 1.27 1.27)))) (property "Value" "LM5164QDDARQ1" (at 254 55.88 0) (effects (font (size 1.27 1.27)))) (property "Footprint" "Package_SO:HSOP-8-1EP_3.9x4.9mm_P1.27mm_EP2.41x3.1mm_ThermalVias" (at 254 76.2 0) (effects (font (size 1.27 1.27)) (hide yes))) (property "Design note" "TI DDA8 + exposed thermal pad9. EP tied GND; use close input/boot loops, Kelvin feedback ground." (at 254 76.2 0) (effects (font (size 1.27 1.27)) (hide yes))) (pin "2") (pin "3") (pin "4") (pin "1") (pin "9") (pin "7") (pin "8") (pin "5") (pin "6") (instances (project "Power8GDI_Core" (path "/f4d21065-0a5b-5086-a08e-1af9469f04bd/d420a403-004b-5e7c-9c34-8708b750eadb" (reference "U501") (unit 1)))))
+(symbol (lib_id "Power8GDI_Core:LM5164DDA") (at 254 76.2 0) (unit 1) (in_bom yes) (on_board yes) (dnp no) (property "Reference" "U501" (at 254 60.96 0) (effects (font (size 1.27 1.27)))) (property "Value" "LM5164QDDARQ1" (at 254 55.88 0) (effects (font (size 1.27 1.27)))) (property "Footprint" "Power8GDI_Board:HSOP8_EP_ThermalVia0p3" (at 254 76.2 0) (effects (font (size 1.27 1.27)) (hide yes))) (property "Design note" "TI DDA8 + exposed thermal pad9. EP tied GND; use close input/boot loops, Kelvin feedback ground." (at 254 76.2 0) (effects (font (size 1.27 1.27)) (hide yes))) (pin "2") (pin "3") (pin "4") (pin "1") (pin "9") (pin "7") (pin "8") (pin "5") (pin "6") (instances (project "Power8GDI_Core" (path "/f4d21065-0a5b-5086-a08e-1af9469f04bd/d420a403-004b-5e7c-9c34-8708b750eadb" (reference "U501") (unit 1)))))
 (wire (pts (xy 241.3 68.58) (xy 233.68 68.58)) (stroke (width 0) (type default)))
 (global_label "VBAT_LOGIC_PROTECTED" (shape bidirectional) (at 233.68 68.58 0) (effects (font (size 1.016 1.016)) (justify right bottom)))
