File: Power8GDI/hardware/design/wbo/wbo2_heater_feed.kicad_sch (KiCad schematic)
At the start: 4 parts

Commit message: Isolate WBO symbol namespace for root schematic integration
Parts:
- C5850, C5851: symbol Power8GDI_Aux:WBO_C -> Power8GDI_WBO:WBO_C
- D5810: symbol Power8GDI_Aux:WBO_STPS5H100BY -> Power8GDI_WBO:WBO_STPS5H100BY
- D5811: symbol Power8GDI_Aux:WBO_SMBJ24CA -> Power8GDI_WBO:WBO_SMBJ24CA
Changed lines of the file:
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@@
 (kicad_sch (version 20250114) (generator "eeschema") (paper "A3") (title_block (title "WBO2: reverse protected heater supply") (rev "Engineering draft 0.1") (comment 1 "UNQUALIFIED: no manufacturing or engine approval"))
 (text "Heater current uses VBAT_MAIN_FUSED and dedicated power return; never +5V_CORE or VBAT_LOGIC_PROTECTED." (at 20 20 0) (effects (font (size 1.5 1.5)) (justify left top)))
-(symbol (lib_id "Power8GDI_Aux:WBO_STPS5H100BY") (at 90.17 74.93 0) (unit 1) (in_bom yes) (on_board yes) (dnp no) (property "Reference" "D5810" (at 90.17 67.31 0) (effects (font (size 1.27 1.27)))) (property "Value" "STPS5H100BY-TR" (at 90.17 82.55000000000001 0) (effects (font (size 1.27 1.27)))) (property "Footprint" "Package_TO_SOT_SMD:TO-252-2" (at 90.17 74.93 0) (effects (font (size 1.27 1.27)) (hide yes))) (property "Design note" "ST DS6906 page1 package: leftlead1 NC, tab2 K, rightlead3 A. External branch fuse coordination and diode thermal validation required." (at 90.17 74.93 0) (effects (font (size 1.27 1.27)) (hide yes))) (pin "1") (pin "2") (pin "3") (instances (project "Power8GDI_Core" (path "/f4d21065-0a5b-5086-a08e-1af9469f04bd/cccd9144-7da5-572f-923b-d8d84647036e" (reference "D5810") (unit 1))) (project "wbo2_heater_feed" (path "/4eb4ac01-3566-535a-8b50-19fc10394afe" (reference "D5810") (unit 1)))))
+(symbol (lib_id "Power8GDI_WBO:WBO_STPS5H100BY") (at 90.17 74.93 0) (unit 1) (in_bom yes) (on_board yes) (dnp no) (property "Reference" "D5810" (at 90.17 67.31 0) (effects (font (size 1.27 1.27)))) (property "Value" "STPS5H100BY-TR" (at 90.17 82.55000000000001 0) (effects (font (size 1.27 1.27)))) (property "Footprint" "Package_TO_SOT_SMD:TO-252-2" (at 90.17 74.93 0) (effects (font (size 1.27 1.27)) (hide yes))) (property "Design note" "ST DS6906 page1 package: leftlead1 NC, tab2 K, rightlead3 A. External branch fuse coordination and diode thermal validation required." (at 90.17 74.93 0) (effects (font (size 1.27 1.27)) (hide yes))) (pin "1") (pin "2") (pin "3") (instances (project "Power8GDI_Core" (path "/f4d21065-0a5b-5086-a08e-1af9469f04bd/cccd9144-7da5-572f-923b-d8d84647036e" (reference "D5810") (unit 1))) (project "wbo2_heater_feed" (path "/4eb4ac01-3566-535a-8b50-19fc10394afe" (reference "D5810") (unit 1)))))
 (no_connect (at 72.39 73.66))
 (wire (pts (xy 72.39 76.2) (xy 64.77 76.2)) (stroke (width 0) (type default)))
@@
 (wire (pts (xy 107.95 73.66) (xy 115.57 73.66)) (stroke (width 0) (type default)))
 (global_label "VBAT_MAIN_FUSED" (shape bidirectional) (at 115.57 73.66 180) (effects (font (size 1.016 1.016)) (justify left bottom)))
-(symbol (lib_id "Power8GDI_Aux:WBO_SMBJ24CA") (at 245.11 74.93 0) (unit 1) (in_bom yes) (on_board yes) (dnp no) (property "Reference" "D5811" (at 245.11 67.31 0) (effects (font (size 1.27 1.27)))) (property "Value" "SMBJ24CA" (at 245.11 82.55000000000001 0) (effects (font (size 1.27 1.27)))) (property "Footprint" "Diode_SMD:D_SMB" (at 245.11 74.93 0) (effects (font (size 1.27 1.27)) (hide yes))) (property "Design note" "38.9V ratedclamp nominal <40V switch minimumclamp; overshoot/pulse energy still unqualified." (at 245.11 74.93 0) (effects (font (size 1.27 1.27)) (hide yes))) (pin "1") (pin "2") (instances (project "Power8GDI_Core" (path "/f4d21065-0a5b-5086-a08e-1af9469f04bd/cccd9144-7da5-572f-923b-d8d84647036e" (reference "D5811") (unit 1))) (project "wbo2_heater_feed" (path "/4eb4ac01-3566-535a-8b50-19fc10394afe" (reference "D5811") (unit 1)))))
+(symbol (lib_id "Power8GDI_WBO:WBO_SMBJ24CA") (at 245.11 74.93 0) (unit 1) (in_bom yes) (on_board yes) (dnp no) (property "Reference" "D5811" (at 245.11 67.31 0) (effects (font (size 1.27 1.27)))) (property "Value" "SMBJ24CA" (at 245.11 82.55000000000001 0) (effects (font (size 1.27 1.27)))) (property "Footprint" "Diode_SMD:D_SMB" (at 245.11 74.93 0) (effects (font (size 1.27 1.27)) (hide yes))) (property "Design note" "38.9V ratedclamp nominal <40V switch minimumclamp; overshoot/pulse energy still unqualified." (at 245.11 74.93 0) (effects (font (size 1.27 1.27)) (hide yes))) (pin "1") (pin "2") (instances (project "Power8GDI_Core" (path "/f4d21065-0a5b-5086-a08e-1af9469f04bd/cccd9144-7da5-572f-923b-d8d84647036e" (reference "D5811") (unit 1))) (project "wbo2_heater_feed" (path "/4eb4ac01-3566-535a-8b50-19fc10394afe" (reference "D5811") (unit 1)))))
 (wire (pts (xy 227.33 74.93) (xy 219.71 74.93)) (stroke (width 0) (type default)))
 (global_label "HARNESS_WBO2_CONTACT4" (shape bidirectional) (at 219.71 74.93 0) (effects (font (size 1.016 1.016)) (justify right bottom)))
 (wire (pts (xy 262.89 74.93) (xy 270.51 74.93)) (stroke (width 0) (type default)))
 (global_label "GND" (shape bidirectional) (at 270.51 74.93 180) (effects (font (size 1.016 1.016)) (justify left bottom)))
-(symbol (lib_id "Power8GDI_Aux:WBO_C") (at 90.17 144.78 0) (unit 1) (in_bom yes) (on_board yes) (dnp no) (property "Reference" "C5850" (at 94.17 143.51 0) (effects (font (size 1.27 1.27)) (justify left))) (property "Value" "100n 100V X7R" (at 94.17 146.05 0) (effects (font (size 1.27 1.27)) (justify left))) (property "Footprint" "Capacitor_SMD:C_0805_2012Metric" (at 90.17 144.78 0) (effects (font (size 1.27 1.27)) (hide yes))) (property "Design note" "" (at 90.17 144.78 0) (effects (font (size 1.27 1.27)) (hide yes))) (pin "1") (pin "2") (instances (project "Power8GDI_Core" (path "/f4d21065-0a5b-5086-a08e-1af9469f04bd/cccd9144-7da5-572f-923b-d8d84647036e" (reference "C5850") (unit 1))) (project "wbo2_heater_feed" (path "/4eb4ac01-3566-535a-8b50-19fc10394afe" (reference "C5850") (unit 1)))))
+(symbol (lib_id "Power8GDI_WBO:WBO_C") (at 90.17 144.78 0) (unit 1) (in_bom yes) (on_board yes) (dnp no) (property "Reference" "C5850" (at 94.17 143.51 0) (effects (font (size 1.27 1.27)) (justify left))) (property "Value" "100n 100V X7R" (at 94.17 146.05 0) (effects (font (size 1.27 1.27)) (justify left))) (property "Footprint" "Capacitor_SMD:C_0805_2012Metric" (at 90.17 144.78 0) (effects (font (size 1.27 1.27)) (hide yes))) (property "Design note" "" (at 90.17 144.78 0) (effects (font (size 1.27 1.27)) (hide yes))) (pin "1") (pin "2") (instances (project "Power8GDI_Core" (path "/f4d21065-0a5b-5086-a08e-1af9469f04bd/cccd9144-7da5-572f-923b-d8d84647036e" (reference "C5850") (unit 1))) (project "wbo2_heater_feed" (path "/4eb4ac01-3566-535a-8b50-19fc10394afe" (reference "C5850") (unit 1)))))
 (wire (pts (xy 85.09 144.78) (xy 77.47 144.78)) (stroke (width 0) (type default)))
 (global_label "HARNESS_WBO2_CONTACT4" (shape bidirectional) (at 77.47 144.78 0) (effects (font (size 1.016 1.016)) (justify right bottom)))
 (wire (pts (xy 95.25 144.78) (xy 102.87 144.78)) (stroke (width 0) (type default)))
 (global_label "GND" (shape bidirectional) (at 102.87 144.78 180) (effects (font (size 1.016 1.016)) (justify left bottom)))
-(symbol (lib_id "Power8GDI_Aux:WBO_C") (at 245.11 144.78 0) (unit 1) (in_bom yes) (on_board yes) (dnp no) (property "Reference" "C5851" (at 249.11 143.51 0) (effects (font (size 1.27 1.27)) (justify left))) (property "Value" "47u 63V lowESR" (at 249.11 146.05 0) (effects (font (size 1.27 1.27)) (justify left))) (property "Footprint" "Capacitor_SMD:CP_Elec_8x10" (at 245.11 144.78 0) (effects (font (size 1.27 1.27)) (hide yes))) (property "Design note" "Provisional bulk MPN/ripple and cold ESR pending." (at 245.11 144.78 0) (effects (font (size 1.27 1.27)) (hide yes))) (pin "1") (pin "2") (instances (project "Power8GDI_Core" (path "/f4d21065-0a5b-5086-a08e-1af9469f04bd/cccd9144-7da5-572f-923b-d8d84647036e" (reference "C5851") (unit 1))) (project "wbo2_heater_feed" (path "/4eb4ac01-3566-535a-8b50-19fc10394afe" (reference "C5851") (unit 1)))))
+(symbol (lib_id "Power8GDI_WBO:WBO_C") (at 245.11 144.78 0) (unit 1) (in_bom yes) (on_board yes) (dnp no) (property "Reference" "C5851" (at 249.11 143.51 0) (effects (font (size 1.27 1.27)) (justify left))) (property "Value" "47u 63V lowESR" (at 249.11 146.05 0) (effects (font (size 1.27 1.27)) (justify left))) (property "Footprint" "Capacitor_SMD:CP_Elec_8x10" (at 245.11 144.78 0) (effects (font (size 1.27 1.27)) (hide yes))) (property "Design note" "Provisional bulk MPN/ripple and cold ESR pending." (at 245.11 144.78 0) (effects (font (size 1.27 1.27)) (hide yes))) (pin "1") (pin "2") (instances (project "Power8GDI_Core" (path "/f4d21065-0a5b-5086-a08e-1af9469f04bd/cccd9144-7da5-572f-923b-d8d84647036e" (reference "C5851") (unit 1))) (project "wbo2_heater_feed" (path "/4eb4ac01-3566-535a-8b50-19fc10394afe" (reference "C5851") (unit 1)))))
 (wire (pts (xy 240.03 144.78) (xy 232.41 144.78)) (stroke (width 0) (type default)))
 (global_label "HARNESS_WBO2_CONTACT4" (shape bidirectional) (at 232.41 144.78 0) (effects (font (size 1.016 1.016)) (justify right bottom)))
