File: Power8GDI/hardware/design/wbo/wbo2_analog.kicad_sch (KiCad schematic)
At the start: 33 parts, among them U5800 MCP6004T-E/ST, U5801 AD8628ARTZ-REEL7, U5803 REF3033AIDBZR

Commit message: Isolate WBO symbol namespace for root schematic integration
Parts:
- C5800, C5801, C5803, C5805, C5807, C5808, C5811, C5812: symbol Power8GDI_Aux:WBO_C -> Power8GDI_WBO:WBO_C
- R5800, R5801, R5802, R5803, R5804, R5805, R5806, R5807, R5808, R5809, R5810, R5811, R5812, R5813, R5814, R5815, R5818, R5819, R5820, R5821, R5823, R5824: symbol Power8GDI_Aux:WBO_R -> Power8GDI_WBO:WBO_R
- U5800: symbol Power8GDI_Aux:WBO_U600_mapped -> Power8GDI_WBO:WBO_U600_mapped
- U5801: symbol Power8GDI_Aux:WBO_U601_mapped -> Power8GDI_WBO:WBO_U601_mapped
- U5803: symbol Power8GDI_Aux:WBO_U603_mapped -> Power8GDI_WBO:WBO_U603_mapped

Commit message: Fix WBO analog net collisions and independently audit source connectivity
Connections:
- net WBO2_Net_C603_Pad1 renamed WBO2_AUTO_Net_2D__28_C603_2D_Pad1_29_
- net WBO2_Net_C605_Pad2 renamed WBO2_AUTO_Net_2D__28_C605_2D_Pad2_29_
- net WBO2_Net_R610_Pad1 renamed WBO2_AUTO_Net_2D__28_R610_2D_Pad1_29_
- net WBO2_Net_R611_Pad1 renamed WBO2_AUTO_Net_2D__28_R611_2D_Pad1_29_
- net WBO2_Net_R621_Pad1 renamed WBO2_AUTO_Net_2D__28_R621_2D_Pad1_29_
- net WBO2_Net_U600A renamed WBO2_AUTO_Net_2D__28_U600A_2D__2D__29_
- net WBO2_AUTO_Net_2D__28_U600A_2D__2D__29_: no longer R5803.1, R5805.2, U5800.3 (+)
- net WBO2_Net_U600B renamed WBO2_AUTO_Net_2D__28_U600B_2D__2B__29_
- net WBO2_AUTO_Net_2D__28_U600B_2D__2B__29_: no longer R5818.2, R5823.1, U5800.6 (-)
- net WBO2_Net_U600D renamed WBO2_AUTO_Net_2D__28_U600D_2D__2B__29_
- net WBO2_Net_U601 renamed WBO2_AUTO_Net_2D__28_U601_2D__2B__29_
- net WBO2_AUTO_Net_2D__28_U601_2D__2B__29_: no longer R5813.1, R5821.2, U5801.4 (-)
- new net WBO2_AUTO_Net_2D__28_U600A_2D__2B__29_: R5803.1, R5805.2, U5800.3 (+)
- new net WBO2_AUTO_Net_2D__28_U600B_2D__2D__29_: R5818.2, R5823.1, U5800.6 (-)
- new net WBO2_AUTO_Net_2D__28_U601_2D__2D__29_: R5813.1, R5821.2, U5801.4 (-)

Commit message: Fix WBO VDDA sequencing with precision buffered common rail and local reset
Parts:
- U5803: Design note Pinned Hellen 0.6 source U603; netlist-derived. -> Pinned Hellen 0.6 source U603; netlist-derived. Precision s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
Connections:
- net WBO2_3V3: now also C5811.1, C5812.1, R5800.1
- removed net WBO2_VDDA: C5811.1, C5812.1, R5800.1, U5803.2 (OUT)
- new net WBO2_REF3V3: U5803.2 (OUT)
Changed lines of the file:
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@@
 (symbol (lib_id "Power8GDI_WBO:WBO_C") (at 335.28 186.69 0) (unit 1) (in_bom yes) (on_board yes) (dnp no) (property "Reference" "C5811" (at 339.28 185.42 0) (effects (font (size 1.27 1.27)) (justify left))) (property "Value" "1u" (at 339.28 187.96 0) (effects (font (size 1.27 1.27)) (justify left))) (property "Footprint" "Capacitor_SMD:C_0603_1608Metric" (at 335.28 186.69 0) (effects (font (size 1.27 1.27)) (hide yes))) (property "Design note" "Pinned Hellen 0.6 source C611; netlist-derived." (at 335.28 186.69 0) (effects (font (size 1.27 1.27)) (hide yes))) (pin "1") (pin "2") (instances (project "Power8GDI_Core" (path "/f4d21065-0a5b-5086-a08e-1af9469f04bd/852d5cb7-b555-5512-bc7b-6a6a13df9b36" (reference "C5811") (unit 1))) (project "wbo2_analog" (path "/a379aa82-67b4-5f35-9573-337734fbe5b3" (reference "C5811") (unit 1)))))
 (wire (pts (xy 330.2 186.69) (xy 322.58 186.69)) (stroke (width 0) (type default)))
-(global_label "WBO2_VDDA" (shape bidirectional) (at 322.58 186.69 0) (effects (font (size 1.016 1.016)) (justify right bottom)))
+(global_label "WBO2_3V3" (shape bidirectional) (at 322.58 186.69 0) (effects (font (size 1.016 1.016)) (justify right bottom)))
 (wire (pts (xy 340.36 186.69) (xy 347.98 186.69)) (stroke (width 0) (type default)))
 (global_label "GND" (shape bidirectional) (at 347.98 186.69 180) (effects (font (size 1.016 1.016)) (justify left bottom)))
 (symbol (lib_id "Power8GDI_WBO:WBO_C") (at 469.9 186.69 0) (unit 1) (in_bom yes) (on_board yes) (dnp no) (property "Reference" "C5812" (at 473.9 185.42 0) (effects (font (size 1.27 1.27)) (justify left))) (property "Value" "100n" (at 473.9 187.96 0) (effects (font (size 1.27 1.27)) (justify left))) (property "Footprint" "Capacitor_SMD:C_0603_1608Metric" (at 469.9 186.69 0) (effects (font (size 1.27 1.27)) (hide yes))) (property "Design note" "Pinned Hellen 0.6 source C612; netlist-derived." (at 469.9 186.69 0) (effects (font (size 1.27 1.27)) (hide yes))) (pin "1") (pin "2") (instances (project "Power8GDI_Core" (path "/f4d21065-0a5b-5086-a08e-1af9469f04bd/852d5cb7-b555-5512-bc7b-6a6a13df9b36" (reference "C5812") (unit 1))) (project "wbo2_analog" (path "/a379aa82-67b4-5f35-9573-337734fbe5b3" (reference "C5812") (unit 1)))))
 (wire (pts (xy 464.82 186.69) (xy 457.2 186.69)) (stroke (width 0) (type default)))
-(global_label "WBO2_VDDA" (shape bidirectional) (at 457.2 186.69 0) (effects (font (size 1.016 1.016)) (justify right bottom)))
+(global_label "WBO2_3V3" (shape bidirectional) (at 457.2 186.69 0) (effects (font (size 1.016 1.016)) (justify right bottom)))
 (wire (pts (xy 474.98 186.69) (xy 482.6 186.69)) (stroke (width 0) (type default)))
 (global_label "GND" (shape bidirectional) (at 482.6 186.69 180) (effects (font (size 1.016 1.016)) (justify left bottom)))
 (symbol (lib_id "Power8GDI_WBO:WBO_R") (at 64.77 209.55 0) (unit 1) (in_bom yes) (on_board yes) (dnp no) (property "Reference" "R5800" (at 68.77 208.28 0) (effects (font (size 1.27 1.27)) (justify left))) (property "Value" "1k" (at 68.77 210.82 0) (effects (font (size 1.27 1.27)) (justify left))) (property "Footprint" "Resistor_SMD:R_0603_1608Metric" (at 64.77 209.55 0) (effects (font (size 1.27 1.27)) (hide yes))) (property "Design note" "Pinned Hellen 0.6 source R600; netlist-derived." (at 64.77 209.55 0) (effects (font (size 1.27 1.27)) (hide yes))) (pin "1") (pin "2") (instances (project "Power8GDI_Core" (path "/f4d21065-0a5b-5086-a08e-1af9469f04bd/852d5cb7-b555-5512-bc7b-6a6a13df9b36" (reference "R5800") (unit 1))) (project "wbo2_analog" (path "/a379aa82-67b4-5f35-9573-337734fbe5b3" (reference "R5800") (unit 1)))))
 (wire (pts (xy 59.69 209.55) (xy 52.07 209.55)) (stroke (width 0) (type default)))
-(global_label "WBO2_VDDA" (shape bidirectional) (at 52.07 209.55 0) (effects (font (size 1.016 1.016)) (justify right bottom)))
+(global_label "WBO2_3V3" (shape bidirectional) (at 52.07 209.55 0) (effects (font (size 1.016 1.016)) (justify right bottom)))
 (wire (pts (xy 69.85 209.55) (xy 77.47 209.55)) (stroke (width 0) (type default)))
 (global_label "WBO2_AUTO_Net_2D__28_U600D_2D__2B__29_" (shape bidirectional) (at 77.47 209.55 180) (effects (font (size 1.016 1.016)) (justify left bottom)))
@@
 (wire (pts (xy 293.37 85.09) (xy 300.99 85.09)) (stroke (width 0) (type default)))
 (global_label "WBO2_3V3" (shape bidirectional) (at 300.99 85.09 180) (effects (font (size 1.016 1.016)) (justify left bottom)))
-(symbol (lib_id "Power8GDI_WBO:WBO_U603_mapped") (at 449.58 85.09 0) (unit 1) (in_bom yes) (on_board yes) (dnp no) (property "Reference" "U5803" (at 449.58 77.47 0) (effects (font (size 1.27 1.27)))) (property "Value" "REF3033AIDBZR" (at 449.58 92.71 0) (effects (font (size 1.27 1.27)))) (property "Footprint" "Package_TO_SOT_SMD:SOT-23" (at 449.58 85.09 0) (effects (font (size 1.27 1.27)) (hide yes))) (property "Design note" "Pinned Hellen 0.6 source U603; netlist-derived." (at 449.58 85.09 0) (effects (font (size 1.27 1.27)) (hide yes))) (pin "1") (pin "2") (pin "3") (instances (project "Power8GDI_Core" (path "/f4d21065-0a5b-5086-a08e-1af9469f04bd/852d5cb7-b555-5512-bc7b-6a6a13df9b36" (reference "U5803") (unit 1))) (project "wbo2_analog" (path "/a379aa82-67b4-5f35-9573-337734fbe5b3" (reference "U5803") (unit 1)))))
+(symbol (lib_id "Power8GDI_WBO:WBO_U603_mapped") (at 449.58 85.09 0) (unit 1) (in_bom yes) (on_board yes) (dnp no) (property "Reference" "U5803" (at 449.58 77.47 0) (effects (font (size 1.27 1.27)))) (property "Value" "REF3033AIDBZR" (at 449.58 92.71 0) (effects (font (size 1.27 1.27)))) (property "Footprint" "Package_TO_SOT_SMD:SOT-23" (at 449.58 85.09 0) (effects (font (size 1.27 1.27)) (hide yes))) (property "Design note" "Pinned Hellen 0.6 source U603; netlist-derived. Precision setpoint only; LT3042 buffers the common VDD/VDDA rail." (at 449.58 85.09 0) (effects (font (size 1.27 1.27)) (hide yes))) (pin "1") (pin "2") (pin "3") (instances (project "Power8GDI_Core" (path "/f4d21065-0a5b-5086-a08e-1af9469f04bd/852d5cb7-b555-5512-bc7b-6a6a13df9b36" (reference "U5803") (unit 1))) (project "wbo2_analog" (path "/a379aa82-67b4-5f35-9573-337734fbe5b3" (reference "U5803") (unit 1)))))
 (wire (pts (xy 431.8 83.82) (xy 424.18 83.82)) (stroke (width 0) (type default)))
 (global_label "+5V_CORE" (shape bidirectional) (at 424.18 83.82 0) (effects (font (size 1.016 1.016)) (justify right bottom)))
 (wire (pts (xy 431.8 86.36) (xy 424.18 86.36)) (stroke (width 0) (type default)))
-(global_label "WBO2_VDDA" (shape bidirectional) (at 424.18 86.36 0) (effects (font (size 1.016 1.016)) (justify right bottom)))
+(global_label "WBO2_REF3V3" (shape bidirectional) (at 424.18 86.36 0) (effects (font (size 1.016 1.016)) (justify right bottom)))
 (wire (pts (xy 467.36 83.82) (xy 474.98 83.82)) (stroke (width 0) (type default)))
 (global_label "GND" (shape bidirectional) (at 474.98 83.82 180) (effects (font (size 1.016 1.016)) (justify left bottom)))
