File: Power8GDI/hardware/design/wbo/wbo2_control.kicad_sch (KiCad schematic)
At the start: 37 parts, among them J5800 Conn_02x03_Odd_Even, Q5800 VND7NV04TR-E, U5802 STM32F042K6T6, U5804 XC6206P332MR-G, U5805 TJA1051T/3/1J, U5810 SN74LVC1G08QDBVRQ1, U5811 SN74AHCT1G125QDBVRQ1

Commit message: Isolate WBO symbol namespace for root schematic integration
Parts:
- C5802, C5809, C5810, C5813, C5814, C5815, C5816, C5817, C5818, C5840, C5841: symbol Power8GDI_Aux:WBO_C -> Power8GDI_WBO:WBO_C
- D5800: symbol Power8GDI_Aux:WBO_D600_mapped -> Power8GDI_WBO:WBO_D600_mapped
- D5801: symbol Power8GDI_Aux:WBO_D601_mapped -> Power8GDI_WBO:WBO_D601_mapped
- D5802: symbol Power8GDI_Aux:WBO_D602_mapped -> Power8GDI_WBO:WBO_D602_mapped
- D5803: symbol Power8GDI_Aux:WBO_D603_mapped -> Power8GDI_WBO:WBO_D603_mapped
- D5804: symbol Power8GDI_Aux:WBO_D604_mapped -> Power8GDI_WBO:WBO_D604_mapped
- J5800: symbol Power8GDI_Aux:WBO_J600_mapped -> Power8GDI_WBO:WBO_J600_mapped
- Q5800: symbol Power8GDI_Aux:WBO_Q600_mapped -> Power8GDI_WBO:WBO_Q600_mapped
- R5816, R5817, R5822, R5825, R5826, R5827, R5828, R5829, R5840, R5841, R5842, R5843, R5844, R5845: symbol Power8GDI_Aux:WBO_R -> Power8GDI_WBO:WBO_R
- U5802: symbol Power8GDI_Aux:WBO_U602_mapped -> Power8GDI_WBO:WBO_U602_mapped
- U5804: symbol Power8GDI_Aux:WBO_U604_mapped -> Power8GDI_WBO:WBO_U604_mapped
- U5805: symbol Power8GDI_Aux:WBO_U605_mapped -> Power8GDI_WBO:WBO_U605_mapped
- U5810: symbol Power8GDI_Aux:WBO_SN74LVC1G08 -> Power8GDI_WBO:WBO_SN74LVC1G08
- U5811: symbol Power8GDI_Aux:WBO_SN74AHCT1G125 -> Power8GDI_WBO:WBO_SN74AHCT1G125

Commit message: Fix WBO analog net collisions and independently audit source connectivity
Connections:
- net WBO2_Net_D600_A renamed WBO2_AUTO_Net_2D__28_D600_2D_A_29_
- net WBO2_Net_D601_K renamed WBO2_AUTO_Net_2D__28_D601_2D_K_29_
- net WBO2_Net_D602_K renamed WBO2_AUTO_Net_2D__28_D602_2D_K_29_
- net WBO2_Net_D603_A renamed WBO2_AUTO_Net_2D__28_D603_2D_A_29_
- net WBO2_Net_Q600_G renamed WBO2_AUTO_Net_2D__28_Q600_2D_G_29_

Commit message: Fix WBO VDDA sequencing with precision buffered common rail and local reset
Parts:
- added C5860, C5863, C5864: 100n 16V X7R, Capacitor_SMD:C_0603_1608Metric, symbol Power8GDI_WBO:WBO_C
- added C5861, C5862: 10u 16V X7R effective>=4.7u, Capacitor_SMD:C_1206_3216Metric, symbol Power8GDI_WBO:WBO_C
- added R5860: 30k 0.1%, Resistor_SMD:R_0603_1608Metric, symbol Power8GDI_WBO:WBO_R
- added R5861: 2.2k 1%, Resistor_SMD:R_0603_1608Metric, symbol Power8GDI_WBO:WBO_R
- added R5862: 10k, Resistor_SMD:R_0603_1608Metric, symbol Power8GDI_WBO:WBO_R
- added R5863: 220R 0.1%, Resistor_SMD:R_0603_1608Metric, symbol Power8GDI_WBO:WBO_R
- added U5812: TPS3808G33QDBVRQ1, Package_TO_SOT_SMD:SOT-23-6, symbol Power8GDI_WBO:WBO_TPS3808G33
- U5804: value XC6206P332MR-G -> LT3042IMSE#WTRPBF; footprint Package_TO_SOT_SMD:SOT-23 -> Package_SO:MSOP-10-1EP_3x3mm_P0.5mm_EP1.68x1.88mm; Design note Pinned Hellen 0.6 source U604; netlist-derived. -> LT3042 RevC p15 external reference buffer; replaces XC6206.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
Connections:
- net WBO2_VDDA is gone; now on net WBO2_3V3: U5802.5 (VDDA)
- net +5V_CORE: now also U5804.1 (IN), U5804.2 (IN), U5804.6 (PGFB), C5861.1
- net GND: now also U5804.11 (EP_GND), U5804.5 (ILIM), U5804.8 (GND), C5860.2, C5861.2, C5862.2, C5863.2, C5864.2, R5860.2, R5861.2, U5812.2 (GND); no longer U5804.1 (GND)
- net WBO2_3V3: now also U5804.10 (OUT), U5804.9 (OUTS), C5862.1, C5863.1, R5861.1, R5862.2, U5812.3 (~{MR}), U5812.5 (SENSE), U5812.6 (VDD); no longer U5804.2 (VO)
- net WBO2_nRESET: now also R5862.1, U5812.1 (~{RESET})
- new net WBO2_REF3V3: C5864.1, R5863.1
- new net WBO2_REF_SET: C5860.1, R5860.1, R5863.2, U5804.7 (SET)
- no-connect marks 10 -> 12
Other:
- moved on the sheet: C5802, C5809, C5810, C5813, C5814, C5815, C5816, C5817, C5818, C5840, C5841, D5800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

Commit message: Keep WBO heater inhibit disabled when main 3V3 is absent
Parts:
- added Q5820: BC847B-QR, Package_TO_SOT_SMD:SOT-23, symbol Power8GDI_WBO:WBO_BC847B_Q
- added R5864: 4.7k 1%, Resistor_SMD:R_0603_1608Metric, symbol Power8GDI_WBO:WBO_R
- added R5865: 10k 1%, Resistor_SMD:R_0603_1608Metric, symbol Power8GDI_WBO:WBO_R
- R5842: value 10k -> 2.2k 1%
- U5811: Design note TTL input accepts3V3; disabled by independent global hardwa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 -> OE local5V pull-up defaults disabled; NPN level shift enabl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
Connections:
- net +3V3 is gone; now on net +5V_CORE: R5842.2
- net GND: now also Q5820.2 (EMITTER), R5865.2
- net HW_ACTUATOR_ENABLE_N renamed WBO2_HEATER_OE_N
- net WBO2_HEATER_OE_N: now also Q5820.3 (COLLECTOR)
- new net HW_ACTUATOR_ENABLE: R5864.1
- new net WBO2_HEATER_OE_BASE: Q5820.1 (BASE), R5864.2, R5865.1
