File: Power8GDI/hardware/design/wbo/wbo1_analog.kicad_sch (KiCad schematic)
At the start: 33 parts, among them U5600 MCP6004T-E/ST, U5601 AD8628ARTZ-REEL7, U5603 REF3033AIDBZR

Commit message: Isolate WBO symbol namespace for root schematic integration
Parts:
- C5600, C5601, C5603, C5605, C5607, C5608, C5611, C5612: symbol Power8GDI_Aux:WBO_C -> Power8GDI_WBO:WBO_C
- R5600, R5601, R5602, R5603, R5604, R5605, R5606, R5607, R5608, R5609, R5610, R5611, R5612, R5613, R5614, R5615, R5618, R5619, R5620, R5621, R5623, R5624: symbol Power8GDI_Aux:WBO_R -> Power8GDI_WBO:WBO_R
- U5600: symbol Power8GDI_Aux:WBO_U600_mapped -> Power8GDI_WBO:WBO_U600_mapped
- U5601: symbol Power8GDI_Aux:WBO_U601_mapped -> Power8GDI_WBO:WBO_U601_mapped
- U5603: symbol Power8GDI_Aux:WBO_U603_mapped -> Power8GDI_WBO:WBO_U603_mapped

Commit message: Fix WBO analog net collisions and independently audit source connectivity
Connections:
- net WBO1_Net_C603_Pad1 renamed WBO1_AUTO_Net_2D__28_C603_2D_Pad1_29_
- net WBO1_Net_C605_Pad2 renamed WBO1_AUTO_Net_2D__28_C605_2D_Pad2_29_
- net WBO1_Net_R610_Pad1 renamed WBO1_AUTO_Net_2D__28_R610_2D_Pad1_29_
- net WBO1_Net_R611_Pad1 renamed WBO1_AUTO_Net_2D__28_R611_2D_Pad1_29_
- net WBO1_Net_R621_Pad1 renamed WBO1_AUTO_Net_2D__28_R621_2D_Pad1_29_
- net WBO1_Net_U600A renamed WBO1_AUTO_Net_2D__28_U600A_2D__2D__29_
- net WBO1_AUTO_Net_2D__28_U600A_2D__2D__29_: no longer R5603.1, R5605.2, U5600.3 (+)
- net WBO1_Net_U600B renamed WBO1_AUTO_Net_2D__28_U600B_2D__2B__29_
- net WBO1_AUTO_Net_2D__28_U600B_2D__2B__29_: no longer R5618.2, R5623.1, U5600.6 (-)
- net WBO1_Net_U600D renamed WBO1_AUTO_Net_2D__28_U600D_2D__2B__29_
- net WBO1_Net_U601 renamed WBO1_AUTO_Net_2D__28_U601_2D__2B__29_
- net WBO1_AUTO_Net_2D__28_U601_2D__2B__29_: no longer R5613.1, R5621.2, U5601.4 (-)
- new net WBO1_AUTO_Net_2D__28_U600A_2D__2B__29_: R5603.1, R5605.2, U5600.3 (+)
- new net WBO1_AUTO_Net_2D__28_U600B_2D__2D__29_: R5618.2, R5623.1, U5600.6 (-)
- new net WBO1_AUTO_Net_2D__28_U601_2D__2D__29_: R5613.1, R5621.2, U5601.4 (-)

Commit message: Fix WBO VDDA sequencing with precision buffered common rail and local reset
Parts:
- U5603: Design note Pinned Hellen 0.6 source U603; netlist-derived. -> Pinned Hellen 0.6 source U603; netlist-derived. Precision s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
Connections:
- net WBO1_3V3: now also C5611.1, C5612.1, R5600.1
- removed net WBO1_VDDA: C5611.1, C5612.1, R5600.1, U5603.2 (OUT)
- new net WBO1_REF3V3: U5603.2 (OUT)
Changed lines of the file:
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@@
 (symbol (lib_id "Power8GDI_WBO:WBO_C") (at 335.28 186.69 0) (unit 1) (in_bom yes) (on_board yes) (dnp no) (property "Reference" "C5611" (at 339.28 185.42 0) (effects (font (size 1.27 1.27)) (justify left))) (property "Value" "1u" (at 339.28 187.96 0) (effects (font (size 1.27 1.27)) (justify left))) (property "Footprint" "Capacitor_SMD:C_0603_1608Metric" (at 335.28 186.69 0) (effects (font (size 1.27 1.27)) (hide yes))) (property "Design note" "Pinned Hellen 0.6 source C611; netlist-derived." (at 335.28 186.69 0) (effects (font (size 1.27 1.27)) (hide yes))) (pin "1") (pin "2") (instances (project "Power8GDI_Core" (path "/f4d21065-0a5b-5086-a08e-1af9469f04bd/cfa31682-b984-58f0-bfeb-60e967219545" (reference "C5611") (unit 1))) (project "wbo1_analog" (path "/1ef3e495-16be-508b-9ed8-3a52dc62787b" (reference "C5611") (unit 1)))))
 (wire (pts (xy 330.2 186.69) (xy 322.58 186.69)) (stroke (width 0) (type default)))
-(global_label "WBO1_VDDA" (shape bidirectional) (at 322.58 186.69 0) (effects (font (size 1.016 1.016)) (justify right bottom)))
+(global_label "WBO1_3V3" (shape bidirectional) (at 322.58 186.69 0) (effects (font (size 1.016 1.016)) (justify right bottom)))
 (wire (pts (xy 340.36 186.69) (xy 347.98 186.69)) (stroke (width 0) (type default)))
 (global_label "GND" (shape bidirectional) (at 347.98 186.69 180) (effects (font (size 1.016 1.016)) (justify left bottom)))
 (symbol (lib_id "Power8GDI_WBO:WBO_C") (at 469.9 186.69 0) (unit 1) (in_bom yes) (on_board yes) (dnp no) (property "Reference" "C5612" (at 473.9 185.42 0) (effects (font (size 1.27 1.27)) (justify left))) (property "Value" "100n" (at 473.9 187.96 0) (effects (font (size 1.27 1.27)) (justify left))) (property "Footprint" "Capacitor_SMD:C_0603_1608Metric" (at 469.9 186.69 0) (effects (font (size 1.27 1.27)) (hide yes))) (property "Design note" "Pinned Hellen 0.6 source C612; netlist-derived." (at 469.9 186.69 0) (effects (font (size 1.27 1.27)) (hide yes))) (pin "1") (pin "2") (instances (project "Power8GDI_Core" (path "/f4d21065-0a5b-5086-a08e-1af9469f04bd/cfa31682-b984-58f0-bfeb-60e967219545" (reference "C5612") (unit 1))) (project "wbo1_analog" (path "/1ef3e495-16be-508b-9ed8-3a52dc62787b" (reference "C5612") (unit 1)))))
 (wire (pts (xy 464.82 186.69) (xy 457.2 186.69)) (stroke (width 0) (type default)))
-(global_label "WBO1_VDDA" (shape bidirectional) (at 457.2 186.69 0) (effects (font (size 1.016 1.016)) (justify right bottom)))
+(global_label "WBO1_3V3" (shape bidirectional) (at 457.2 186.69 0) (effects (font (size 1.016 1.016)) (justify right bottom)))
 (wire (pts (xy 474.98 186.69) (xy 482.6 186.69)) (stroke (width 0) (type default)))
 (global_label "GND" (shape bidirectional) (at 482.6 186.69 180) (effects (font (size 1.016 1.016)) (justify left bottom)))
 (symbol (lib_id "Power8GDI_WBO:WBO_R") (at 64.77 209.55 0) (unit 1) (in_bom yes) (on_board yes) (dnp no) (property "Reference" "R5600" (at 68.77 208.28 0) (effects (font (size 1.27 1.27)) (justify left))) (property "Value" "1k" (at 68.77 210.82 0) (effects (font (size 1.27 1.27)) (justify left))) (property "Footprint" "Resistor_SMD:R_0603_1608Metric" (at 64.77 209.55 0) (effects (font (size 1.27 1.27)) (hide yes))) (property "Design note" "Pinned Hellen 0.6 source R600; netlist-derived." (at 64.77 209.55 0) (effects (font (size 1.27 1.27)) (hide yes))) (pin "1") (pin "2") (instances (project "Power8GDI_Core" (path "/f4d21065-0a5b-5086-a08e-1af9469f04bd/cfa31682-b984-58f0-bfeb-60e967219545" (reference "R5600") (unit 1))) (project "wbo1_analog" (path "/1ef3e495-16be-508b-9ed8-3a52dc62787b" (reference "R5600") (unit 1)))))
 (wire (pts (xy 59.69 209.55) (xy 52.07 209.55)) (stroke (width 0) (type default)))
-(global_label "WBO1_VDDA" (shape bidirectional) (at 52.07 209.55 0) (effects (font (size 1.016 1.016)) (justify right bottom)))
+(global_label "WBO1_3V3" (shape bidirectional) (at 52.07 209.55 0) (effects (font (size 1.016 1.016)) (justify right bottom)))
 (wire (pts (xy 69.85 209.55) (xy 77.47 209.55)) (stroke (width 0) (type default)))
 (global_label "WBO1_AUTO_Net_2D__28_U600D_2D__2B__29_" (shape bidirectional) (at 77.47 209.55 180) (effects (font (size 1.016 1.016)) (justify left bottom)))
@@
 (wire (pts (xy 293.37 85.09) (xy 300.99 85.09)) (stroke (width 0) (type default)))
 (global_label "WBO1_3V3" (shape bidirectional) (at 300.99 85.09 180) (effects (font (size 1.016 1.016)) (justify left bottom)))
-(symbol (lib_id "Power8GDI_WBO:WBO_U603_mapped") (at 449.58 85.09 0) (unit 1) (in_bom yes) (on_board yes) (dnp no) (property "Reference" "U5603" (at 449.58 77.47 0) (effects (font (size 1.27 1.27)))) (property "Value" "REF3033AIDBZR" (at 449.58 92.71 0) (effects (font (size 1.27 1.27)))) (property "Footprint" "Package_TO_SOT_SMD:SOT-23" (at 449.58 85.09 0) (effects (font (size 1.27 1.27)) (hide yes))) (property "Design note" "Pinned Hellen 0.6 source U603; netlist-derived." (at 449.58 85.09 0) (effects (font (size 1.27 1.27)) (hide yes))) (pin "1") (pin "2") (pin "3") (instances (project "Power8GDI_Core" (path "/f4d21065-0a5b-5086-a08e-1af9469f04bd/cfa31682-b984-58f0-bfeb-60e967219545" (reference "U5603") (unit 1))) (project "wbo1_analog" (path "/1ef3e495-16be-508b-9ed8-3a52dc62787b" (reference "U5603") (unit 1)))))
+(symbol (lib_id "Power8GDI_WBO:WBO_U603_mapped") (at 449.58 85.09 0) (unit 1) (in_bom yes) (on_board yes) (dnp no) (property "Reference" "U5603" (at 449.58 77.47 0) (effects (font (size 1.27 1.27)))) (property "Value" "REF3033AIDBZR" (at 449.58 92.71 0) (effects (font (size 1.27 1.27)))) (property "Footprint" "Package_TO_SOT_SMD:SOT-23" (at 449.58 85.09 0) (effects (font (size 1.27 1.27)) (hide yes))) (property "Design note" "Pinned Hellen 0.6 source U603; netlist-derived. Precision setpoint only; LT3042 buffers the common VDD/VDDA rail." (at 449.58 85.09 0) (effects (font (size 1.27 1.27)) (hide yes))) (pin "1") (pin "2") (pin "3") (instances (project "Power8GDI_Core" (path "/f4d21065-0a5b-5086-a08e-1af9469f04bd/cfa31682-b984-58f0-bfeb-60e967219545" (reference "U5603") (unit 1))) (project "wbo1_analog" (path "/1ef3e495-16be-508b-9ed8-3a52dc62787b" (reference "U5603") (unit 1)))))
 (wire (pts (xy 431.8 83.82) (xy 424.18 83.82)) (stroke (width 0) (type default)))
 (global_label "+5V_CORE" (shape bidirectional) (at 424.18 83.82 0) (effects (font (size 1.016 1.016)) (justify right bottom)))
 (wire (pts (xy 431.8 86.36) (xy 424.18 86.36)) (stroke (width 0) (type default)))
-(global_label "WBO1_VDDA" (shape bidirectional) (at 424.18 86.36 0) (effects (font (size 1.016 1.016)) (justify right bottom)))
+(global_label "WBO1_REF3V3" (shape bidirectional) (at 424.18 86.36 0) (effects (font (size 1.016 1.016)) (justify right bottom)))
 (wire (pts (xy 467.36 83.82) (xy 474.98 83.82)) (stroke (width 0) (type default)))
 (global_label "GND" (shape bidirectional) (at 474.98 83.82 180) (effects (font (size 1.016 1.016)) (justify left bottom)))

Commit message: Review B58 injector power stage and bind selected GDI6 BOM
Parts:
- C5600, C5607, C5611: Hardware_Qualification (none) -> BOARD_QUALIFICATION_PENDING; MPN (none) -> C0603C105K3RACTU; Manufacturer (none) -> KEMET; Procurement_Status (none) -> SELECTED_CATALOG_ITEM; Purchase_Released (none) -> false; Selection_Gaps (none) -> []; Selection_ID (none) -> SEL-4bca20b134b8; Selection_Ratings (none) -> {"capacitance_pf": 1000000, "dc_bias_qualification": "PENDI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; Selection_Source_URLs (none) -> https://search.kemet.com/download/specsheet/C0603C105K3RACTU
- C5601, C5605, C5608, C5612: Hardware_Qualification (none) -> BOARD_QUALIFICATION_PENDING; MPN (none) -> C0603C104K5RACTU; Manufacturer (none) -> KEMET; Procurement_Status (none) -> SELECTED_CATALOG_ITEM; Purchase_Released (none) -> false; Selection_Gaps (none) -> []; Selection_ID (none) -> SEL-6bf9727c4e40; Selection_Ratings (none) -> {"capacitance_pf": 100000, "dielectric": "X7R", "rated_volt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; Selection_Source_URLs (none) -> https://search.kemet.com/download/specsheet/C0603C104K5RACTU
- C5603: Hardware_Qualification (none) -> BOARD_QUALIFICATION_PENDING; MPN (none) -> C0603C333K5RACTU; Manufacturer (none) -> KEMET; Procurement_Status (none) -> SELECTED_CATALOG_ITEM; Purchase_Released (none) -> false; Selection_Gaps (none) -> []; Selection_ID (none) -> SEL-b5fe8cb304b7; Selection_Ratings (none) -> {"capacitance_pf": 33000, "dielectric": "X7R", "rated_volta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; Selection_Source_URLs (none) -> https://www.digikey.com/en/products/detail/kemet/C0603C333K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
- R5600, R5601: Hardware_Qualification (none) -> BOARD_QUALIFICATION_PENDING; MPN (none) -> CRCW06031K00FKEA; Manufacturer (none) -> Vishay; Procurement_Status (none) -> SELECTED_FAMILY_CODE; Purchase_Released (none) -> false; Selection_Gaps (none) -> []; Selection_ID (none) -> SEL-38197231a947; Selection_Ratings (none) -> {"aec_q200": true, "derating": "Use manufacturer power vers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; Selection_Source_URLs (none) -> https://www.vishay.com/docs/20035/dcrcwe3.pdf
- R5602, R5603: Hardware_Qualification (none) -> BOARD_QUALIFICATION_PENDING; MPN (none) -> CRCW060368K0FKEA; Manufacturer (none) -> Vishay; Procurement_Status (none) -> SELECTED_FAMILY_CODE; Purchase_Released (none) -> false; Selection_Gaps (none) -> []; Selection_ID (none) -> SEL-61df849432a4; Selection_Ratings (none) -> {"aec_q200": true, "derating": "Use manufacturer power vers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; Selection_Source_URLs (none) -> https://www.vishay.com/docs/20035/dcrcwe3.pdf
- R5604, R5605, R5613, R5614, R5618, R5619: Hardware_Qualification (none) -> BOARD_QUALIFICATION_PENDING; MPN (none) -> CRCW060310K0FKEA; Manufacturer (none) -> Vishay; Procurement_Status (none) -> SELECTED_FAMILY_CODE; Purchase_Released (none) -> false; Selection_Gaps (none) -> []; Selection_ID (none) -> SEL-9c0806476875; Selection_Ratings (none) -> {"aec_q200": true, "derating": "Use manufacturer power vers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; Selection_Source_URLs (none) -> https://www.vishay.com/docs/20035/dcrcwe3.pdf
- R5606: Hardware_Qualification (none) -> BOARD_QUALIFICATION_PENDING; MPN (none) -> CRCW060310R0FKEA; Manufacturer (none) -> Vishay; Procurement_Status (none) -> SELECTED_FAMILY_CODE; Purchase_Released (none) -> false; Selection_Gaps (none) -> []; Selection_ID (none) -> SEL-887dce68fe1a; Selection_Ratings (none) -> {"aec_q200": true, "derating": "Use manufacturer power vers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; Selection_Source_URLs (none) -> https://www.vishay.com/docs/20035/dcrcwe3.pdf
- R5607: Hardware_Qualification (none) -> BOARD_QUALIFICATION_PENDING; MPN (none) -> CRCW060322K0FKEA; Manufacturer (none) -> Vishay; Procurement_Status (none) -> SELECTED_FAMILY_CODE; Purchase_Released (none) -> false; Selection_Gaps (none) -> []; Selection_ID (none) -> SEL-e938f00a98c2; Selection_Ratings (none) -> {"aec_q200": true, "derating": "Use manufacturer power vers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; Selection_Source_URLs (none) -> https://www.vishay.com/docs/20035/dcrcwe3.pdf
- R5608: Hardware_Qualification (none) -> BOARD_QUALIFICATION_PENDING; MPN (none) -> CRCW060347R0FKEA; Manufacturer (none) -> Vishay; Procurement_Status (none) -> SELECTED_FAMILY_CODE; Purchase_Released (none) -> false; Selection_Gaps (none) -> []; Selection_ID (none) -> SEL-092784c899c7; Selection_Ratings (none) -> {"aec_q200": true, "derating": "Use manufacturer power vers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; Selection_Source_URLs (none) -> https://www.vishay.com/docs/20035/dcrcwe3.pdf
- R5609: Hardware_Qualification (none) -> BOARD_QUALIFICATION_PENDING; MPN (none) -> CRCW060361R9FKEA; Manufacturer (none) -> Vishay; Procurement_Status (none) -> SELECTED_FAMILY_CODE; Purchase_Released (none) -> false; Selection_Gaps (none) -> []; Selection_ID (none) -> SEL-62b659f4bb9e; Selection_Ratings (none) -> {"aec_q200": true, "derating": "Use manufacturer power vers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; Selection_Source_URLs (none) -> https://www.vishay.com/docs/20035/dcrcwe3.pdf
- R5610, R5611, R5612: Hardware_Qualification (none) -> BOARD_QUALIFICATION_PENDING; MPN (none) -> CRCW060320K0FKEA; Manufacturer (none) -> Vishay; Procurement_Status (none) -> SELECTED_FAMILY_CODE; Purchase_Released (none) -> false; Selection_Gaps (none) -> []; Selection_ID (none) -> SEL-cefcb9c24d02; Selection_Ratings (none) -> {"aec_q200": true, "derating": "Use manufacturer power vers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; Selection_Source_URLs (none) -> https://www.vishay.com/docs/20035/dcrcwe3.pdf
- R5615, R5621: Hardware_Qualification (none) -> BOARD_QUALIFICATION_PENDING; MPN (none) -> CRCW0603100KFKEA; Manufacturer (none) -> Vishay; Procurement_Status (none) -> SELECTED_FAMILY_CODE; Purchase_Released (none) -> false; Selection_Gaps (none) -> []; Selection_ID (none) -> SEL-4e3f06cba0aa; Selection_Ratings (none) -> {"aec_q200": true, "derating": "Use manufacturer power vers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; Selection_Source_URLs (none) -> https://www.vishay.com/docs/20035/dcrcwe3.pdf
- R5620, R5623: Hardware_Qualification (none) -> BOARD_QUALIFICATION_PENDING; MPN (none) -> CRCW060327K0FKEA; Manufacturer (none) -> Vishay; Procurement_Status (none) -> SELECTED_FAMILY_CODE; Purchase_Released (none) -> false; Selection_Gaps (none) -> []; Selection_ID (none) -> SEL-5e84dc48ae0c; Selection_Ratings (none) -> {"aec_q200": true, "derating": "Use manufacturer power vers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; Selection_Source_URLs (none) -> https://www.vishay.com/docs/20035/dcrcwe3.pdf
- R5624: Hardware_Qualification (none) -> BOARD_QUALIFICATION_PENDING; MPN (none) -> CRCW06033K30FKEA; Manufacturer (none) -> Vishay; Procurement_Status (none) -> SELECTED_FAMILY_CODE; Purchase_Released (none) -> false; Selection_Gaps (none) -> []; Selection_ID (none) -> SEL-140c192365bc; Selection_Ratings (none) -> {"aec_q200": true, "derating": "Use manufacturer power vers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; Selection_Source_URLs (none) -> https://www.vishay.com/docs/20035/dcrcwe3.pdf
- U5600: Hardware_Qualification (none) -> PINOUT_RATINGS_AND_DELIVERY_SUFFIX_REVIEW_PENDING; MPN (none) -> MCP6004T-E/ST; Manufacturer (none) -> Microchip Technology; Procurement_Status (none) -> REFERENCE_MPN_RETAINED; Purchase_Released (none) -> false; Selection_Gaps (none) -> ["Existing schematic MPN retained. Complete circuit rating/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; Selection_ID (none) -> SEL-784590d885fa; Selection_Ratings (none) -> {}; Selection_Source_URLs (none) -> https://www.microchip.com/en-us/product/MCP6004
- U5601: Hardware_Qualification (none) -> PINOUT_RATINGS_AND_DELIVERY_SUFFIX_REVIEW_PENDING; MPN (none) -> AD8628ARTZ-REEL7; Manufacturer (none) -> Analog Devices; Procurement_Status (none) -> REFERENCE_MPN_RETAINED; Purchase_Released (none) -> false; Selection_Gaps (none) -> ["Existing schematic MPN retained. Complete circuit rating/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; Selection_ID (none) -> SEL-c8711f618b70; Selection_Ratings (none) -> {}; Selection_Source_URLs (none) -> https://www.analog.com/en/search.html?q=AD8628ARTZ-REEL7
- U5603: Hardware_Qualification (none) -> PINOUT_RATINGS_AND_DELIVERY_SUFFIX_REVIEW_PENDING; MPN (none) -> REF3033AIDBZR; Manufacturer (none) -> Texas Instruments; Procurement_Status (none) -> REFERENCE_MPN_RETAINED; Purchase_Released (none) -> false; Selection_Gaps (none) -> ["Existing schematic MPN retained. Complete circuit rating/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; Selection_ID (none) -> SEL-a6de3922b9e9; Selection_Ratings (none) -> {}; Selection_Source_URLs (none) -> https://www.ti.com/product/REF3033/part-details/REF3033AIDB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
