File: Power8GDI/hardware/design/wbo/wbo1_heater_feed.kicad_sch (KiCad schematic)
At the start: 4 parts

Commit message: Isolate WBO symbol namespace for root schematic integration
Parts:
- C5650, C5651: symbol Power8GDI_Aux:WBO_C -> Power8GDI_WBO:WBO_C
- D5610: symbol Power8GDI_Aux:WBO_STPS5H100BY -> Power8GDI_WBO:WBO_STPS5H100BY
- D5611: symbol Power8GDI_Aux:WBO_SMBJ24CA -> Power8GDI_WBO:WBO_SMBJ24CA
Changed lines of the file:
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@@
 (kicad_sch (version 20250114) (generator "eeschema") (paper "A3") (title_block (title "WBO1: reverse protected heater supply") (rev "Engineering draft 0.1") (comment 1 "UNQUALIFIED: no manufacturing or engine approval"))
 (text "Heater current uses VBAT_MAIN_FUSED and dedicated power return; never +5V_CORE or VBAT_LOGIC_PROTECTED." (at 20 20 0) (effects (font (size 1.5 1.5)) (justify left top)))
-(symbol (lib_id "Power8GDI_Aux:WBO_STPS5H100BY") (at 90.17 74.93 0) (unit 1) (in_bom yes) (on_board yes) (dnp no) (property "Reference" "D5610" (at 90.17 67.31 0) (effects (font (size 1.27 1.27)))) (property "Value" "STPS5H100BY-TR" (at 90.17 82.55000000000001 0) (effects (font (size 1.27 1.27)))) (property "Footprint" "Package_TO_SOT_SMD:TO-252-2" (at 90.17 74.93 0) (effects (font (size 1.27 1.27)) (hide yes))) (property "Design note" "ST DS6906 page1 package: leftlead1 NC, tab2 K, rightlead3 A. External branch fuse coordination and diode thermal validation required." (at 90.17 74.93 0) (effects (font (size 1.27 1.27)) (hide yes))) (pin "1") (pin "2") (pin "3") (instances (project "Power8GDI_Core" (path "/f4d21065-0a5b-5086-a08e-1af9469f04bd/30a46de9-e11a-54b6-8706-ae1bab93f93c" (reference "D5610") (unit 1))) (project "wbo1_heater_feed" (path "/a54f5754-f64a-5b39-be6f-e9eea49aaacf" (reference "D5610") (unit 1)))))
+(symbol (lib_id "Power8GDI_WBO:WBO_STPS5H100BY") (at 90.17 74.93 0) (unit 1) (in_bom yes) (on_board yes) (dnp no) (property "Reference" "D5610" (at 90.17 67.31 0) (effects (font (size 1.27 1.27)))) (property "Value" "STPS5H100BY-TR" (at 90.17 82.55000000000001 0) (effects (font (size 1.27 1.27)))) (property "Footprint" "Package_TO_SOT_SMD:TO-252-2" (at 90.17 74.93 0) (effects (font (size 1.27 1.27)) (hide yes))) (property "Design note" "ST DS6906 page1 package: leftlead1 NC, tab2 K, rightlead3 A. External branch fuse coordination and diode thermal validation required." (at 90.17 74.93 0) (effects (font (size 1.27 1.27)) (hide yes))) (pin "1") (pin "2") (pin "3") (instances (project "Power8GDI_Core" (path "/f4d21065-0a5b-5086-a08e-1af9469f04bd/30a46de9-e11a-54b6-8706-ae1bab93f93c" (reference "D5610") (unit 1))) (project "wbo1_heater_feed" (path "/a54f5754-f64a-5b39-be6f-e9eea49aaacf" (reference "D5610") (unit 1)))))
 (no_connect (at 72.39 73.66))
 (wire (pts (xy 72.39 76.2) (xy 64.77 76.2)) (stroke (width 0) (type default)))
@@
 (wire (pts (xy 107.95 73.66) (xy 115.57 73.66)) (stroke (width 0) (type default)))
 (global_label "VBAT_MAIN_FUSED" (shape bidirectional) (at 115.57 73.66 180) (effects (font (size 1.016 1.016)) (justify left bottom)))
-(symbol (lib_id "Power8GDI_Aux:WBO_SMBJ24CA") (at 245.11 74.93 0) (unit 1) (in_bom yes) (on_board yes) (dnp no) (property "Reference" "D5611" (at 245.11 67.31 0) (effects (font (size 1.27 1.27)))) (property "Value" "SMBJ24CA" (at 245.11 82.55000000000001 0) (effects (font (size 1.27 1.27)))) (property "Footprint" "Diode_SMD:D_SMB" (at 245.11 74.93 0) (effects (font (size 1.27 1.27)) (hide yes))) (property "Design note" "38.9V ratedclamp nominal <40V switch minimumclamp; overshoot/pulse energy still unqualified." (at 245.11 74.93 0) (effects (font (size 1.27 1.27)) (hide yes))) (pin "1") (pin "2") (instances (project "Power8GDI_Core" (path "/f4d21065-0a5b-5086-a08e-1af9469f04bd/30a46de9-e11a-54b6-8706-ae1bab93f93c" (reference "D5611") (unit 1))) (project "wbo1_heater_feed" (path "/a54f5754-f64a-5b39-be6f-e9eea49aaacf" (reference "D5611") (unit 1)))))
+(symbol (lib_id "Power8GDI_WBO:WBO_SMBJ24CA") (at 245.11 74.93 0) (unit 1) (in_bom yes) (on_board yes) (dnp no) (property "Reference" "D5611" (at 245.11 67.31 0) (effects (font (size 1.27 1.27)))) (property "Value" "SMBJ24CA" (at 245.11 82.55000000000001 0) (effects (font (size 1.27 1.27)))) (property "Footprint" "Diode_SMD:D_SMB" (at 245.11 74.93 0) (effects (font (size 1.27 1.27)) (hide yes))) (property "Design note" "38.9V ratedclamp nominal <40V switch minimumclamp; overshoot/pulse energy still unqualified." (at 245.11 74.93 0) (effects (font (size 1.27 1.27)) (hide yes))) (pin "1") (pin "2") (instances (project "Power8GDI_Core" (path "/f4d21065-0a5b-5086-a08e-1af9469f04bd/30a46de9-e11a-54b6-8706-ae1bab93f93c" (reference "D5611") (unit 1))) (project "wbo1_heater_feed" (path "/a54f5754-f64a-5b39-be6f-e9eea49aaacf" (reference "D5611") (unit 1)))))
 (wire (pts (xy 227.33 74.93) (xy 219.71 74.93)) (stroke (width 0) (type default)))
 (global_label "HARNESS_WBO1_CONTACT4" (shape bidirectional) (at 219.71 74.93 0) (effects (font (size 1.016 1.016)) (justify right bottom)))
 (wire (pts (xy 262.89 74.93) (xy 270.51 74.93)) (stroke (width 0) (type default)))
 (global_label "GND" (shape bidirectional) (at 270.51 74.93 180) (effects (font (size 1.016 1.016)) (justify left bottom)))
-(symbol (lib_id "Power8GDI_Aux:WBO_C") (at 90.17 144.78 0) (unit 1) (in_bom yes) (on_board yes) (dnp no) (property "Reference" "C5650" (at 94.17 143.51 0) (effects (font (size 1.27 1.27)) (justify left))) (property "Value" "100n 100V X7R" (at 94.17 146.05 0) (effects (font (size 1.27 1.27)) (justify left))) (property "Footprint" "Capacitor_SMD:C_0805_2012Metric" (at 90.17 144.78 0) (effects (font (size 1.27 1.27)) (hide yes))) (property "Design note" "" (at 90.17 144.78 0) (effects (font (size 1.27 1.27)) (hide yes))) (pin "1") (pin "2") (instances (project "Power8GDI_Core" (path "/f4d21065-0a5b-5086-a08e-1af9469f04bd/30a46de9-e11a-54b6-8706-ae1bab93f93c" (reference "C5650") (unit 1))) (project "wbo1_heater_feed" (path "/a54f5754-f64a-5b39-be6f-e9eea49aaacf" (reference "C5650") (unit 1)))))
+(symbol (lib_id "Power8GDI_WBO:WBO_C") (at 90.17 144.78 0) (unit 1) (in_bom yes) (on_board yes) (dnp no) (property "Reference" "C5650" (at 94.17 143.51 0) (effects (font (size 1.27 1.27)) (justify left))) (property "Value" "100n 100V X7R" (at 94.17 146.05 0) (effects (font (size 1.27 1.27)) (justify left))) (property "Footprint" "Capacitor_SMD:C_0805_2012Metric" (at 90.17 144.78 0) (effects (font (size 1.27 1.27)) (hide yes))) (property "Design note" "" (at 90.17 144.78 0) (effects (font (size 1.27 1.27)) (hide yes))) (pin "1") (pin "2") (instances (project "Power8GDI_Core" (path "/f4d21065-0a5b-5086-a08e-1af9469f04bd/30a46de9-e11a-54b6-8706-ae1bab93f93c" (reference "C5650") (unit 1))) (project "wbo1_heater_feed" (path "/a54f5754-f64a-5b39-be6f-e9eea49aaacf" (reference "C5650") (unit 1)))))
 (wire (pts (xy 85.09 144.78) (xy 77.47 144.78)) (stroke (width 0) (type default)))
 (global_label "HARNESS_WBO1_CONTACT4" (shape bidirectional) (at 77.47 144.78 0) (effects (font (size 1.016 1.016)) (justify right bottom)))
 (wire (pts (xy 95.25 144.78) (xy 102.87 144.78)) (stroke (width 0) (type default)))
 (global_label "GND" (shape bidirectional) (at 102.87 144.78 180) (effects (font (size 1.016 1.016)) (justify left bottom)))
-(symbol (lib_id "Power8GDI_Aux:WBO_C") (at 245.11 144.78 0) (unit 1) (in_bom yes) (on_board yes) (dnp no) (property "Reference" "C5651" (at 249.11 143.51 0) (effects (font (size 1.27 1.27)) (justify left))) (property "Value" "47u 63V lowESR" (at 249.11 146.05 0) (effects (font (size 1.27 1.27)) (justify left))) (property "Footprint" "Capacitor_SMD:CP_Elec_8x10" (at 245.11 144.78 0) (effects (font (size 1.27 1.27)) (hide yes))) (property "Design note" "Provisional bulk MPN/ripple and cold ESR pending." (at 245.11 144.78 0) (effects (font (size 1.27 1.27)) (hide yes))) (pin "1") (pin "2") (instances (project "Power8GDI_Core" (path "/f4d21065-0a5b-5086-a08e-1af9469f04bd/30a46de9-e11a-54b6-8706-ae1bab93f93c" (reference "C5651") (unit 1))) (project "wbo1_heater_feed" (path "/a54f5754-f64a-5b39-be6f-e9eea49aaacf" (reference "C5651") (unit 1)))))
+(symbol (lib_id "Power8GDI_WBO:WBO_C") (at 245.11 144.78 0) (unit 1) (in_bom yes) (on_board yes) (dnp no) (property "Reference" "C5651" (at 249.11 143.51 0) (effects (font (size 1.27 1.27)) (justify left))) (property "Value" "47u 63V lowESR" (at 249.11 146.05 0) (effects (font (size 1.27 1.27)) (justify left))) (property "Footprint" "Capacitor_SMD:CP_Elec_8x10" (at 245.11 144.78 0) (effects (font (size 1.27 1.27)) (hide yes))) (property "Design note" "Provisional bulk MPN/ripple and cold ESR pending." (at 245.11 144.78 0) (effects (font (size 1.27 1.27)) (hide yes))) (pin "1") (pin "2") (instances (project "Power8GDI_Core" (path "/f4d21065-0a5b-5086-a08e-1af9469f04bd/30a46de9-e11a-54b6-8706-ae1bab93f93c" (reference "C5651") (unit 1))) (project "wbo1_heater_feed" (path "/a54f5754-f64a-5b39-be6f-e9eea49aaacf" (reference "C5651") (unit 1)))))
 (wire (pts (xy 240.03 144.78) (xy 232.41 144.78)) (stroke (width 0) (type default)))
 (global_label "HARNESS_WBO1_CONTACT4" (shape bidirectional) (at 232.41 144.78 0) (effects (font (size 1.016 1.016)) (justify right bottom)))

Commit message: Review B58 injector power stage and bind selected GDI6 BOM
Parts:
- C5650: Hardware_Qualification (none) -> BOARD_QUALIFICATION_PENDING; MPN (none) -> C0805C104K1RACTU; Manufacturer (none) -> KEMET; Procurement_Status (none) -> SELECTED_CATALOG_ITEM; Purchase_Released (none) -> false; Selection_Gaps (none) -> []; Selection_ID (none) -> SEL-50b208aec5b1; Selection_Ratings (none) -> {"capacitance_pf": 100000, "dielectric": "X7R", "rated_volt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; Selection_Source_URLs (none) -> https://www.mouser.com/datasheet/3/72/1/C0805C104K1RACTU.pdf
- C5651: Hardware_Qualification (none) -> LAND_PATTERN_AND_RIPPLE_REVIEW_REQUIRED; MPN (none) -> EEH-ZC1J470P; Manufacturer (none) -> Panasonic Industry; Procurement_Status (none) -> SELECTED_CONDITIONAL; Purchase_Released (none) -> false; Selection_Gaps (none) -> ["Source footprint CP_Elec_8x10; selected part maximum seat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; Selection_ID (none) -> SEL-43cb48863fb5; Selection_Ratings (none) -> {"aec_q200": true, "capacitance_pf": 47000000, "diameter_mm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; Selection_Source_URLs (none) -> https://www.digikey.com/en/products/detail/panasonic-indust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
- D5610: Hardware_Qualification (none) -> PINOUT_RATINGS_AND_DELIVERY_SUFFIX_REVIEW_PENDING; MPN (none) -> STPS5H100BY-TR; Manufacturer (none) -> STMicroelectronics; Procurement_Status (none) -> REFERENCE_MPN_RETAINED; Purchase_Released (none) -> false; Selection_Gaps (none) -> ["Existing schematic MPN retained. Complete circuit rating/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; Selection_ID (none) -> SEL-474c4e2ea71d; Selection_Ratings (none) -> {}; Selection_Source_URLs (none) -> https://www.st.com/en/search.html#q=STPS5H100BY-TR
- D5611: Hardware_Qualification (none) -> PINOUT_RATINGS_AND_DELIVERY_SUFFIX_REVIEW_PENDING; MPN (none) -> SMBJ24CA; Manufacturer (none) -> Littelfuse; Procurement_Status (none) -> REFERENCE_MPN_RETAINED; Purchase_Released (none) -> false; Selection_Gaps (none) -> ["Existing schematic MPN retained. Complete circuit rating/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; Selection_ID (none) -> SEL-9a26101f9da7; Selection_Ratings (none) -> {}; Selection_Source_URLs (none) -> https://www.littelfuse.com/products/tvs-diodes/surface-moun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
