File: Power8GDI/hardware/design/wbo/wbo1_control.kicad_sch (KiCad schematic)
At the start: 37 parts, among them J5600 Conn_02x03_Odd_Even, Q5600 VND7NV04TR-E, U5602 STM32F042K6T6, U5604 XC6206P332MR-G, U5605 TJA1051T/3/1J, U5610 SN74LVC1G08QDBVRQ1, U5611 SN74AHCT1G125QDBVRQ1

Commit message: Isolate WBO symbol namespace for root schematic integration
Parts:
- C5602, C5609, C5610, C5613, C5614, C5615, C5616, C5617, C5618, C5640, C5641: symbol Power8GDI_Aux:WBO_C -> Power8GDI_WBO:WBO_C
- D5600: symbol Power8GDI_Aux:WBO_D600_mapped -> Power8GDI_WBO:WBO_D600_mapped
- D5601: symbol Power8GDI_Aux:WBO_D601_mapped -> Power8GDI_WBO:WBO_D601_mapped
- D5602: symbol Power8GDI_Aux:WBO_D602_mapped -> Power8GDI_WBO:WBO_D602_mapped
- D5603: symbol Power8GDI_Aux:WBO_D603_mapped -> Power8GDI_WBO:WBO_D603_mapped
- D5604: symbol Power8GDI_Aux:WBO_D604_mapped -> Power8GDI_WBO:WBO_D604_mapped
- J5600: symbol Power8GDI_Aux:WBO_J600_mapped -> Power8GDI_WBO:WBO_J600_mapped
- Q5600: symbol Power8GDI_Aux:WBO_Q600_mapped -> Power8GDI_WBO:WBO_Q600_mapped
- R5616, R5617, R5622, R5625, R5626, R5627, R5628, R5629, R5640, R5641, R5642, R5643, R5644, R5645: symbol Power8GDI_Aux:WBO_R -> Power8GDI_WBO:WBO_R
- U5602: symbol Power8GDI_Aux:WBO_U602_mapped -> Power8GDI_WBO:WBO_U602_mapped
- U5604: symbol Power8GDI_Aux:WBO_U604_mapped -> Power8GDI_WBO:WBO_U604_mapped
- U5605: symbol Power8GDI_Aux:WBO_U605_mapped -> Power8GDI_WBO:WBO_U605_mapped
- U5610: symbol Power8GDI_Aux:WBO_SN74LVC1G08 -> Power8GDI_WBO:WBO_SN74LVC1G08
- U5611: symbol Power8GDI_Aux:WBO_SN74AHCT1G125 -> Power8GDI_WBO:WBO_SN74AHCT1G125

Commit message: Fix WBO analog net collisions and independently audit source connectivity
Connections:
- net WBO1_Net_D600_A renamed WBO1_AUTO_Net_2D__28_D600_2D_A_29_
- net WBO1_Net_D601_K renamed WBO1_AUTO_Net_2D__28_D601_2D_K_29_
- net WBO1_Net_D602_K renamed WBO1_AUTO_Net_2D__28_D602_2D_K_29_
- net WBO1_Net_D603_A renamed WBO1_AUTO_Net_2D__28_D603_2D_A_29_
- net WBO1_Net_Q600_G renamed WBO1_AUTO_Net_2D__28_Q600_2D_G_29_

Commit message: Fix WBO VDDA sequencing with precision buffered common rail and local reset
Parts:
- added C5660, C5663, C5664: 100n 16V X7R, Capacitor_SMD:C_0603_1608Metric, symbol Power8GDI_WBO:WBO_C
- added C5661, C5662: 10u 16V X7R effective>=4.7u, Capacitor_SMD:C_1206_3216Metric, symbol Power8GDI_WBO:WBO_C
- added R5660: 30k 0.1%, Resistor_SMD:R_0603_1608Metric, symbol Power8GDI_WBO:WBO_R
- added R5661: 2.2k 1%, Resistor_SMD:R_0603_1608Metric, symbol Power8GDI_WBO:WBO_R
- added R5662: 10k, Resistor_SMD:R_0603_1608Metric, symbol Power8GDI_WBO:WBO_R
- added R5663: 220R 0.1%, Resistor_SMD:R_0603_1608Metric, symbol Power8GDI_WBO:WBO_R
- added U5612: TPS3808G33QDBVRQ1, Package_TO_SOT_SMD:SOT-23-6, symbol Power8GDI_WBO:WBO_TPS3808G33
- U5604: value XC6206P332MR-G -> LT3042IMSE#WTRPBF; footprint Package_TO_SOT_SMD:SOT-23 -> Package_SO:MSOP-10-1EP_3x3mm_P0.5mm_EP1.68x1.88mm; Design note Pinned Hellen 0.6 source U604; netlist-derived. -> LT3042 RevC p15 external reference buffer; replaces XC6206.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
Connections:
- net WBO1_VDDA is gone; now on net WBO1_3V3: U5602.5 (VDDA)
- net +5V_CORE: now also U5604.1 (IN), U5604.2 (IN), U5604.6 (PGFB), C5661.1
- net GND: now also U5604.11 (EP_GND), U5604.5 (ILIM), U5604.8 (GND), C5660.2, C5661.2, C5662.2, C5663.2, C5664.2, R5660.2, R5661.2, U5612.2 (GND); no longer U5604.1 (GND)
- net WBO1_3V3: now also U5604.10 (OUT), U5604.9 (OUTS), C5662.1, C5663.1, R5661.1, R5662.2, U5612.3 (~{MR}), U5612.5 (SENSE), U5612.6 (VDD); no longer U5604.2 (VO)
- net WBO1_nRESET: now also R5662.1, U5612.1 (~{RESET})
- new net WBO1_REF3V3: C5664.1, R5663.1
- new net WBO1_REF_SET: C5660.1, R5660.1, R5663.2, U5604.7 (SET)
- no-connect marks 10 -> 12
Other:
- moved on the sheet: C5602, C5609, C5610, C5613, C5614, C5615, C5616, C5617, C5618, C5640, C5641, D5600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

Commit message: Keep WBO heater inhibit disabled when main 3V3 is absent
Parts:
- added Q5620: BC847B-QR, Package_TO_SOT_SMD:SOT-23, symbol Power8GDI_WBO:WBO_BC847B_Q
- added R5664: 4.7k 1%, Resistor_SMD:R_0603_1608Metric, symbol Power8GDI_WBO:WBO_R
- added R5665: 10k 1%, Resistor_SMD:R_0603_1608Metric, symbol Power8GDI_WBO:WBO_R
- R5642: value 10k -> 2.2k 1%
- U5611: Design note TTL input accepts3V3; disabled by independent global hardwa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 -> OE local5V pull-up defaults disabled; NPN level shift enabl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
Connections:
- net +3V3 is gone; now on net +5V_CORE: R5642.2
- net GND: now also Q5620.2 (EMITTER), R5665.2
- net HW_ACTUATOR_ENABLE_N renamed WBO1_HEATER_OE_N
- net WBO1_HEATER_OE_N: now also Q5620.3 (COLLECTOR)
- new net HW_ACTUATOR_ENABLE: R5664.1
- new net WBO1_HEATER_OE_BASE: Q5620.1 (BASE), R5664.2, R5665.1

Commit message: Review B58 injector power stage and bind selected GDI6 BOM
Parts:
- C5602, C5613, C5614, C5615, C5617, C5618, C5640, C5641, C5660, C5663, C5664: Hardware_Qualification (none) -> BOARD_QUALIFICATION_PENDING; MPN (none) -> C0603C104K5RACTU; Manufacturer (none) -> KEMET; Procurement_Status (none) -> SELECTED_CATALOG_ITEM; Purchase_Released (none) -> false; Selection_Gaps (none) -> []; Selection_ID (none) -> SEL-6bf9727c4e40; Selection_Ratings (none) -> {"capacitance_pf": 100000, "dielectric": "X7R", "rated_volt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; Selection_Source_URLs (none) -> https://search.kemet.com/download/specsheet/C0603C104K5RACTU
- C5609, C5610: Hardware_Qualification (none) -> BOARD_QUALIFICATION_PENDING; MPN (none) -> C0603C105K3RACTU; Manufacturer (none) -> KEMET; Procurement_Status (none) -> SELECTED_CATALOG_ITEM; Purchase_Released (none) -> false; Selection_Gaps (none) -> []; Selection_ID (none) -> SEL-4bca20b134b8; Selection_Ratings (none) -> {"capacitance_pf": 1000000, "dc_bias_qualification": "PENDI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; Selection_Source_URLs (none) -> https://search.kemet.com/download/specsheet/C0603C105K3RACTU
- C5616: Hardware_Qualification (none) -> BOARD_QUALIFICATION_PENDING; MPN (none) -> GMC10X7R475K16NT; Manufacturer (none) -> Cal-Chip Electronics; Procurement_Status (none) -> SELECTED_CATALOG_ITEM; Purchase_Released (none) -> false; Selection_Gaps (none) -> []; Selection_ID (none) -> SEL-541f7eb877a5; Selection_Ratings (none) -> {"capacitance_pf": 4700000, "dc_bias_qualification": "PENDI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; Selection_Source_URLs (none) -> https://www.digikey.com/en/products/detail/cal-chip-electro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
- C5661, C5662: Hardware_Qualification (none) -> BOARD_QUALIFICATION_PENDING; MPN (none) -> C1206C106K4RACTU; Manufacturer (none) -> KEMET; Procurement_Status (none) -> SELECTED_CATALOG_ITEM; Purchase_Released (none) -> false; Selection_Gaps (none) -> ["Required effective capacitance not yet verified with supp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; Selection_ID (none) -> SEL-790f6da303d4; Selection_Ratings (none) -> {"capacitance_pf": 10000000, "dc_bias_qualification": "PEND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; Selection_Source_URLs (none) -> https://search.kemet.com/component-documentation/download/s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
- D5600, D5603: Hardware_Qualification (none) -> LED_CURRENT_AND_VISIBILITY_REVIEW_REQUIRED; MPN (none) -> APT1608SURCK; Manufacturer (none) -> Kingbright; Procurement_Status (none) -> SELECTED_CONDITIONAL; Purchase_Released (none) -> false; Selection_Gaps (none) -> ["20mA is catalog test current, not a configured operating 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; Selection_ID (none) -> SEL-b0d3a57d6d36; Selection_Ratings (none) -> {"body_mm": [1.6, 0.8, 0.75], "color": "red", "test_current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; Selection_Source_URLs (none) -> https://www.kingbrightusa.com/product.asp?catalog_name=LED&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
- D5601: Hardware_Qualification (none) -> LED_CURRENT_AND_VISIBILITY_REVIEW_REQUIRED; MPN (none) -> APT1608SGC; Manufacturer (none) -> Kingbright; Procurement_Status (none) -> SELECTED_CONDITIONAL; Purchase_Released (none) -> false; Selection_Gaps (none) -> ["20mA is catalog test current, not a configured operating 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; Selection_ID (none) -> SEL-3fb09a4358af; Selection_Ratings (none) -> {"body_mm": [1.6, 0.8, 0.75], "color": "green", "test_curre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; Selection_Source_URLs (none) -> https://www.digikey.com/en/products/detail/kingbright/APT16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
- D5602: Hardware_Qualification (none) -> LED_CURRENT_AND_VISIBILITY_REVIEW_REQUIRED; MPN (none) -> APT1608QBC/D; Manufacturer (none) -> Kingbright; Procurement_Status (none) -> SELECTED_CONDITIONAL; Purchase_Released (none) -> false; Selection_Gaps (none) -> ["20mA is catalog test current, not a configured operating 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; Selection_ID (none) -> SEL-3cd22f0f3fe3; Selection_Ratings (none) -> {"body_mm": [1.6, 0.8, 0.75], "color": "blue", "test_curren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; Selection_Source_URLs (none) -> https://www.digikey.com/en/products/detail/kingbright/APT16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
- D5604: Hardware_Qualification (none) -> PINOUT_RATINGS_AND_DELIVERY_SUFFIX_REVIEW_PENDING; MPN (none) -> PESD1CAN,215; Manufacturer (none) -> Nexperia; Procurement_Status (none) -> REFERENCE_MPN_RETAINED; Purchase_Released (none) -> false; Selection_Gaps (none) -> ["Existing schematic MPN retained. Complete circuit rating/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; Selection_ID (none) -> SEL-3e2f1ed25b55; Selection_Ratings (none) -> {}; Selection_Source_URLs (none) -> https://www.nexperia.com/product/PESD1CAN
- Q5600: Hardware_Qualification (none) -> PINOUT_RATINGS_AND_DELIVERY_SUFFIX_REVIEW_PENDING; MPN (none) -> VND7NV04TR-E; Manufacturer (none) -> STMicroelectronics; Procurement_Status (none) -> REFERENCE_MPN_RETAINED; Purchase_Released (none) -> false; Selection_Gaps (none) -> ["Existing schematic MPN retained. Complete circuit rating/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; Selection_ID (none) -> SEL-8ffb4f1a4ad4; Selection_Ratings (none) -> {}; Selection_Source_URLs (none) -> https://www.st.com/en/search.html#q=VND7NV04TR-E
- Q5620: Hardware_Qualification (none) -> PINOUT_RATINGS_AND_DELIVERY_SUFFIX_REVIEW_PENDING; MPN (none) -> BC847B-QR; Manufacturer (none) -> Nexperia; Procurement_Status (none) -> REFERENCE_MPN_RETAINED; Purchase_Released (none) -> false; Selection_Gaps (none) -> ["Existing schematic MPN retained. Complete circuit rating/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; Selection_ID (none) -> SEL-5f4a29315a6b; Selection_Ratings (none) -> {}; Selection_Source_URLs (none) -> https://www.nexperia.com/product/BC847B-QR
- R5616, R5617, R5622, R5626, R5627, R5628: Hardware_Qualification (none) -> BOARD_QUALIFICATION_PENDING; MPN (none) -> CRCW06031K00FKEA; Manufacturer (none) -> Vishay; Procurement_Status (none) -> SELECTED_FAMILY_CODE; Purchase_Released (none) -> false; Selection_Gaps (none) -> []; Selection_ID (none) -> SEL-38197231a947; Selection_Ratings (none) -> {"aec_q200": true, "derating": "Use manufacturer power vers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; Selection_Source_URLs (none) -> https://www.vishay.com/docs/20035/dcrcwe3.pdf
- R5625, R5640, R5641, R5643, R5662, R5665: Hardware_Qualification (none) -> BOARD_QUALIFICATION_PENDING; MPN (none) -> CRCW060310K0FKEA; Manufacturer (none) -> Vishay; Procurement_Status (none) -> SELECTED_FAMILY_CODE; Purchase_Released (none) -> false; Selection_Gaps (none) -> []; Selection_ID (none) -> SEL-9c0806476875; Selection_Ratings (none) -> {"aec_q200": true, "derating": "Use manufacturer power vers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; Selection_Source_URLs (none) -> https://www.vishay.com/docs/20035/dcrcwe3.pdf
- R5642, R5661: Hardware_Qualification (none) -> BOARD_QUALIFICATION_PENDING; MPN (none) -> CRCW06032K20FKEA; Manufacturer (none) -> Vishay; Procurement_Status (none) -> SELECTED_FAMILY_CODE; Purchase_Released (none) -> false; Selection_Gaps (none) -> []; Selection_ID (none) -> SEL-77653d639f50; Selection_Ratings (none) -> {"aec_q200": true, "derating": "Use manufacturer power vers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; Selection_Source_URLs (none) -> https://www.vishay.com/docs/20035/dcrcwe3.pdf
- R5644: Hardware_Qualification (none) -> BOARD_QUALIFICATION_PENDING; MPN (none) -> CRCW06030000Z0EA; Manufacturer (none) -> Vishay; Procurement_Status (none) -> SELECTED_FAMILY_CODE; Purchase_Released (none) -> false; Selection_Gaps (none) -> []; Selection_ID (none) -> SEL-8473f02313b2; Selection_Ratings (none) -> {"aec_q200": true, "current_a": 2, "power_reference_tempera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; Selection_Source_URLs (none) -> https://www.vishay.com/docs/20035/dcrcwe3.pdf
- R5645: Hardware_Qualification (none) -> BOARD_QUALIFICATION_PENDING; MPN (none) -> CRCW0603100KFKEA; Manufacturer (none) -> Vishay; Procurement_Status (none) -> SELECTED_FAMILY_CODE; Purchase_Released (none) -> false; Selection_Gaps (none) -> []; Selection_ID (none) -> SEL-4e3f06cba0aa; Selection_Ratings (none) -> {"aec_q200": true, "derating": "Use manufacturer power vers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; Selection_Source_URLs (none) -> https://www.vishay.com/docs/20035/dcrcwe3.pdf
- R5660: Hardware_Qualification (none) -> BOARD_QUALIFICATION_PENDING; MPN (none) -> RNCF0603BTE30K0; Manufacturer (none) -> Stackpole Electronics; Procurement_Status (none) -> SELECTED_CATALOG_ITEM; Purchase_Released (none) -> false; Selection_Gaps (none) -> []; Selection_ID (none) -> SEL-f81c6e7cae8d; Selection_Ratings (none) -> {"aec_q200": true, "derating": "Use manufacturer power vers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; Selection_Source_URLs (none) -> https://www.digikey.com/en/products/detail/stackpole-electr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
- R5663: Hardware_Qualification (none) -> BOARD_QUALIFICATION_PENDING; MPN (none) -> RNCF0603BTE220R; Manufacturer (none) -> Stackpole Electronics; Procurement_Status (none) -> SELECTED_CATALOG_ITEM; Purchase_Released (none) -> false; Selection_Gaps (none) -> []; Selection_ID (none) -> SEL-b9ddc1a3febb; Selection_Ratings (none) -> {"aec_q200": true, "derating": "Use manufacturer power vers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; Selection_Source_URLs (none) -> https://www.mouser.ca/en/ProductDetail/SEI-Stackpole/RNCF06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
- R5664: Hardware_Qualification (none) -> BOARD_QUALIFICATION_PENDING; MPN (none) -> CRCW06034K70FKEA; Manufacturer (none) -> Vishay; Procurement_Status (none) -> SELECTED_FAMILY_CODE; Purchase_Released (none) -> false; Selection_Gaps (none) -> []; Selection_ID (none) -> SEL-1f010ac9622d; Selection_Ratings (none) -> {"aec_q200": true, "derating": "Use manufacturer power vers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; Selection_Source_URLs (none) -> https://www.vishay.com/docs/20035/dcrcwe3.pdf
- U5602: Hardware_Qualification (none) -> PINOUT_RATINGS_AND_DELIVERY_SUFFIX_REVIEW_PENDING; MPN (none) -> STM32F042K6T6; Manufacturer (none) -> STMicroelectronics; Procurement_Status (none) -> REFERENCE_MPN_RETAINED; Purchase_Released (none) -> false; Selection_Gaps (none) -> ["Existing schematic MPN retained. Complete circuit rating/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; Selection_ID (none) -> SEL-819996afcb95; Selection_Ratings (none) -> {}; Selection_Source_URLs (none) -> https://www.st.com/en/search.html#q=STM32F042K6T6
- U5604: Hardware_Qualification (none) -> OUTPUT_CAPACITY_AND_THERMAL_REVIEW_REQUIRED; MPN (none) -> LT3042IMSE#WTRPBF; Manufacturer (none) -> Analog Devices; Procurement_Status (none) -> SELECTED_CONDITIONAL; Purchase_Released (none) -> false; Selection_Gaps (none) -> ["Automotive W order suffix retained; pricing must not sile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; Selection_ID (none) -> SEL-3841e4a3c00c; Selection_Ratings (none) -> {"output_current_catalog_a": 0.2, "output_max_v": 15, "outp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; Selection_Source_URLs (none) -> https://www.analog.com/en/products/lt3042.html
- U5605: Hardware_Qualification (none) -> PINOUT_RATINGS_AND_DELIVERY_SUFFIX_REVIEW_PENDING; MPN (none) -> TJA1051T/3/1J; Manufacturer (none) -> NXP Semiconductors; Procurement_Status (none) -> REFERENCE_MPN_RETAINED; Purchase_Released (none) -> false; Selection_Gaps (none) -> ["Existing schematic MPN retained. Complete circuit rating/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; Selection_ID (none) -> SEL-ec8a3bf80ff2; Selection_Ratings (none) -> {}; Selection_Source_URLs (none) -> https://www.nxp.com/docs/en/data-sheet/TJA1051.pdf
- U5610: Hardware_Qualification (none) -> PINOUT_RATINGS_AND_DELIVERY_SUFFIX_REVIEW_PENDING; MPN (none) -> SN74LVC1G08QDBVRQ1; Manufacturer (none) -> Texas Instruments; Procurement_Status (none) -> REFERENCE_MPN_RETAINED; Purchase_Released (none) -> false; Selection_Gaps (none) -> ["Existing schematic MPN retained. Complete circuit rating/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; Selection_ID (none) -> SEL-617c05649839; Selection_Ratings (none) -> {}; Selection_Source_URLs (none) -> https://www.ti.com/product/SN74LVC1G08-Q1/part-details/SN74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
- U5611: Hardware_Qualification (none) -> PINOUT_RATINGS_AND_DELIVERY_SUFFIX_REVIEW_PENDING; MPN (none) -> SN74AHCT1G125QDBVRQ1; Manufacturer (none) -> Texas Instruments; Procurement_Status (none) -> REFERENCE_MPN_RETAINED; Purchase_Released (none) -> false; Selection_Gaps (none) -> ["Existing schematic MPN retained. Complete circuit rating/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; Selection_ID (none) -> SEL-209b18127c6b; Selection_Ratings (none) -> {}; Selection_Source_URLs (none) -> https://www.ti.com/product/SN74AHCT1G125-Q1/part-details/SN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
- U5612: Hardware_Qualification (none) -> PINOUT_RATINGS_AND_DELIVERY_SUFFIX_REVIEW_PENDING; MPN (none) -> TPS3808G33QDBVRQ1; Manufacturer (none) -> Texas Instruments; Procurement_Status (none) -> REFERENCE_MPN_RETAINED; Purchase_Released (none) -> false; Selection_Gaps (none) -> ["Existing schematic MPN retained. Complete circuit rating/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; Selection_ID (none) -> SEL-36c2480848bd; Selection_Ratings (none) -> {}; Selection_Source_URLs (none) -> https://www.ti.com/product/TPS3808-Q1/part-details/TPS3808G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

Commit message: fix(gdi6): clear D5604 silk with a matched local footprint
Parts:
- D5604: footprint Package_TO_SOT_SMD:SOT-23 -> Power8GDI_Board:SOT-23_D5604_J5600_Clearance
Changed lines of the file:
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@@
         (font
           (size 1.27 1.27))))
-    (property "Footprint" "Package_TO_SOT_SMD:SOT-23"
+    (property "Footprint" "Power8GDI_Board:SOT-23_D5604_J5600_Clearance"
       (at 449.58 199.39 0)
       (effects
