File: Power8GDI/hardware/design/Power8GDI_Core.kicad_sch (KiCad schematic)
At the start: 0 parts

Commit message: Integrate connected ECU schematic and auditable review PCB
Other:
- added sheet Buffered analog inputs 1..4 (io/analog_1.kicad_sch)
- added sheet Buffered analog inputs 13..16 (io/analog_4.kicad_sch)
- added sheet Buffered analog inputs 17..17 (io/analog_5.kicad_sch)
- added sheet Buffered analog inputs 5..8 (io/analog_2.kicad_sch)
- added sheet Buffered analog inputs 9..12 (io/analog_3.kicad_sch)
- added sheet DBW H-bridge candidate (motor/dbw_driver.kicad_sch)
- added sheet Differential VR crank receiver (io/crank_vr.kicad_sch)
- added sheet EWG H-bridge candidate (motor/ewg_driver.kicad_sch)
- added sheet Four TE34 harness connectors (board/connectors.kicad_sch)
- added sheet Hall and SENT receiver bank 1 (io/digital_1.kicad_sch)
- added sheet Hall and SENT receiver bank 2 (io/digital_2.kicad_sch)
- added sheet Latched hardware permission (safety/safety_gate.kicad_sch)
- note added: "Each sheet uses explicit global net names. HARNESS names remain separate from MCU logic. No ERC exclusions or power flags conceal missing supplies. DNP assembly flags must be preserved. GDI enable, injector/pump models, missing domains and full routing remain release blockers."
- note added: "Power8GDI electrical candidate / NOT RELEASED Connected hierarchy: MCU, input supply, two GDI stages, safety, motor candidates, sensor frontends and harness. Outstanding channels and load qualification are tracked in INTEGRATION_2026_10_21_ELECTRICAL.md."
- note removed: "Power8GDI electrical candidate / NOT RELEASED Real MCU/power/CAN connectivity; GDI and input protection integrated as separate source-owned sheets. Mapped signal names denote 3V3 logic only. Unmapped channels and electrical frontends remain blocked."
- note removed: "Root supply port +5V_CORE requires root-owned power_input sheet. No PWR_FLAG or ERC exclusion is added to conceal missing supply evidence. U101 unused pins are explicitly NC; these do not satisfy outstanding functional requirements."

Commit message: Add 24 direct protected low-side output circuits with hardware inhibit
Other:
- added sheet Direct protected low-side AUX_PWM1, AUX_PWM2, AUX_PWM3, AUX_PWM4 (outputs/ls_bank_4.kicad_sch)
- added sheet Direct protected low-side AUX_PWM5, AUX_PWM6, AUX_PWM7, AUX_PWM8 (outputs/ls_bank_5.kicad_sch)
- added sheet Direct protected low-side LS_AUX1, LS_AUX2, LS_AUX3, LS_AUX4 (outputs/ls_bank_6.kicad_sch)
- added sheet Direct protected low-side PI1, PI2, PI3, PI4 (outputs/ls_bank_1.kicad_sch)
- added sheet Direct protected low-side PI5, PI6, PI7, PI8 (outputs/ls_bank_2.kicad_sch)
- added sheet Direct protected low-side VVT1, VVT2, VVT3, VVT4 (outputs/ls_bank_3.kicad_sch)
- added sheet Low-side shared SPI and reset (outputs/ls_control.kicad_sch)

Commit message: Checkpoint integrated 37-sheet schematic before Huge scope revision
Other:
- added sheet Additional Hall, flex and digital inputs bank 1 (interfaces/digital_aux_1.kicad_sch)
- added sheet Additional Hall, flex and digital inputs bank 2 (interfaces/digital_aux_2.kicad_sch)
- added sheet CAN2 and LIN2 physical interfaces (interfaces/comms2.kicad_sch)
- added sheet Dual sensor trackers and star returns (interfaces/sensor_power.kicad_sch)
- added sheet Self-powered USB FS device: host VBUS never powers ECU (interfaces/usb_fs.kicad_sch)
- added sheet knock dual (interfaces_aux/knock_dual.kicad_sch)
- added sheet microSD SPI3 logging candidate (interfaces/sd_spi.kicad_sch)
- added sheet wbo adc control (interfaces_aux/wbo_adc_control.kicad_sch)
- added sheet wbo1 analog (interfaces_aux/wbo1_analog.kicad_sch)
- added sheet wbo2 analog (interfaces_aux/wbo2_analog.kicad_sch)
Changed lines of the file:
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@@
 (sheet (at 39.37 435.61) (size 154.94 54.61) (stroke (width 0.254) (type default)) (fill (color 0 0 0 0)) (property "Sheetname" "EWG H-bridge candidate" (at 39.37 434.34 0) (effects (font (size 1.27 1.27)) (justify left))) (property "Sheetfile" "motor/ewg_driver.kicad_sch" (at 39.37 491.49 0) (effects (font (size 1.27 1.27)) (justify left))) (instances (project "Power8GDI_Core" (path "/f4d21065-0a5b-5086-a08e-1af9469f04bd" (page "45")))))
 (sheet (at 229.87 435.61) (size 154.94 54.61) (stroke (width 0.254) (type default)) (fill (color 0 0 0 0)) (property "Sheetname" "Four TE34 harness connectors" (at 229.87 434.34 0) (effects (font (size 1.27 1.27)) (justify left))) (property "Sheetfile" "board/connectors.kicad_sch" (at 229.87 491.49 0) (effects (font (size 1.27 1.27)) (justify left))) (instances (project "Power8GDI_Core" (path "/f4d21065-0a5b-5086-a08e-1af9469f04bd" (page "46")))))
+(sheet (at 420.37 435.61) (size 154.94 54.61) (stroke (width 0.254) (type default)) (fill (color 0 0 0 0)) (property "Sheetname" "CAN2 and LIN2 physical interfaces" (at 420.37 434.34 0) (effects (font (size 1.27 1.27)) (justify left))) (property "Sheetfile" "interfaces/comms2.kicad_sch" (at 420.37 491.49 0) (effects (font (size 1.27 1.27)) (justify left))) (instances (project "Power8GDI_Core" (path "/f4d21065-0a5b-5086-a08e-1af9469f04bd" (page "47")))))
+(sheet (at 609.6 435.61) (size 154.94 54.61) (stroke (width 0.254) (type default)) (fill (color 0 0 0 0)) (property "Sheetname" "Self-powered USB FS device: host VBUS never powers ECU" (at 609.6 434.34 0) (effects (font (size 1.27 1.27)) (justify left))) (property "Sheetfile" "interfaces/usb_fs.kicad_sch" (at 609.6 491.49 0) (effects (font (size 1.27 1.27)) (justify left))) (instances (project "Power8GDI_Core" (path "/f4d21065-0a5b-5086-a08e-1af9469f04bd" (page "48")))))
+(sheet (at 800.1 435.61) (size 154.94 54.61) (stroke (width 0.254) (type default)) (fill (color 0 0 0 0)) (property "Sheetname" "microSD SPI3 logging candidate" (at 800.1 434.34 0) (effects (font (size 1.27 1.27)) (justify left))) (property "Sheetfile" "interfaces/sd_spi.kicad_sch" (at 800.1 491.49 0) (effects (font (size 1.27 1.27)) (justify left))) (instances (project "Power8GDI_Core" (path "/f4d21065-0a5b-5086-a08e-1af9469f04bd" (page "49")))))
+(sheet (at 990.6 435.61) (size 154.94 54.61) (stroke (width 0.254) (type default)) (fill (color 0 0 0 0)) (property "Sheetname" "Dual sensor trackers and star returns" (at 990.6 434.34 0) (effects (font (size 1.27 1.27)) (justify left))) (property "Sheetfile" "interfaces/sensor_power.kicad_sch" (at 990.6 491.49 0) (effects (font (size 1.27 1.27)) (justify left))) (instances (project "Power8GDI_Core" (path "/f4d21065-0a5b-5086-a08e-1af9469f04bd" (page "50")))))
+(sheet (at 39.37 524.51) (size 154.94 54.61) (stroke (width 0.254) (type default)) (fill (color 0 0 0 0)) (property "Sheetname" "Additional Hall, flex and digital inputs bank 1" (at 39.37 523.24 0) (effects (font (size 1.27 1.27)) (justify left))) (property "Sheetfile" "interfaces/digital_aux_1.kicad_sch" (at 39.37 580.39 0) (effects (font (size 1.27 1.27)) (justify left))) (instances (project "Power8GDI_Core" (path "/f4d21065-0a5b-5086-a08e-1af9469f04bd" (page "51")))))
+(sheet (at 229.87 524.51) (size 154.94 54.61) (stroke (width 0.254) (type default)) (fill (color 0 0 0 0)) (property "Sheetname" "Additional Hall, flex and digital inputs bank 2" (at 229.87 523.24 0) (effects (font (size 1.27 1.27)) (justify left))) (property "Sheetfile" "interfaces/digital_aux_2.kicad_sch" (at 229.87 580.39 0) (effects (font (size 1.27 1.27)) (justify left))) (instances (project "Power8GDI_Core" (path "/f4d21065-0a5b-5086-a08e-1af9469f04bd" (page "52")))))
+(sheet (at 420.37 524.51) (size 154.94 54.61) (stroke (width 0.254) (type default)) (fill (color 0 0 0 0)) (property "Sheetname" "knock dual" (at 420.37 523.24 0) (effects (font (size 1.27 1.27)) (justify left))) (property "Sheetfile" "interfaces_aux/knock_dual.kicad_sch" (at 420.37 580.39 0) (effects (font (size 1.27 1.27)) (justify left))) (instances (project "Power8GDI_Core" (path "/f4d21065-0a5b-5086-a08e-1af9469f04bd" (page "53")))))
+(sheet (at 609.6 524.51) (size 154.94 54.61) (stroke (width 0.254) (type default)) (fill (color 0 0 0 0)) (property "Sheetname" "wbo1 analog" (at 609.6 523.24 0) (effects (font (size 1.27 1.27)) (justify left))) (property "Sheetfile" "interfaces_aux/wbo1_analog.kicad_sch" (at 609.6 580.39 0) (effects (font (size 1.27 1.27)) (justify left))) (instances (project "Power8GDI_Core" (path "/f4d21065-0a5b-5086-a08e-1af9469f04bd" (page "54")))))
+(sheet (at 800.1 524.51) (size 154.94 54.61) (stroke (width 0.254) (type default)) (fill (color 0 0 0 0)) (property "Sheetname" "wbo2 analog" (at 800.1 523.24 0) (effects (font (size 1.27 1.27)) (justify left))) (property "Sheetfile" "interfaces_aux/wbo2_analog.kicad_sch" (at 800.1 580.39 0) (effects (font (size 1.27 1.27)) (justify left))) (instances (project "Power8GDI_Core" (path "/f4d21065-0a5b-5086-a08e-1af9469f04bd" (page "55")))))
+(sheet (at 990.6 524.51) (size 154.94 54.61) (stroke (width 0.254) (type default)) (fill (color 0 0 0 0)) (property "Sheetname" "wbo adc control" (at 990.6 523.24 0) (effects (font (size 1.27 1.27)) (justify left))) (property "Sheetfile" "interfaces_aux/wbo_adc_control.kicad_sch" (at 990.6 580.39 0) (effects (font (size 1.27 1.27)) (justify left))) (instances (project "Power8GDI_Core" (path "/f4d21065-0a5b-5086-a08e-1af9469f04bd" (page "56")))))
 (text "Each sheet uses explicit global net names. HARNESS names remain separate from MCU logic.\nNo ERC exclusions or power flags conceal missing supplies. DNP assembly flags must be preserved.\nGDI enable, injector/pump models, missing domains and full routing remain release blockers." (at 25.4 745 0) (effects (font (size 1.27 1.27)) (justify left top)))
 (sheet_instances (path "/" (page "1"))))

Commit message: Integrate protected GDI and CAN wideband nodes with Huge channel allocation
Other:
- removed sheet Additional Hall, flex and digital inputs bank 2
- removed sheet wbo adc control
- removed sheet wbo1 analog
- removed sheet wbo2 analog
- added sheet gdi/permission (gdi/permission.kicad_sch)
- added sheet gdi/protection a (gdi/protection_a.kicad_sch)
- added sheet gdi/protection b (gdi/protection_b.kicad_sch)
- added sheet wbo/wbo1 analog (wbo/wbo1_analog.kicad_sch)
- added sheet wbo/wbo1 control (wbo/wbo1_control.kicad_sch)
- added sheet wbo/wbo1 heater feed (wbo/wbo1_heater_feed.kicad_sch)
- added sheet wbo/wbo2 analog (wbo/wbo2_analog.kicad_sch)
- added sheet wbo/wbo2 control (wbo/wbo2_control.kicad_sch)
- added sheet wbo/wbo2 heater feed (wbo/wbo2_heater_feed.kicad_sch)
Changed lines of the file:
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@@
 (sheet (at 990.6 435.61) (size 154.94 54.61) (stroke (width 0.254) (type default)) (fill (color 0 0 0 0)) (property "Sheetname" "Dual sensor trackers and star returns" (at 990.6 434.34 0) (effects (font (size 1.27 1.27)) (justify left))) (property "Sheetfile" "interfaces/sensor_power.kicad_sch" (at 990.6 491.49 0) (effects (font (size 1.27 1.27)) (justify left))) (instances (project "Power8GDI_Core" (path "/f4d21065-0a5b-5086-a08e-1af9469f04bd" (page "50")))))
 (sheet (at 39.37 524.51) (size 154.94 54.61) (stroke (width 0.254) (type default)) (fill (color 0 0 0 0)) (property "Sheetname" "Additional Hall, flex and digital inputs bank 1" (at 39.37 523.24 0) (effects (font (size 1.27 1.27)) (justify left))) (property "Sheetfile" "interfaces/digital_aux_1.kicad_sch" (at 39.37 580.39 0) (effects (font (size 1.27 1.27)) (justify left))) (instances (project "Power8GDI_Core" (path "/f4d21065-0a5b-5086-a08e-1af9469f04bd" (page "51")))))
-(sheet (at 229.87 524.51) (size 154.94 54.61) (stroke (width 0.254) (type default)) (fill (color 0 0 0 0)) (property "Sheetname" "Additional Hall, flex and digital inputs bank 2" (at 229.87 523.24 0) (effects (font (size 1.27 1.27)) (justify left))) (property "Sheetfile" "interfaces/digital_aux_2.kicad_sch" (at 229.87 580.39 0) (effects (font (size 1.27 1.27)) (justify left))) (instances (project "Power8GDI_Core" (path "/f4d21065-0a5b-5086-a08e-1af9469f04bd" (page "52")))))
-(sheet (at 420.37 524.51) (size 154.94 54.61) (stroke (width 0.254) (type default)) (fill (color 0 0 0 0)) (property "Sheetname" "knock dual" (at 420.37 523.24 0) (effects (font (size 1.27 1.27)) (justify left))) (property "Sheetfile" "interfaces_aux/knock_dual.kicad_sch" (at 420.37 580.39 0) (effects (font (size 1.27 1.27)) (justify left))) (instances (project "Power8GDI_Core" (path "/f4d21065-0a5b-5086-a08e-1af9469f04bd" (page "53")))))
-(sheet (at 609.6 524.51) (size 154.94 54.61) (stroke (width 0.254) (type default)) (fill (color 0 0 0 0)) (property "Sheetname" "wbo1 analog" (at 609.6 523.24 0) (effects (font (size 1.27 1.27)) (justify left))) (property "Sheetfile" "interfaces_aux/wbo1_analog.kicad_sch" (at 609.6 580.39 0) (effects (font (size 1.27 1.27)) (justify left))) (instances (project "Power8GDI_Core" (path "/f4d21065-0a5b-5086-a08e-1af9469f04bd" (page "54")))))
-(sheet (at 800.1 524.51) (size 154.94 54.61) (stroke (width 0.254) (type default)) (fill (color 0 0 0 0)) (property "Sheetname" "wbo2 analog" (at 800.1 523.24 0) (effects (font (size 1.27 1.27)) (justify left))) (property "Sheetfile" "interfaces_aux/wbo2_analog.kicad_sch" (at 800.1 580.39 0) (effects (font (size 1.27 1.27)) (justify left))) (instances (project "Power8GDI_Core" (path "/f4d21065-0a5b-5086-a08e-1af9469f04bd" (page "55")))))
-(sheet (at 990.6 524.51) (size 154.94 54.61) (stroke (width 0.254) (type default)) (fill (color 0 0 0 0)) (property "Sheetname" "wbo adc control" (at 990.6 523.24 0) (effects (font (size 1.27 1.27)) (justify left))) (property "Sheetfile" "interfaces_aux/wbo_adc_control.kicad_sch" (at 990.6 580.39 0) (effects (font (size 1.27 1.27)) (justify left))) (instances (project "Power8GDI_Core" (path "/f4d21065-0a5b-5086-a08e-1af9469f04bd" (page "56")))))
+(sheet (at 229.87 524.51) (size 154.94 54.61) (stroke (width 0.254) (type default)) (fill (color 0 0 0 0)) (property "Sheetname" "knock dual" (at 229.87 523.24 0) (effects (font (size 1.27 1.27)) (justify left))) (property "Sheetfile" "interfaces_aux/knock_dual.kicad_sch" (at 229.87 580.39 0) (effects (font (size 1.27 1.27)) (justify left))) (instances (project "Power8GDI_Core" (path "/f4d21065-0a5b-5086-a08e-1af9469f04bd" (page "52")))))
+(sheet (at 420.37 524.51) (size 154.94 54.61) (stroke (width 0.254) (type default)) (fill (color 0 0 0 0)) (property "Sheetname" "gdi/protection a" (at 420.37 523.24 0) (effects (font (size 1.27 1.27)) (justify left))) (property "Sheetfile" "gdi/protection_a.kicad_sch" (at 420.37 580.39 0) (effects (font (size 1.27 1.27)) (justify left))) (instances (project "Power8GDI_Core" (path "/f4d21065-0a5b-5086-a08e-1af9469f04bd" (page "53")))))
+(sheet (at 609.6 524.51) (size 154.94 54.61) (stroke (width 0.254) (type default)) (fill (color 0 0 0 0)) (property "Sheetname" "gdi/protection b" (at 609.6 523.24 0) (effects (font (size 1.27 1.27)) (justify left))) (property "Sheetfile" "gdi/protection_b.kicad_sch" (at 609.6 580.39 0) (effects (font (size 1.27 1.27)) (justify left))) (instances (project "Power8GDI_Core" (path "/f4d21065-0a5b-5086-a08e-1af9469f04bd" (page "54")))))
+(sheet (at 800.1 524.51) (size 154.94 54.61) (stroke (width 0.254) (type default)) (fill (color 0 0 0 0)) (property "Sheetname" "gdi/permission" (at 800.1 523.24 0) (effects (font (size 1.27 1.27)) (justify left))) (property "Sheetfile" "gdi/permission.kicad_sch" (at 800.1 580.39 0) (effects (font (size 1.27 1.27)) (justify left))) (instances (project "Power8GDI_Core" (path "/f4d21065-0a5b-5086-a08e-1af9469f04bd" (page "55")))))
+(sheet (at 990.6 524.51) (size 154.94 54.61) (stroke (width 0.254) (type default)) (fill (color 0 0 0 0)) (property "Sheetname" "wbo/wbo1 analog" (at 990.6 523.24 0) (effects (font (size 1.27 1.27)) (justify left))) (property "Sheetfile" "wbo/wbo1_analog.kicad_sch" (at 990.6 580.39 0) (effects (font (size 1.27 1.27)) (justify left))) (instances (project "Power8GDI_Core" (path "/f4d21065-0a5b-5086-a08e-1af9469f04bd" (page "56")))))
+(sheet (at 39.37 614.68) (size 154.94 54.61) (stroke (width 0.254) (type default)) (fill (color 0 0 0 0)) (property "Sheetname" "wbo/wbo1 control" (at 39.37 613.41 0) (effects (font (size 1.27 1.27)) (justify left))) (property "Sheetfile" "wbo/wbo1_control.kicad_sch" (at 39.37 670.56 0) (effects (font (size 1.27 1.27)) (justify left))) (instances (project "Power8GDI_Core" (path "/f4d21065-0a5b-5086-a08e-1af9469f04bd" (page "57")))))
+(sheet (at 229.87 614.68) (size 154.94 54.61) (stroke (width 0.254) (type default)) (fill (color 0 0 0 0)) (property "Sheetname" "wbo/wbo1 heater feed" (at 229.87 613.41 0) (effects (font (size 1.27 1.27)) (justify left))) (property "Sheetfile" "wbo/wbo1_heater_feed.kicad_sch" (at 229.87 670.56 0) (effects (font (size 1.27 1.27)) (justify left))) (instances (project "Power8GDI_Core" (path "/f4d21065-0a5b-5086-a08e-1af9469f04bd" (page "58")))))
+(sheet (at 420.37 614.68) (size 154.94 54.61) (stroke (width 0.254) (type default)) (fill (color 0 0 0 0)) (property "Sheetname" "wbo/wbo2 analog" (at 420.37 613.41 0) (effects (font (size 1.27 1.27)) (justify left))) (property "Sheetfile" "wbo/wbo2_analog.kicad_sch" (at 420.37 670.56 0) (effects (font (size 1.27 1.27)) (justify left))) (instances (project "Power8GDI_Core" (path "/f4d21065-0a5b-5086-a08e-1af9469f04bd" (page "59")))))
+(sheet (at 609.6 614.68) (size 154.94 54.61) (stroke (width 0.254) (type default)) (fill (color 0 0 0 0)) (property "Sheetname" "wbo/wbo2 control" (at 609.6 613.41 0) (effects (font (size 1.27 1.27)) (justify left))) (property "Sheetfile" "wbo/wbo2_control.kicad_sch" (at 609.6 670.56 0) (effects (font (size 1.27 1.27)) (justify left))) (instances (project "Power8GDI_Core" (path "/f4d21065-0a5b-5086-a08e-1af9469f04bd" (page "60")))))
+(sheet (at 800.1 614.68) (size 154.94 54.61) (stroke (width 0.254) (type default)) (fill (color 0 0 0 0)) (property "Sheetname" "wbo/wbo2 heater feed" (at 800.1 613.41 0) (effects (font (size 1.27 1.27)) (justify left))) (property "Sheetfile" "wbo/wbo2_heater_feed.kicad_sch" (at 800.1 670.56 0) (effects (font (size 1.27 1.27)) (justify left))) (instances (project "Power8GDI_Core" (path "/f4d21065-0a5b-5086-a08e-1af9469f04bd" (page "61")))))
 (text "Each sheet uses explicit global net names. HARNESS names remain separate from MCU logic.\nNo ERC exclusions or power flags conceal missing supplies. DNP assembly flags must be preserved.\nGDI enable, injector/pump models, missing domains and full routing remain release blockers." (at 25.4 745 0) (effects (font (size 1.27 1.27)) (justify left top)))
 (sheet_instances (path "/" (page "1"))))

Commit message: Connect eight passive-coil stages to global fault latch and validate revised hierarchy
Other:
- removed sheet Eight smart-coil logic candidates
- added sheet Ignition 1 - timed primary and OC latch (ignition/ignition_1.kicad_sch)
- added sheet Ignition 2 - timed primary and OC latch (ignition/ignition_2.kicad_sch)
- added sheet Ignition 3 - timed primary and OC latch (ignition/ignition_3.kicad_sch)
- added sheet Ignition 4 - timed primary and OC latch (ignition/ignition_4.kicad_sch)
- added sheet Ignition 5 - timed primary and OC latch (ignition/ignition_5.kicad_sch)
- added sheet Ignition 6 - timed primary and OC latch (ignition/ignition_6.kicad_sch)
- added sheet Ignition 7 - timed primary and OC latch (ignition/ignition_7.kicad_sch)
- added sheet Ignition 8 - timed primary and OC latch (ignition/ignition_8.kicad_sch)
- added sheet Ignition permission and four dual gate drivers (ignition/ignition_common.kicad_sch)

Commit message: Integrate sequenced logic supply and four protected motor bridges
Other:
- removed sheet 3V3 logic post-regulator
- removed sheet DBW H-bridge candidate
- removed sheet EWG H-bridge candidate
- removed sheet Protected logic battery input
- added sheet logic power/logic 3v3 (logic_power/logic_3v3.kicad_sch)
- added sheet logic power/logic 5v (logic_power/logic_5v.kicad_sch)
- added sheet motor4/dbw (motor4/dbw.kicad_sch)
- added sheet motor4/ewg (motor4/ewg.kicad_sch)
- added sheet motor4/motor13 power (motor4/motor13_power.kicad_sch)
- added sheet motor4/motor24 power (motor4/motor24_power.kicad_sch)
- added sheet motor4/motor3 (motor4/motor3.kicad_sch)
- added sheet motor4/motor4 (motor4/motor4.kicad_sch)
- added sheet motor4/spi (motor4/spi.kicad_sch)
