File: Power8GDI/hardware/design/Power8GDI_Core.kicad_sch (KiCad schematic)
At the start: 0 parts

Commit message: Redesign sport target as six DI/PI channels with two motors and one lambda
Other:
- sheet Direct protected low-side AUX_PWM1, AUX_PWM2, AUX_PWM3, AUX_PWM4 renamed Direct protected low-side AUX_PWM3, AUX_PWM4, AUX_PWM5, AUX_PWM6
- sheet Direct protected low-side AUX_PWM5, AUX_PWM6, AUX_PWM7, AUX_PWM8 renamed Direct protected low-side AUX_PWM7, AUX_PWM8, LS_AUX1, LS_AUX2
- sheet Direct protected low-side LS_AUX1, LS_AUX2, LS_AUX3, LS_AUX4 renamed Direct protected low-side LS_AUX3, LS_AUX4
- sheet Direct protected low-side PI5, PI6, PI7, PI8 renamed Direct protected low-side PI5, PI6, VVT1, VVT2
- sheet Direct protected low-side VVT1, VVT2, VVT3, VVT4 renamed Direct protected low-side VVT3, VVT4, AUX_PWM1, AUX_PWM2
- sheet Ignition permission and four dual gate drivers renamed Ignition permission and three dual gate drivers
- removed sheet Ignition 7 - timed primary and OC latch
- removed sheet Ignition 8 - timed primary and OC latch
- removed sheet motor4/motor3
- removed sheet motor4/motor4
- removed sheet wbo/wbo2 analog
- removed sheet wbo/wbo2 control
- removed sheet wbo/wbo2 heater feed
- added sheet Documented power sources across passive paths (power_sources.kicad_sch)
- note added: "Each sheet uses explicit global net names. HARNESS names remain separate from MCU logic. No ERC exclusions. Power flags have explicit independently checked source paths. DNP assembly flags must be preserved. GDI enable, injector/pump models, missing domains and full routing remain release blockers."
- note added: "Power6GDI electrical candidate / NOT RELEASED Connected hierarchy: MCU, input supply, two GDI stages, safety, motor candidates, sensor frontends and harness. Outstanding channels and load qualification are tracked in INTEGRATION_2026_10_21_ELECTRICAL.md."
- note removed: "Each sheet uses explicit global net names. HARNESS names remain separate from MCU logic. No ERC exclusions or power flags conceal missing supplies. DNP assembly flags must be preserved. GDI enable, injector/pump models, missing domains and full routing remain release blockers."
- note removed: "Power8GDI electrical candidate / NOT RELEASED Connected hierarchy: MCU, input supply, two GDI stages, safety, motor candidates, sensor frontends and harness. Outstanding channels and load qualification are tracked in INTEGRATION_2026_10_21_ELECTRICAL.md."
