File: Power8GDI/hardware/design/core_mcu.kicad_sch (KiCad schematic)
At the start: 31 parts, among them J101 SWD 3V3 target reference, U101 STM32F767IIT6, Y101 ASEM1-8.000MHZ-LC-T

Commit message: Checkpoint integrated 37-sheet schematic before Huge scope revision
Connections:
- net KNOCK_INT_HOLD: now reaches U101.11 (PI9)
- net SD_CS: now reaches U101.119 (PA8)
- net WBO1_CS_N: now reaches U101.12 (PI10)
- net USB_VBUS_PRESENT_N: now reaches U101.120 (PA9)
- net WBO1_HEATER_PWM: now reaches U101.121 (PA10)
- net USB_DM: now reaches U101.122 (PA11)
- net USB_DP: now reaches U101.123 (PA12)
- net HALL1: now reaches U101.129 (PH14)
- net DIN8: now reaches U101.13 (PI11)
- net HALL2: now reaches U101.130 (PH15)
- net HALL3: now reaches U101.131 (PI0)
- net KNOCK_CS_N: now reaches U101.132 (PI1)
- net DIN5: now reaches U101.133 (PI2)
- net DIN6: now reaches U101.134 (PI3)
- net SD_SPI3_SCK: now reaches U101.139 (PC10)
- net SD_SPI3_MISO: now reaches U101.140 (PC11)
- net SD_SPI3_MOSI: now reaches U101.141 (PC12)
- net SD_CD: now reaches U101.154 (PG11)
- net CAN2_STB: now reaches U101.155 (PG12)
- net LIN2_EN: now reaches U101.156 (PG13)
- net WBO_ADC_CS_N: now reaches U101.162 (PB4)
- net CAN2_RX: now reaches U101.163 (PB5)
- net CAN2_TX: now reaches U101.164 (PB6)
- net DIN7: now reaches U101.173 (PI4)
- net HALL4: now reaches U101.176 (PI7)
- net WBO2_HEATER_PWM: now reaches U101.58 (PB2)
- net FLEX_FREQ: now reaches U101.7 (PI8)
- net LIN2_TX: now reaches U101.79 (PB10)
- net LIN2_RX: now reaches U101.80 (PB11)
- net WBO2_CS_N: now reaches U101.96 (PD8)
- net KNOCK1: no longer names the net of U101.25 (PF7)
- net KNOCK2: no longer names the net of U101.21 (PF5)
- no-connect marks 35 -> 7
Other:
- note added: "176 physical pads; source: DS11532 Rev9 + official KiCad9.0.9 symbol. GPIO labels are logic-side draft functions, NEVER harness/actuator connections. USB FS and SPI3 microSD use dedicated interface sheets. PH1, PC14/15 reserved unused; HSE bypass input only."
- note removed: "176 physical pads; source: DS11532 Rev9 + official KiCad9.0.9 symbol. GPIO labels are logic-side draft functions, NEVER harness/actuator connections. No USB or SD route is fitted. PH1, PC14/15 reserved unused; HSE bypass input only."

Commit message: Integrate protected GDI and CAN wideband nodes with Huge channel allocation
Connections:
- net DIN5 is gone; now on net DBW_DIR: U101.133 (PI2)
- net WBO2_CS_N is gone; now on net HPFP1: U101.96 (PD8)
- net DBW_DIR: no longer U101.116 (PC7)
- net HPFP1: no longer U101.118 (PC9)
- net DIN6 renamed MOTOR3_DIR
- net DIN7 renamed MOTOR4_DIR
- net DIN8 renamed MOTOR4_DISABLE
- net WBO1_CS_N renamed MOTOR3_DISABLE
- net WBO_ADC_CS_N renamed MOTOR_CS_N
- new net MOTOR3_PWM: U101.116 (PC7)
- new net MOTOR4_PWM: U101.118 (PC9)
Changed lines of the file:
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@@
 (global_label "KNOCK_CS_N" (shape bidirectional) (at 104.14 93.98 0) (effects (font (size 1.016 1.016)) (justify right bottom)))
 (wire (pts (xy 111.76 96.52) (xy 104.14 96.52)) (stroke (width 0) (type default)))
-(global_label "DIN5" (shape bidirectional) (at 104.14 96.52 0) (effects (font (size 1.016 1.016)) (justify right bottom)))
+(global_label "DBW_DIR" (shape bidirectional) (at 104.14 96.52 0) (effects (font (size 1.016 1.016)) (justify right bottom)))
 (wire (pts (xy 111.76 99.06) (xy 104.14 99.06)) (stroke (width 0) (type default)))
-(global_label "DIN6" (shape bidirectional) (at 104.14 99.06 0) (effects (font (size 1.016 1.016)) (justify right bottom)))
+(global_label "MOTOR3_DIR" (shape bidirectional) (at 104.14 99.06 0) (effects (font (size 1.016 1.016)) (justify right bottom)))
 (wire (pts (xy 111.76 101.6) (xy 104.14 101.6)) (stroke (width 0) (type default)))
-(global_label "DIN7" (shape bidirectional) (at 104.14 101.6 0) (effects (font (size 1.016 1.016)) (justify right bottom)))
+(global_label "MOTOR4_DIR" (shape bidirectional) (at 104.14 101.6 0) (effects (font (size 1.016 1.016)) (justify right bottom)))
 (wire (pts (xy 111.76 104.14) (xy 104.14 104.14)) (stroke (width 0) (type default)))
 (global_label "CAM3" (shape bidirectional) (at 104.14 104.14 0) (effects (font (size 1.016 1.016)) (justify right bottom)))
@@
 (global_label "KNOCK_INT_HOLD" (shape bidirectional) (at 104.14 114.3 0) (effects (font (size 1.016 1.016)) (justify right bottom)))
 (wire (pts (xy 111.76 116.84) (xy 104.14 116.84)) (stroke (width 0) (type default)))
-(global_label "WBO1_CS_N" (shape bidirectional) (at 104.14 116.84 0) (effects (font (size 1.016 1.016)) (justify right bottom)))
+(global_label "MOTOR3_DISABLE" (shape bidirectional) (at 104.14 116.84 0) (effects (font (size 1.016 1.016)) (justify right bottom)))
 (wire (pts (xy 111.76 119.38) (xy 104.14 119.38)) (stroke (width 0) (type default)))
-(global_label "DIN8" (shape bidirectional) (at 104.14 119.38 0) (effects (font (size 1.016 1.016)) (justify right bottom)))
+(global_label "MOTOR4_DISABLE" (shape bidirectional) (at 104.14 119.38 0) (effects (font (size 1.016 1.016)) (justify right bottom)))
 (wire (pts (xy 111.76 124.46) (xy 104.14 124.46)) (stroke (width 0) (type default)))
 (global_label "MCU_HSE_IN" (shape bidirectional) (at 104.14 124.46 0) (effects (font (size 1.016 1.016)) (justify right bottom)))
@@
 (global_label "SWO" (shape bidirectional) (at 200.66 121.92 180) (effects (font (size 1.016 1.016)) (justify left bottom)))
 (wire (pts (xy 193.04 124.46) (xy 200.66 124.46)) (stroke (width 0) (type default)))
-(global_label "WBO_ADC_CS_N" (shape bidirectional) (at 200.66 124.46 180) (effects (font (size 1.016 1.016)) (justify left bottom)))
+(global_label "MOTOR_CS_N" (shape bidirectional) (at 200.66 124.46 180) (effects (font (size 1.016 1.016)) (justify left bottom)))
 (wire (pts (xy 193.04 127) (xy 200.66 127)) (stroke (width 0) (type default)))
 (global_label "CAN2_RX" (shape bidirectional) (at 200.66 127 180) (effects (font (size 1.016 1.016)) (justify left bottom)))
@@
 (global_label "DBW_PWM" (shape bidirectional) (at 200.66 172.72 180) (effects (font (size 1.016 1.016)) (justify left bottom)))
 (wire (pts (xy 193.04 175.26) (xy 200.66 175.26)) (stroke (width 0) (type default)))
-(global_label "DBW_DIR" (shape bidirectional) (at 200.66 175.26 180) (effects (font (size 1.016 1.016)) (justify left bottom)))
+(global_label "MOTOR3_PWM" (shape bidirectional) (at 200.66 175.26 180) (effects (font (size 1.016 1.016)) (justify left bottom)))
 (wire (pts (xy 193.04 177.8) (xy 200.66 177.8)) (stroke (width 0) (type default)))
 (global_label "EWG_PWM" (shape bidirectional) (at 200.66 177.8 180) (effects (font (size 1.016 1.016)) (justify left bottom)))
 (wire (pts (xy 193.04 180.34) (xy 200.66 180.34)) (stroke (width 0) (type default)))
-(global_label "HPFP1" (shape bidirectional) (at 200.66 180.34 180) (effects (font (size 1.016 1.016)) (justify left bottom)))
+(global_label "MOTOR4_PWM" (shape bidirectional) (at 200.66 180.34 180) (effects (font (size 1.016 1.016)) (justify left bottom)))
 (wire (pts (xy 193.04 182.88) (xy 200.66 182.88)) (stroke (width 0) (type default)))
 (global_label "SD_SPI3_SCK" (shape bidirectional) (at 200.66 182.88 180) (effects (font (size 1.016 1.016)) (justify left bottom)))
@@
 (global_label "LS_AUX4" (shape bidirectional) (at 200.66 218.44 180) (effects (font (size 1.016 1.016)) (justify left bottom)))
 (wire (pts (xy 193.04 220.98) (xy 200.66 220.98)) (stroke (width 0) (type default)))
-(global_label "WBO2_CS_N" (shape bidirectional) (at 200.66 220.98 180) (effects (font (size 1.016 1.016)) (justify left bottom)))
+(global_label "HPFP1" (shape bidirectional) (at 200.66 220.98 180) (effects (font (size 1.016 1.016)) (justify left bottom)))
 (wire (pts (xy 193.04 223.52) (xy 200.66 223.52)) (stroke (width 0) (type default)))
 (global_label "DI5" (shape bidirectional) (at 200.66 223.52 180) (effects (font (size 1.016 1.016)) (justify left bottom)))

Commit message: Redesign sport target as six DI/PI channels with two motors and one lambda
Connections:
- net DI7 is gone; now on net DI6: U101.63 (PF13)
- net DI4: now also U101.97 (PD9); no longer U101.98 (PD10)
- net DI5: now also U101.60 (PF12); no longer U101.97 (PD9)
- net DI6: no longer U101.60 (PF12)
- net DI8: no longer names the net of U101.64 (PF14)
- net IGN7: no longer names the net of U101.168 (PB9)
- net IGN8: no longer names the net of U101.5 (PE6)
- net MOTOR3_DIR: no longer names the net of U101.134 (PI3)
- net MOTOR3_DISABLE: no longer names the net of U101.12 (PI10)
- net MOTOR3_PWM: no longer names the net of U101.116 (PC7)
- net MOTOR4_DIR: no longer names the net of U101.173 (PI4)
- net MOTOR4_DISABLE: no longer names the net of U101.13 (PI11)
- net MOTOR4_PWM: no longer names the net of U101.118 (PC9)
- net PI7: no longer names the net of U101.17 (PF1)
- net PI8: no longer names the net of U101.18 (PF2)
- net WBO2_HEATER_PWM: no longer names the net of U101.58 (PB2)
- no-connect marks 7 -> 20
Changed lines of the file:
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@@
 (wire (pts (xy 111.76 96.52) (xy 104.14 96.52)) (stroke (width 0) (type default)))
 (global_label "DBW_DIR" (shape bidirectional) (at 104.14 96.52 0) (effects (font (size 1.016 1.016)) (justify right bottom)))
-(wire (pts (xy 111.76 99.06) (xy 104.14 99.06)) (stroke (width 0) (type default)))
-(global_label "MOTOR3_DIR" (shape bidirectional) (at 104.14 99.06 0) (effects (font (size 1.016 1.016)) (justify right bottom)))
-(wire (pts (xy 111.76 101.6) (xy 104.14 101.6)) (stroke (width 0) (type default)))
-(global_label "MOTOR4_DIR" (shape bidirectional) (at 104.14 101.6 0) (effects (font (size 1.016 1.016)) (justify right bottom)))
+(no_connect (at 111.76 99.06))
+(no_connect (at 111.76 101.6))
 (wire (pts (xy 111.76 104.14) (xy 104.14 104.14)) (stroke (width 0) (type default)))
 (global_label "CAM3" (shape bidirectional) (at 104.14 104.14 0) (effects (font (size 1.016 1.016)) (justify right bottom)))
@@
 (wire (pts (xy 111.76 114.3) (xy 104.14 114.3)) (stroke (width 0) (type default)))
 (global_label "KNOCK_INT_HOLD" (shape bidirectional) (at 104.14 114.3 0) (effects (font (size 1.016 1.016)) (justify right bottom)))
-(wire (pts (xy 111.76 116.84) (xy 104.14 116.84)) (stroke (width 0) (type default)))
-(global_label "MOTOR3_DISABLE" (shape bidirectional) (at 104.14 116.84 0) (effects (font (size 1.016 1.016)) (justify right bottom)))
-(wire (pts (xy 111.76 119.38) (xy 104.14 119.38)) (stroke (width 0) (type default)))
-(global_label "MOTOR4_DISABLE" (shape bidirectional) (at 104.14 119.38 0) (effects (font (size 1.016 1.016)) (justify right bottom)))
+(no_connect (at 111.76 116.84))
+(no_connect (at 111.76 119.38))
 (wire (pts (xy 111.76 124.46) (xy 104.14 124.46)) (stroke (width 0) (type default)))
 (global_label "MCU_HSE_IN" (shape bidirectional) (at 104.14 124.46 0) (effects (font (size 1.016 1.016)) (justify right bottom)))
@@
 (wire (pts (xy 111.76 210.82) (xy 104.14 210.82)) (stroke (width 0) (type default)))
 (global_label "PI6" (shape bidirectional) (at 104.14 210.82 0) (effects (font (size 1.016 1.016)) (justify right bottom)))
-(wire (pts (xy 111.76 213.36) (xy 104.14 213.36)) (stroke (width 0) (type default)))
-(global_label "PI7" (shape bidirectional) (at 104.14 213.36 0) (effects (font (size 1.016 1.016)) (justify right bottom)))
-(wire (pts (xy 111.76 215.9) (xy 104.14 215.9)) (stroke (width 0) (type default)))
-(global_label "PI8" (shape bidirectional) (at 104.14 215.9 0) (effects (font (size 1.016 1.016)) (justify right bottom)))
+(no_connect (at 111.76 213.36))
+(no_connect (at 111.76 215.9))
 (wire (pts (xy 111.76 218.44) (xy 104.14 218.44)) (stroke (width 0) (type default)))
 (global_label "CAM1" (shape bidirectional) (at 104.14 218.44 0) (effects (font (size 1.016 1.016)) (justify right bottom)))
@@
 (global_label "VVT2" (shape bidirectional) (at 104.14 238.76 0) (effects (font (size 1.016 1.016)) (justify right bottom)))
 (wire (pts (xy 111.76 241.3) (xy 104.14 241.3)) (stroke (width 0) (type default)))
-(global_label "DI6" (shape bidirectional) (at 104.14 241.3 0) (effects (font (size 1.016 1.016)) (justify right bottom)))
+(global_label "DI5" (shape bidirectional) (at 104.14 241.3 0) (effects (font (size 1.016 1.016)) (justify right bottom)))
 (wire (pts (xy 111.76 243.84) (xy 104.14 243.84)) (stroke (width 0) (type default)))
-(global_label "DI7" (shape bidirectional) (at 104.14 243.84 0) (effects (font (size 1.016 1.016)) (justify right bottom)))
-(wire (pts (xy 111.76 246.38) (xy 104.14 246.38)) (stroke (width 0) (type default)))
-(global_label "DI8" (shape bidirectional) (at 104.14 246.38 0) (effects (font (size 1.016 1.016)) (justify right bottom)))
+(global_label "DI6" (shape bidirectional) (at 104.14 243.84 0) (effects (font (size 1.016 1.016)) (justify right bottom)))
+(no_connect (at 111.76 246.38))
 (wire (pts (xy 111.76 248.92) (xy 104.14 248.92)) (stroke (width 0) (type default)))
 (global_label "VVT3" (shape bidirectional) (at 104.14 248.92 0) (effects (font (size 1.016 1.016)) (justify right bottom)))
@@
 (wire (pts (xy 193.04 116.84) (xy 200.66 116.84)) (stroke (width 0) (type default)))
 (global_label "CRANK" (shape bidirectional) (at 200.66 116.84 180) (effects (font (size 1.016 1.016)) (justify left bottom)))
-(wire (pts (xy 193.04 119.38) (xy 200.66 119.38)) (stroke (width 0) (type default)))
-(global_label "WBO2_HEATER_PWM" (shape bidirectional) (at 200.66 119.38 180) (effects (font (size 1.016 1.016)) (justify left bottom)))
+(no_connect (at 193.04 119.38))
 (wire (pts (xy 193.04 121.92) (xy 200.66 121.92)) (stroke (width 0) (type default)))
 (global_label "SWO" (shape bidirectional) (at 200.66 121.92 180) (effects (font (size 1.016 1.016)) (justify left bottom)))
@@
 (wire (pts (xy 193.04 134.62) (xy 200.66 134.62)) (stroke (width 0) (type default)))
 (global_label "IGN6" (shape bidirectional) (at 200.66 134.62 180) (effects (font (size 1.016 1.016)) (justify left bottom)))
-(wire (pts (xy 193.04 137.16) (xy 200.66 137.16)) (stroke (width 0) (type default)))
-(global_label "IGN7" (shape bidirectional) (at 200.66 137.16 180) (effects (font (size 1.016 1.016)) (justify left bottom)))
+(no_connect (at 193.04 137.16))
 (wire (pts (xy 193.04 139.7) (xy 200.66 139.7)) (stroke (width 0) (type default)))
 (global_label "LIN2_TX" (shape bidirectional) (at 200.66 139.7 180) (effects (font (size 1.016 1.016)) (justify left bottom)))
@@
 (wire (pts (xy 193.04 172.72) (xy 200.66 172.72)) (stroke (width 0) (type default)))
 (global_label "DBW_PWM" (shape bidirectional) (at 200.66 172.72 180) (effects (font (size 1.016 1.016)) (justify left bottom)))
-(wire (pts (xy 193.04 175.26) (xy 200.66 175.26)) (stroke (width 0) (type default)))
-(global_label "MOTOR3_PWM" (shape bidirectional) (at 200.66 175.26 180) (effects (font (size 1.016 1.016)) (justify left bottom)))
+(no_connect (at 193.04 175.26))
 (wire (pts (xy 193.04 177.8) (xy 200.66 177.8)) (stroke (width 0) (type default)))
 (global_label "EWG_PWM" (shape bidirectional) (at 200.66 177.8 180) (effects (font (size 1.016 1.016)) (justify left bottom)))
-(wire (pts (xy 193.04 180.34) (xy 200.66 180.34)) (stroke (width 0) (type default)))
-(global_label "MOTOR4_PWM" (shape bidirectional) (at 200.66 180.34 180) (effects (font (size 1.016 1.016)) (justify left bottom)))
+(no_connect (at 193.04 180.34))
 (wire (pts (xy 193.04 182.88) (xy 200.66 182.88)) (stroke (width 0) (type default)))
 (global_label "SD_SPI3_SCK" (shape bidirectional) (at 200.66 182.88 180) (effects (font (size 1.016 1.016)) (justify left bottom)))
@@
 (global_label "HPFP1" (shape bidirectional) (at 200.66 220.98 180) (effects (font (size 1.016 1.016)) (justify left bottom)))
 (wire (pts (xy 193.04 223.52) (xy 200.66 223.52)) (stroke (width 0) (type default)))
-(global_label "DI5" (shape bidirectional) (at 200.66 223.52 180) (effects (font (size 1.016 1.016)) (justify left bottom)))
-(wire (pts (xy 193.04 226.06) (xy 200.66 226.06)) (stroke (width 0) (type default)))
-(global_label "DI4" (shape bidirectional) (at 200.66 226.06 180) (effects (font (size 1.016 1.016)) (justify left bottom)))
+(global_label "DI4" (shape bidirectional) (at 200.66 223.52 180) (effects (font (size 1.016 1.016)) (justify left bottom)))
+(no_connect (at 193.04 226.06))
 (wire (pts (xy 193.04 228.6) (xy 200.66 228.6)) (stroke (width 0) (type default)))
 (global_label "DI3" (shape bidirectional) (at 200.66 228.6 180) (effects (font (size 1.016 1.016)) (justify left bottom)))
@@
 (wire (pts (xy 193.04 256.54) (xy 200.66 256.54)) (stroke (width 0) (type default)))
 (global_label "IGN2" (shape bidirectional) (at 200.66 256.54 180) (effects (font (size 1.016 1.016)) (justify left bottom)))
-(wire (pts (xy 193.04 259.08) (xy 200.66 259.08)) (stroke (width 0) (type default)))
-(global_label "IGN8" (shape bidirectional) (at 200.66 259.08 180) (effects (font (size 1.016 1.016)) (justify left bottom)))
+(no_connect (at 193.04 259.08))
 (wire (pts (xy 193.04 261.62) (xy 200.66 261.62)) (stroke (width 0) (type default)))
 (global_label "PI3" (shape bidirectional) (at 200.66 261.62 180) (effects (font (size 1.016 1.016)) (justify left bottom)))
