File: Power8GDI/hardware/design/board/layout_candidate/Power8GDI_Review.kicad_pcb (KiCad board)
At the start: 4 copper layers, 245 x 165 mm, 1236 parts, among them J101 SWD 3V3 target reference, J1501 Molex 1050170001, J1502 Molex 1040310811, J5600 Conn_02x03_Odd_Even, J5800 Conn_02x03_Odd_Even, J601 6437288-1 / KEY1 CANDIDATE, J602 6437288-1 / KEY1 CANDIDATE, J603 6437288-1 / KEY1 CANDIDATE, J604 6437288-1 / KEY1 CANDIDATE, Q1510 2N7002,215, Q201 BUK9230-100B, Q202 BUK9230-100B, Q203 BUK9230-100B, Q204 BUK9230-100B, Q205 BUK9230-100B, Q206 BUK9230-100B, Q207 BUK9230-100B, Q208 BUK9230-100B, Q209 BUK9230-100B, Q210 BUK9230-100B, Q211 BUK9230-100B, Q212 BUK9230-100B, Q213 BUK9230-100B, Q301 BUK9230-100B, Q302 BUK9230-100B, Q303 BUK9230-100B, Q304 BUK9230-100B, Q305 BUK9230-100B, Q306 BUK9230-100B, Q307 BUK9230-100B, Q308 BUK9230-100B, Q309 BUK9230-100B, Q310 BUK9230-100B, Q311 BUK9230-100B, Q312 BUK9230-100B, Q313 BUK9230-100B, Q5001 IPD90N10S4-06, Q5002 IPD90N10S4-06, Q5051 IPD90N10S4-06, Q5052 IPD90N10S4-06, Q5420 STGB18N40LZT4, Q5440 STGB18N40LZT4, Q5460 STGB18N40LZT4, Q5480 STGB18N40LZT4, Q5500 STGB18N40LZT4, Q5520 STGB18N40LZT4, Q5540 STGB18N40LZT4, Q5560 STGB18N40LZT4, Q5600 VND7NV04TR-E, Q5800 VND7NV04TR-E, Q6200 IPD90N10S4-06, Q6201 IPD90N10S4-06, Q6250 IPD90N10S4-06, Q6251 IPD90N10S4-06, U101 STM32F767IIT6, U103 TCAN1042HGVDRQ1, U104 TLIN1029ADRQ1, U1101 TLE9104SHXUMA1, U1102 TLE9104SHXUMA1, U1103 TLE9104SHXUMA1, U1104 TLE9104SHXUMA1, U1105 TLE9104SHXUMA1, U1106 TLE9104SHXUMA1, U1121 SN74LVC14AQPWRQ1, U1122 SN74LVC14AQPWRQ1, U1123 SN74LVC14AQPWRQ1, U1124 SN74LVC14AQPWRQ1, U1125 SN74LVC14AQPWRQ1, U1126 SN74LVC14AQPWRQ1, U1140 SN74LVC1G17QDBVRQ1, U1501 TCAN1042HGVDRQ1, U1502 TLIN1029ADRQ1, U1530 TPS7B4253QDDARQ1, U1531 TPS7B4253QDDARQ1, U1600 SN74LVC14AQPWRQ1, U1701 TPIC8101DWR, U1702 SN74AHCT244QPWRQ1, U1703 CLVC1G125QDBVRQ1, U201 MC33PT2001AE, U249 NCV78M05ABDTRKG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

Commit message: Checkpoint actual 1262-part PCB with capped DRC and matching rule provenance
Parts:
- added C5660: 100n 16V X7R, Capacitor_SMD:C_0603_1608Metric, B.Cu at (172.8, 85.0)
- added C5661: 10u 16V X7R effective>=4.7u, Capacitor_SMD:C_1206_3216Metric, B.Cu at (174.1, 97.4)
- added C5662: 10u 16V X7R effective>=4.7u, Capacitor_SMD:C_1206_3216Metric, B.Cu at (163.9, 102.1)
- added C5663: 100n 16V X7R, Capacitor_SMD:C_0603_1608Metric, B.Cu at (163.8, 87.5)
- added C5664: 100n 16V X7R, Capacitor_SMD:C_0603_1608Metric, B.Cu at (154.5, 95.3)
- added C5860: 100n 16V X7R, Capacitor_SMD:C_0603_1608Metric, B.Cu at (231.8, 88.5)
- added C5861: 10u 16V X7R effective>=4.7u, Capacitor_SMD:C_1206_3216Metric, B.Cu at (218.6, 101.4)
- added C5862: 10u 16V X7R effective>=4.7u, Capacitor_SMD:C_1206_3216Metric, B.Cu at (214.4, 101.1)
- added C5863: 100n 16V X7R, Capacitor_SMD:C_0603_1608Metric, B.Cu at (228.3, 86.0)
- added C5864: 100n 16V X7R, Capacitor_SMD:C_0603_1608Metric, B.Cu at (232.3, 86.0)
- added Q5620: BC847B-QR, Package_TO_SOT_SMD:SOT-23, B.Cu at (155.0, 130.7)
- added Q5820: BC847B-QR, Package_TO_SOT_SMD:SOT-23, B.Cu at (209.5, 101.2)
- added R5660: 30k 0.1%, Resistor_SMD:R_0603_1608Metric, B.Cu at (169.3, 82.0)
- added R5661: 2.2k 1%, Resistor_SMD:R_0603_1608Metric, B.Cu at (173.8, 80.0)
- added R5662: 10k, Resistor_SMD:R_0603_1608Metric, B.Cu at (159.8, 81.5)
- added R5663: 220R 0.1%, Resistor_SMD:R_0603_1608Metric, B.Cu at (163.8, 80.0)
- added R5664: 4.7k 1%, Resistor_SMD:R_0603_1608Metric, B.Cu at (154.0, 83.3)
- added R5665: 10k 1%, Resistor_SMD:R_0603_1608Metric, B.Cu at (156.5, 81.8)
- added R5860: 30k 0.1%, Resistor_SMD:R_0603_1608Metric, B.Cu at (237.8, 79.5)
- added R5861: 2.2k 1%, Resistor_SMD:R_0603_1608Metric, B.Cu at (237.8, 77.0)
- added R5862: 10k, Resistor_SMD:R_0603_1608Metric, B.Cu at (207.5, 66.8)
- added R5863: 220R 0.1%, Resistor_SMD:R_0603_1608Metric, B.Cu at (239.8, 74.5)
- added R5864: 4.7k 1%, Resistor_SMD:R_0603_1608Metric, B.Cu at (210.8, 66.5)
- added R5865: 10k 1%, Resistor_SMD:R_0603_1608Metric, B.Cu at (204.3, 65.5)
- added U5612: TPS3808G33QDBVRQ1, Package_TO_SOT_SMD:SOT-23-6, B.Cu at (173.8, 121.0)
- added U5812: TPS3808G33QDBVRQ1, Package_TO_SOT_SMD:SOT-23-6, B.Cu at (209.8, 121.5)
- R5642, R5842: value 10k -> 2.2k 1%
- U5604, U5804: value XC6206P332MR-G -> LT3042IMSE#WTRPBF; footprint Package_TO_SOT_SMD:SOT-23 -> Package_SO:MSOP-10-1EP_3x3mm_P0.5mm_EP1.68x1.88mm
- moved R5052 204.2 mm to (209.0, 26.8)
- moved C5052 199.1 mm to (209.8, 20.0), turned to 90 degrees
- moved R5055 196.1 mm to (201.8, 31.0), turned to 0 degrees
- moved R5051 194.5 mm to (206.0, 26.2)
- moved C5051 193.3 mm to (207.5, 16.3)
- moved Q5052 191.8 mm to (200.2, 13.8), turned to 0 degrees
- moved U5051 188.9 mm to (206.0, 22.7)
- moved Q5051 187.8 mm to (199.8, 23.0)
- moved R5056 184.3 mm to (200.3, 8.50), turned to 0 degrees
- moved R5057 179.9 mm to (191.3, 13.0)
- moved R5053 178.8 mm to (205.8, 28.5)
- moved R5054 169.7 mm to (205.8, 31.0)
- moved C5055 145.1 mm to (190.0, 32.8), turned to 0 degrees
- moved R5058 144.3 mm to (193.8, 32.0), turned to 0 degrees
- moved C398 139.2 mm to (191.5, 18.8), turned to 0 degrees
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Connections:
- C5611 pad 1: WBO1_VDDA -> WBO1_3V3
- C5612 pad 1: WBO1_VDDA -> WBO1_3V3
- C5811 pad 1: WBO2_VDDA -> WBO2_3V3
- C5812 pad 1: WBO2_VDDA -> WBO2_3V3
- R5600 pad 1: WBO1_VDDA -> WBO1_3V3
- R5642 pad 1: HW_ACTUATOR_ENABLE_N -> WBO1_HEATER_OE_N
- R5642 pad 2: +3V3 -> +5V_CORE
- R5800 pad 1: WBO2_VDDA -> WBO2_3V3
- R5842 pad 1: HW_ACTUATOR_ENABLE_N -> WBO2_HEATER_OE_N
- R5842 pad 2: +3V3 -> +5V_CORE
- U5602 pad 5: WBO1_VDDA -> WBO1_3V3
- U5603 pad 2: WBO1_VDDA -> WBO1_REF3V3
- U5604 pad 1: GND -> +5V_CORE
- U5604 pad 2: WBO1_3V3 -> +5V_CORE
- U5611 pad 1: HW_ACTUATOR_ENABLE_N -> WBO1_HEATER_OE_N
- U5802 pad 5: WBO2_VDDA -> WBO2_3V3
- U5803 pad 2: WBO2_VDDA -> WBO2_REF3V3
- U5804 pad 1: GND -> +5V_CORE
- U5804 pad 2: WBO2_3V3 -> +5V_CORE
- U5811 pad 1: HW_ACTUATOR_ENABLE_N -> WBO2_HEATER_OE_N
