File: Power8GDI/hardware/design/board/connectors.kicad_sch (KiCad schematic)
At the start: 4 parts, among them J601 6437288-1 / KEY1 CANDIDATE, J602 6437288-1 / KEY1 CANDIDATE, J603 6437288-1 / KEY1 CANDIDATE, J604 6437288-1 / KEY1 CANDIDATE

Commit message: Checkpoint integrated 37-sheet schematic before Huge scope revision
Connections:
- net HARNESS_DI2_HIGH is gone; now on net PTA_H1: J601.3
- net HARNESS_DI4_HIGH is gone; now on net PTA_H3: J601.7
- net HARNESS_DI6_HIGH is gone; now on net PTB_H1: J601.11
- net HARNESS_DI8_HIGH is gone; now on net PTB_H3: J601.15
- net HARNESS_PGND_GDI_A_1 is gone; now on net GND: J601.25
- net HARNESS_PGND_GDI_A_2 is gone; now on net GND: J601.26
- net HARNESS_PGND_GDI_B_1 is gone; now on net GND: J601.27
- net HARNESS_PGND_GDI_B_2 is gone; now on net GND: J601.28
- net HARNESS_PGND_MAIN_4 is gone; now on net GND: J601.32
- net HARNESS_PGND_MAIN_B is gone; now on net GND: J602.34
- net HARNESS_CAN2_H renamed CAN2_H
- net HARNESS_CAN2_L renamed CAN2_L
- net HARNESS_CHASSIS_GND renamed USB_SHIELD
- net HARNESS_DI1_HIGH renamed PTA_H1
- net HARNESS_DI1_LOW renamed PTA_L1
- net HARNESS_DI2_LOW renamed PTA_L2
- net HARNESS_DI3_HIGH renamed PTA_H3
- net HARNESS_DI3_LOW renamed PTA_L3
- net HARNESS_DI4_LOW renamed PTA_L4
- net HARNESS_DI5_HIGH renamed PTB_H1
- net HARNESS_DI5_LOW renamed PTB_L1
- net HARNESS_DI6_LOW renamed PTB_L2
- net HARNESS_DI7_HIGH renamed PTB_H3
- net HARNESS_DI7_LOW renamed PTB_L3
- net HARNESS_DI8_LOW renamed PTB_L4
- net HARNESS_HPFP1_HIGH renamed PTA_H5PUMP
- net HARNESS_HPFP1_LOW renamed PTA_L6PUMP
- net HARNESS_HPFP2_HIGH renamed PTB_H5PUMP
- net HARNESS_HPFP2_LOW renamed PTB_L6PUMP
- net HARNESS_LIN2_BUS renamed LIN2_BUS
- net HARNESS_SENSOR_5V_A renamed SENSOR_5V_A
- net HARNESS_SENSOR_5V_B renamed SENSOR_5V_B

Commit message: Integrate protected GDI and CAN wideband nodes with Huge channel allocation
Connections:
- net HARNESS_VBAT_GDI_A_2 is gone; now on net VBAT_GDI_A_FUSED: J601.22
- net HARNESS_VBAT_GDI_B_2 is gone; now on net VBAT_GDI_B_FUSED: J601.24
- net HARNESS_DIN5 renamed MOTOR3_MOTOR_A
- net HARNESS_DIN6 renamed MOTOR3_MOTOR_B
- net HARNESS_DIN7 renamed MOTOR4_MOTOR_A
- net HARNESS_DIN8 renamed MOTOR4_MOTOR_B
- net HARNESS_VBAT_GDI_A_1 renamed VBAT_GDI_A_FUSED
- net HARNESS_VBAT_GDI_B_1 renamed VBAT_GDI_B_FUSED
Changed lines of the file:
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@@
 (global_label "PTB_L6PUMP" (shape bidirectional) (at 160.02 85.09 180) (effects (font (size 1.016 1.016)) (justify left bottom)))
 (wire (pts (xy 152.4 87.63) (xy 160.02 87.63)) (stroke (width 0) (type default)))
-(global_label "HARNESS_VBAT_GDI_A_1" (shape bidirectional) (at 160.02 87.63 180) (effects (font (size 1.016 1.016)) (justify left bottom)))
+(global_label "VBAT_GDI_A_FUSED" (shape bidirectional) (at 160.02 87.63 180) (effects (font (size 1.016 1.016)) (justify left bottom)))
 (wire (pts (xy 152.4 90.17) (xy 160.02 90.17)) (stroke (width 0) (type default)))
-(global_label "HARNESS_VBAT_GDI_A_2" (shape bidirectional) (at 160.02 90.17 180) (effects (font (size 1.016 1.016)) (justify left bottom)))
+(global_label "VBAT_GDI_A_FUSED" (shape bidirectional) (at 160.02 90.17 180) (effects (font (size 1.016 1.016)) (justify left bottom)))
 (wire (pts (xy 152.4 92.71) (xy 160.02 92.71)) (stroke (width 0) (type default)))
-(global_label "HARNESS_VBAT_GDI_B_1" (shape bidirectional) (at 160.02 92.71 180) (effects (font (size 1.016 1.016)) (justify left bottom)))
+(global_label "VBAT_GDI_B_FUSED" (shape bidirectional) (at 160.02 92.71 180) (effects (font (size 1.016 1.016)) (justify left bottom)))
 (wire (pts (xy 152.4 95.25) (xy 160.02 95.25)) (stroke (width 0) (type default)))
-(global_label "HARNESS_VBAT_GDI_B_2" (shape bidirectional) (at 160.02 95.25 180) (effects (font (size 1.016 1.016)) (justify left bottom)))
+(global_label "VBAT_GDI_B_FUSED" (shape bidirectional) (at 160.02 95.25 180) (effects (font (size 1.016 1.016)) (justify left bottom)))
 (wire (pts (xy 152.4 97.79) (xy 160.02 97.79)) (stroke (width 0) (type default)))
 (global_label "GND" (shape bidirectional) (at 160.02 97.79 180) (effects (font (size 1.016 1.016)) (justify left bottom)))
@@
 (global_label "CAN2_L" (shape bidirectional) (at 400.05 273.05 0) (effects (font (size 1.016 1.016)) (justify right bottom)))
 (wire (pts (xy 407.67 275.59) (xy 400.05 275.59)) (stroke (width 0) (type default)))
-(global_label "HARNESS_DIN5" (shape bidirectional) (at 400.05 275.59 0) (effects (font (size 1.016 1.016)) (justify right bottom)))
+(global_label "MOTOR3_MOTOR_A" (shape bidirectional) (at 400.05 275.59 0) (effects (font (size 1.016 1.016)) (justify right bottom)))
 (wire (pts (xy 407.67 278.13) (xy 400.05 278.13)) (stroke (width 0) (type default)))
-(global_label "HARNESS_DIN6" (shape bidirectional) (at 400.05 278.13 0) (effects (font (size 1.016 1.016)) (justify right bottom)))
+(global_label "MOTOR3_MOTOR_B" (shape bidirectional) (at 400.05 278.13 0) (effects (font (size 1.016 1.016)) (justify right bottom)))
 (wire (pts (xy 407.67 280.67) (xy 400.05 280.67)) (stroke (width 0) (type default)))
-(global_label "HARNESS_DIN7" (shape bidirectional) (at 400.05 280.67 0) (effects (font (size 1.016 1.016)) (justify right bottom)))
+(global_label "MOTOR4_MOTOR_A" (shape bidirectional) (at 400.05 280.67 0) (effects (font (size 1.016 1.016)) (justify right bottom)))
 (wire (pts (xy 433.07 240.03) (xy 440.69 240.03)) (stroke (width 0) (type default)))
-(global_label "HARNESS_DIN8" (shape bidirectional) (at 440.69 240.03 180) (effects (font (size 1.016 1.016)) (justify left bottom)))
+(global_label "MOTOR4_MOTOR_B" (shape bidirectional) (at 440.69 240.03 180) (effects (font (size 1.016 1.016)) (justify left bottom)))
 (wire (pts (xy 433.07 242.57) (xy 440.69 242.57)) (stroke (width 0) (type default)))
 (global_label "HARNESS_AUX_ANALOG1" (shape bidirectional) (at 440.69 242.57 180) (effects (font (size 1.016 1.016)) (justify left bottom)))

Commit message: Connect eight passive-coil stages to global fault latch and validate revised hierarchy
Connections:
- net IGN1_LOGIC_OUT renamed HARNESS_IGN1
- net IGN2_LOGIC_OUT renamed HARNESS_IGN2
- net IGN3_LOGIC_OUT renamed HARNESS_IGN3
- net IGN4_LOGIC_OUT renamed HARNESS_IGN4
- net IGN5_LOGIC_OUT renamed HARNESS_IGN5
- net IGN6_LOGIC_OUT renamed HARNESS_IGN6
- net IGN7_LOGIC_OUT renamed HARNESS_IGN7
- net IGN8_LOGIC_OUT renamed HARNESS_IGN8
Changed lines of the file:
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@@
 (symbol (lib_id "Power8GDI_Board:TE_6437288_1_34") (at 420.37 100.33 0) (unit 1) (in_bom yes) (on_board yes) (dnp no) (property "Reference" "J602" (at 420.37 77.47 0) (effects (font (size 1.27 1.27)))) (property "Value" "6437288-1 / KEY1 CANDIDATE" (at 420.37 123.19 0) (effects (font (size 1.27 1.27)))) (property "Footprint" "Power8GDI_Board:TE_6437288-1_34way" (at 420.37 100.33 0) (effects (font (size 1.27 1.27)) (hide yes))) (property "Design note" "TE header C-9-1437287-8 A1 sheet2; numbering from mating housing RevP sheet3. Mechanical/continuity/keying review pending. Unimplemented circuits remain isolated HARNESS nets." (at 420.37 100.33 0) (effects (font (size 1.27 1.27)) (hide yes))) (pin "1") (pin "2") (pin "3") (pin "4") (pin "5") (pin "6") (pin "7") (pin "8") (pin "9") (pin "10") (pin "11") (pin "12") (pin "13") (pin "14") (pin "15") (pin "16") (pin "17") (pin "18") (pin "19") (pin "20") (pin "21") (pin "22") (pin "23") (pin "24") (pin "25") (pin "26") (pin "27") (pin "28") (pin "29") (pin "30") (pin "31") (pin "32") (pin "33") (pin "34") (instances (project "Power8GDI_Core" (path "/f4d21065-0a5b-5086-a08e-1af9469f04bd/df0c5f3e-1ee1-56be-91e2-4072c6105289" (reference "J602") (unit 1)))))
 (wire (pts (xy 407.67 80.01) (xy 400.05 80.01)) (stroke (width 0) (type default)))
-(global_label "IGN1_LOGIC_OUT" (shape bidirectional) (at 400.05 80.01 0) (effects (font (size 1.016 1.016)) (justify right bottom)))
+(global_label "HARNESS_IGN1" (shape bidirectional) (at 400.05 80.01 0) (effects (font (size 1.016 1.016)) (justify right bottom)))
 (wire (pts (xy 407.67 82.55) (xy 400.05 82.55)) (stroke (width 0) (type default)))
-(global_label "IGN2_LOGIC_OUT" (shape bidirectional) (at 400.05 82.55 0) (effects (font (size 1.016 1.016)) (justify right bottom)))
+(global_label "HARNESS_IGN2" (shape bidirectional) (at 400.05 82.55 0) (effects (font (size 1.016 1.016)) (justify right bottom)))
 (wire (pts (xy 407.67 85.09) (xy 400.05 85.09)) (stroke (width 0) (type default)))
-(global_label "IGN3_LOGIC_OUT" (shape bidirectional) (at 400.05 85.09 0) (effects (font (size 1.016 1.016)) (justify right bottom)))
+(global_label "HARNESS_IGN3" (shape bidirectional) (at 400.05 85.09 0) (effects (font (size 1.016 1.016)) (justify right bottom)))
 (wire (pts (xy 407.67 87.63) (xy 400.05 87.63)) (stroke (width 0) (type default)))
-(global_label "IGN4_LOGIC_OUT" (shape bidirectional) (at 400.05 87.63 0) (effects (font (size 1.016 1.016)) (justify right bottom)))
+(global_label "HARNESS_IGN4" (shape bidirectional) (at 400.05 87.63 0) (effects (font (size 1.016 1.016)) (justify right bottom)))
 (wire (pts (xy 407.67 90.17) (xy 400.05 90.17)) (stroke (width 0) (type default)))
-(global_label "IGN5_LOGIC_OUT" (shape bidirectional) (at 400.05 90.17 0) (effects (font (size 1.016 1.016)) (justify right bottom)))
+(global_label "HARNESS_IGN5" (shape bidirectional) (at 400.05 90.17 0) (effects (font (size 1.016 1.016)) (justify right bottom)))
 (wire (pts (xy 407.67 92.71) (xy 400.05 92.71)) (stroke (width 0) (type default)))
-(global_label "IGN6_LOGIC_OUT" (shape bidirectional) (at 400.05 92.71 0) (effects (font (size 1.016 1.016)) (justify right bottom)))
+(global_label "HARNESS_IGN6" (shape bidirectional) (at 400.05 92.71 0) (effects (font (size 1.016 1.016)) (justify right bottom)))
 (wire (pts (xy 407.67 95.25) (xy 400.05 95.25)) (stroke (width 0) (type default)))
-(global_label "IGN7_LOGIC_OUT" (shape bidirectional) (at 400.05 95.25 0) (effects (font (size 1.016 1.016)) (justify right bottom)))
+(global_label "HARNESS_IGN7" (shape bidirectional) (at 400.05 95.25 0) (effects (font (size 1.016 1.016)) (justify right bottom)))
 (wire (pts (xy 407.67 97.79) (xy 400.05 97.79)) (stroke (width 0) (type default)))
-(global_label "IGN8_LOGIC_OUT" (shape bidirectional) (at 400.05 97.79 0) (effects (font (size 1.016 1.016)) (justify right bottom)))
+(global_label "HARNESS_IGN8" (shape bidirectional) (at 400.05 97.79 0) (effects (font (size 1.016 1.016)) (justify right bottom)))
 (wire (pts (xy 407.67 100.33) (xy 400.05 100.33)) (stroke (width 0) (type default)))
 (global_label "HARNESS_PI1" (shape bidirectional) (at 400.05 100.33 0) (effects (font (size 1.016 1.016)) (justify right bottom)))

Commit message: Redesign sport target as six DI/PI channels with two motors and one lambda
Connections:
- net PTA_H3: no longer J601.7
- net PTB_H3: no longer J601.15
- net HARNESS_IGN7: no longer names the net of J602.7
- net HARNESS_IGN8: no longer names the net of J602.8
- net HARNESS_PI7: no longer names the net of J602.15
- net HARNESS_PI8: no longer names the net of J602.16
- net HARNESS_WBO2_CONTACT1: no longer names the net of J604.27
- net HARNESS_WBO2_CONTACT2: no longer names the net of J604.28
- net HARNESS_WBO2_CONTACT3: no longer names the net of J604.29
- net HARNESS_WBO2_CONTACT4: no longer names the net of J604.30
- net HARNESS_WBO2_CONTACT5: no longer names the net of J604.31
- net HARNESS_WBO2_CONTACT6: no longer names the net of J604.32
- net MOTOR3_MOTOR_A: no longer names the net of J604.15
- net MOTOR3_MOTOR_B: no longer names the net of J604.16
- net MOTOR4_MOTOR_A: no longer names the net of J604.17
- net MOTOR4_MOTOR_B: no longer names the net of J604.18
- net PTA_L4: no longer names the net of J601.8
- net PTB_L4: no longer names the net of J601.16
- no-connect marks 0 -> 18
Other:
- title: Power8GDI TE34 harness boundary / UNQUALIFIED -> Power6GDI TE34 harness boundary / UNQUALIFIED
Changed lines of the file:
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@@
-(kicad_sch (version 20250114) (generator "eeschema") (paper "A2") (title_block (title "Power8GDI TE34 harness boundary / UNQUALIFIED") (rev "Engineering draft 0.1") (comment 1 "UNQUALIFIED: no manufacturing or engine approval"))
+(kicad_sch (version 20250114) (generator "eeschema") (paper "A2") (title_block (title "Power6GDI TE34 harness boundary / UNQUALIFIED") (rev "Engineering draft 0.1") (comment 1 "UNQUALIFIED: no manufacturing or engine approval"))
 (symbol (lib_id "Power8GDI_Board:TE_6437288_1_34") (at 139.7 100.33 0) (unit 1) (in_bom yes) (on_board yes) (dnp no) (property "Reference" "J601" (at 139.7 77.47 0) (effects (font (size 1.27 1.27)))) (property "Value" "6437288-1 / KEY1 CANDIDATE" (at 139.7 123.19 0) (effects (font (size 1.27 1.27)))) (property "Footprint" "Power8GDI_Board:TE_6437288-1_34way" (at 139.7 100.33 0) (effects (font (size 1.27 1.27)) (hide yes))) (property "Design note" "TE header C-9-1437287-8 A1 sheet2; numbering from mating housing RevP sheet3. Mechanical/continuity/keying review pending. Unimplemented circuits remain isolated HARNESS nets." (at 139.7 100.33 0) (effects (font (size 1.27 1.27)) (hide yes))) (pin "1") (pin "2") (pin "3") (pin "4") (pin "5") (pin "6") (pin "7") (pin "8") (pin "9") (pin "10") (pin "11") (pin "12") (pin "13") (pin "14") (pin "15") (pin "16") (pin "17") (pin "18") (pin "19") (pin "20") (pin "21") (pin "22") (pin "23") (pin "24") (pin "25") (pin "26") (pin "27") (pin "28") (pin "29") (pin "30") (pin "31") (pin "32") (pin "33") (pin "34") (instances (project "Power8GDI_Core" (path "/f4d21065-0a5b-5086-a08e-1af9469f04bd/df0c5f3e-1ee1-56be-91e2-4072c6105289" (reference "J601") (unit 1)))))
 (wire (pts (xy 127 80.01) (xy 119.38 80.01)) (stroke (width 0) (type default)))
@@
 (wire (pts (xy 127 92.71) (xy 119.38 92.71)) (stroke (width 0) (type default)))
 (global_label "PTA_L3" (shape bidirectional) (at 119.38 92.71 0) (effects (font (size 1.016 1.016)) (justify right bottom)))
-(wire (pts (xy 127 95.25) (xy 119.38 95.25)) (stroke (width 0) (type default)))
-(global_label "PTA_H3" (shape bidirectional) (at 119.38 95.25 0) (effects (font (size 1.016 1.016)) (justify right bottom)))
-(wire (pts (xy 127 97.79) (xy 119.38 97.79)) (stroke (width 0) (type default)))
-(global_label "PTA_L4" (shape bidirectional) (at 119.38 97.79 0) (effects (font (size 1.016 1.016)) (justify right bottom)))
+(no_connect (at 127 95.25))
+(no_connect (at 127 97.79))
 (wire (pts (xy 127 100.33) (xy 119.38 100.33)) (stroke (width 0) (type default)))
 (global_label "PTB_H1" (shape bidirectional) (at 119.38 100.33 0) (effects (font (size 1.016 1.016)) (justify right bottom)))
@@
 (wire (pts (xy 127 113.03) (xy 119.38 113.03)) (stroke (width 0) (type default)))
 (global_label "PTB_L3" (shape bidirectional) (at 119.38 113.03 0) (effects (font (size 1.016 1.016)) (justify right bottom)))
-(wire (pts (xy 127 115.57) (xy 119.38 115.57)) (stroke (width 0) (type default)))
-(global_label "PTB_H3" (shape bidirectional) (at 119.38 115.57 0) (effects (font (size 1.016 1.016)) (justify right bottom)))
-(wire (pts (xy 127 118.11) (xy 119.38 118.11)) (stroke (width 0) (type default)))
-(global_label "PTB_L4" (shape bidirectional) (at 119.38 118.11 0) (effects (font (size 1.016 1.016)) (justify right bottom)))
+(no_connect (at 127 115.57))
+(no_connect (at 127 118.11))
 (wire (pts (xy 127 120.65) (xy 119.38 120.65)) (stroke (width 0) (type default)))
 (global_label "PTA_H5PUMP" (shape bidirectional) (at 119.38 120.65 0) (effects (font (size 1.016 1.016)) (justify right bottom)))
@@
 (wire (pts (xy 407.67 92.71) (xy 400.05 92.71)) (stroke (width 0) (type default)))
 (global_label "HARNESS_IGN6" (shape bidirectional) (at 400.05 92.71 0) (effects (font (size 1.016 1.016)) (justify right bottom)))
-(wire (pts (xy 407.67 95.25) (xy 400.05 95.25)) (stroke (width 0) (type default)))
-(global_label "HARNESS_IGN7" (shape bidirectional) (at 400.05 95.25 0) (effects (font (size 1.016 1.016)) (justify right bottom)))
-(wire (pts (xy 407.67 97.79) (xy 400.05 97.79)) (stroke (width 0) (type default)))
-(global_label "HARNESS_IGN8" (shape bidirectional) (at 400.05 97.79 0) (effects (font (size 1.016 1.016)) (justify right bottom)))
+(no_connect (at 407.67 95.25))
+(no_connect (at 407.67 97.79))
 (wire (pts (xy 407.67 100.33) (xy 400.05 100.33)) (stroke (width 0) (type default)))
 (global_label "HARNESS_PI1" (shape bidirectional) (at 400.05 100.33 0) (effects (font (size 1.016 1.016)) (justify right bottom)))
@@
 (wire (pts (xy 407.67 113.03) (xy 400.05 113.03)) (stroke (width 0) (type default)))
 (global_label "HARNESS_PI6" (shape bidirectional) (at 400.05 113.03 0) (effects (font (size 1.016 1.016)) (justify right bottom)))
-(wire (pts (xy 407.67 115.57) (xy 400.05 115.57)) (stroke (width 0) (type default)))
-(global_label "HARNESS_PI7" (shape bidirectional) (at 400.05 115.57 0) (effects (font (size 1.016 1.016)) (justify right bottom)))
-(wire (pts (xy 407.67 118.11) (xy 400.05 118.11)) (stroke (width 0) (type default)))
-(global_label "HARNESS_PI8" (shape bidirectional) (at 400.05 118.11 0) (effects (font (size 1.016 1.016)) (justify right bottom)))
+(no_connect (at 407.67 115.57))
+(no_connect (at 407.67 118.11))
 (wire (pts (xy 407.67 120.65) (xy 400.05 120.65)) (stroke (width 0) (type default)))
 (global_label "HARNESS_VVT1" (shape bidirectional) (at 400.05 120.65 0) (effects (font (size 1.016 1.016)) (justify right bottom)))
@@
 (wire (pts (xy 407.67 273.05) (xy 400.05 273.05)) (stroke (width 0) (type default)))
 (global_label "CAN2_L" (shape bidirectional) (at 400.05 273.05 0) (effects (font (size 1.016 1.016)) (justify right bottom)))
-(wire (pts (xy 407.67 275.59) (xy 400.05 275.59)) (stroke (width 0) (type default)))
-(global_label "MOTOR3_MOTOR_A" (shape bidirectional) (at 400.05 275.59 0) (effects (font (size 1.016 1.016)) (justify right bottom)))
-(wire (pts (xy 407.67 278.13) (xy 400.05 278.13)) (stroke (width 0) (type default)))
-(global_label "MOTOR3_MOTOR_B" (shape bidirectional) (at 400.05 278.13 0) (effects (font (size 1.016 1.016)) (justify right bottom)))
-(wire (pts (xy 407.67 280.67) (xy 400.05 280.67)) (stroke (width 0) (type default)))
-(global_label "MOTOR4_MOTOR_A" (shape bidirectional) (at 400.05 280.67 0) (effects (font (size 1.016 1.016)) (justify right bottom)))
-(wire (pts (xy 433.07 240.03) (xy 440.69 240.03)) (stroke (width 0) (type default)))
-(global_label "MOTOR4_MOTOR_B" (shape bidirectional) (at 440.69 240.03 180) (effects (font (size 1.016 1.016)) (justify left bottom)))
+(no_connect (at 407.67 275.59))
+(no_connect (at 407.67 278.13))
+(no_connect (at 407.67 280.67))
+(no_connect (at 433.07 240.03))
 (wire (pts (xy 433.07 242.57) (xy 440.69 242.57)) (stroke (width 0) (type default)))
 (global_label "HARNESS_AUX_ANALOG1" (shape bidirectional) (at 440.69 242.57 180) (effects (font (size 1.016 1.016)) (justify left bottom)))
@@
 (wire (pts (xy 433.07 260.35) (xy 440.69 260.35)) (stroke (width 0) (type default)))
 (global_label "HARNESS_WBO1_CONTACT6" (shape bidirectional) (at 440.69 260.35 180) (effects (font (size 1.016 1.016)) (justify left bottom)))
-(wire (pts (xy 433.07 262.89) (xy 440.69 262.89)) (stroke (width 0) (type default)))
-(global_label "HARNESS_WBO2_CONTACT1" (shape bidirectional) (at 440.69 262.89 180) (effects (font (size 1.016 1.016)) (justify left bottom)))
-(wire (pts (xy 433.07 265.43) (xy 440.69 265.43)) (stroke (width 0) (type default)))
-(global_label "HARNESS_WBO2_CONTACT2" (shape bidirectional) (at 440.69 265.43 180) (effects (font (size 1.016 1.016)) (justify left bottom)))
-(wire (pts (xy 433.07 267.97) (xy 440.69 267.97)) (stroke (width 0) (type default)))
-(global_label "HARNESS_WBO2_CONTACT3" (shape bidirectional) (at 440.69 267.97 180) (effects (font (size 1.016 1.016)) (justify left bottom)))
-(wire (pts (xy 433.07 270.51) (xy 440.69 270.51)) (stroke (width 0) (type default)))
-(global_label "HARNESS_WBO2_CONTACT4" (shape bidirectional) (at 440.69 270.51 180) (effects (font (size 1.016 1.016)) (justify left bottom)))
-(wire (pts (xy 433.07 273.05) (xy 440.69 273.05)) (stroke (width 0) (type default)))
-(global_label "HARNESS_WBO2_CONTACT5" (shape bidirectional) (at 440.69 273.05 180) (effects (font (size 1.016 1.016)) (justify left bottom)))
-(wire (pts (xy 433.07 275.59) (xy 440.69 275.59)) (stroke (width 0) (type default)))
-(global_label "HARNESS_WBO2_CONTACT6" (shape bidirectional) (at 440.69 275.59 180) (effects (font (size 1.016 1.016)) (justify left bottom)))
+(no_connect (at 433.07 262.89))
+(no_connect (at 433.07 265.43))
+(no_connect (at 433.07 267.97))
+(no_connect (at 433.07 270.51))
+(no_connect (at 433.07 273.05))
+(no_connect (at 433.07 275.59))
 (wire (pts (xy 433.07 278.13) (xy 440.69 278.13)) (stroke (width 0) (type default)))
 (global_label "USB_SHIELD" (shape bidirectional) (at 440.69 278.13 180) (effects (font (size 1.016 1.016)) (justify left bottom)))

Commit message: Review B58 injector power stage and bind selected GDI6 BOM
Parts:
- J601, J602, J603, J604: Hardware_Qualification (none) -> PINOUT_RATINGS_AND_DELIVERY_SUFFIX_REVIEW_PENDING; MPN (none) -> 6437288-1; Manufacturer (none) -> TE Connectivity; Procurement_Status (none) -> REFERENCE_MPN_RETAINED; Purchase_Released (none) -> false; Selection_Gaps (none) -> ["Existing schematic MPN retained. Complete circuit rating/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; Selection_ID (none) -> SEL-752f08db694c; Selection_Ratings (none) -> {}; Selection_Source_URLs (none) -> https://www.te.com/en/product-6437288-1.html
