File: Power8GDI/hardware/design/gdi/permission.kicad_sch (KiCad schematic)
At the start: 8 parts, among them U5101 SN74LVC2G08QDCURQ1

Commit message: Review B58 injector power stage and bind selected GDI6 BOM
Parts:
- C5101: Hardware_Qualification (none) -> BOARD_QUALIFICATION_PENDING; MPN (none) -> C0805C104K1RACTU; Manufacturer (none) -> KEMET; Procurement_Status (none) -> SELECTED_CATALOG_ITEM; Purchase_Released (none) -> false; Selection_Gaps (none) -> []; Selection_ID (none) -> SEL-50b208aec5b1; Selection_Ratings (none) -> {"capacitance_pf": 100000, "dielectric": "X7R", "rated_volt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; Selection_Source_URLs (none) -> https://www.mouser.com/datasheet/3/72/1/C0805C104K1RACTU.pdf
- R5101, R5102, R5103, R5104, R5105, R5106: Hardware_Qualification (none) -> BOARD_QUALIFICATION_PENDING; MPN (none) -> CRCW060310K0FKEA; Manufacturer (none) -> Vishay; Procurement_Status (none) -> SELECTED_FAMILY_CODE; Purchase_Released (none) -> false; Selection_Gaps (none) -> []; Selection_ID (none) -> SEL-9c0806476875; Selection_Ratings (none) -> {"aec_q200": true, "derating": "Use manufacturer power vers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; Selection_Source_URLs (none) -> https://www.vishay.com/docs/20035/dcrcwe3.pdf
- U5101: Hardware_Qualification (none) -> PINOUT_RATINGS_AND_DELIVERY_SUFFIX_REVIEW_PENDING; MPN (none) -> SN74LVC2G08QDCURQ1; Manufacturer (none) -> Texas Instruments; Procurement_Status (none) -> REFERENCE_MPN_RETAINED; Purchase_Released (none) -> false; Selection_Gaps (none) -> ["Existing schematic MPN retained. Complete circuit rating/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; Selection_ID (none) -> SEL-d966fefb13e0; Selection_Ratings (none) -> {}; Selection_Source_URLs (none) -> https://www.ti.com/product/SN74LVC2G08-Q1/part-details/SN74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
