File: Power8GDI/hardware/design/gdi/stage_a.kicad_sch (KiCad schematic)
At the start: 134 parts, among them Q201 BUK9230-100B, Q202 BUK9230-100B, Q203 BUK9230-100B, Q204 BUK9230-100B, Q205 BUK9230-100B, Q206 BUK9230-100B, Q207 BUK9230-100B, Q208 BUK9230-100B, Q209 BUK9230-100B, Q210 BUK9230-100B, Q211 BUK9230-100B, Q212 BUK9230-100B, Q213 BUK9230-100B, U201 MC33PT2001AE, U249 NCV78M05ABDTRKG, Y201 1MHz

Commit message: Checkpoint GDI protected feeds and permissions before server handoff
Connections:
- net PTA_DRVEN renamed PTA_DRVEN_GATED
- net PTA_START6 renamed HPFP1
Other:
- note added: "Independent 5V candidate: 7-20V regulation range; 35V ABS MAX is not a surge rating. PT2001 VCC5/VCCIO current UNKNOWN; 500mA requires adequate heatsinking. VBAT_GDI_A comes from LM74800 protection sheet; external fuse and transient tests required."
- note added: "R299 remains DNP pending PT electrical/shutdown qualification. HPFP START6 is wired; loaded microcode/mask still requires verification. Hardware permission and protected battery input are on separate GDI sheets."
- note removed: "DO NOT ENERGIZE: hardware inhibit missing; R299 MUST REMAIN DNP. HPFP1/2 to START5/6 mapping unresolved. Source values are NOT load-qualified."
- note removed: "Independent 5V candidate: 7-20V regulation range; 35V ABS MAX is not a surge rating. PT2001 VCC5/VCCIO current UNKNOWN; 500mA requires adequate heatsinking. Source VBAT_GDI_A requires external fuse/reverse/load-dump protection."
Changed lines of the file:
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@@
       (justify left bottom))
 )
-  (global_label "PTA_START6"
+  (global_label "HPFP1"
     (shape bidirectional)
     (at 179.07 57.15 180)
@@
           (reference "R299")
           (unit 1)))))
-  (global_label "PTA_DRVEN"
+  (global_label "PTA_DRVEN_GATED"
     (shape bidirectional)
     (at 218.44 15.24 0)
@@
       (justify left))
 )
-  (text "DO NOT ENERGIZE: hardware inhibit missing; R299 MUST REMAIN DNP.\nHPFP1/2 to START5/6 mapping unresolved. Source values are NOT load-qualified."
+  (text "R299 remains DNP pending PT electrical/shutdown qualification.\nHPFP START6 is wired; loaded microcode/mask still requires verification.\nHardware permission and protected battery input are on separate GDI sheets."
     (at 15.24 17.78 0)
     (effects
@@
       (justify left))
 )
-  (text "Independent 5V candidate: 7-20V regulation range; 35V ABS MAX is not a surge rating.\nPT2001 VCC5/VCCIO current UNKNOWN; 500mA requires adequate heatsinking.\nSource VBAT_GDI_A requires external fuse/reverse/load-dump protection."
+  (text "Independent 5V candidate: 7-20V regulation range; 35V ABS MAX is not a surge rating.\nPT2001 VCC5/VCCIO current UNKNOWN; 500mA requires adequate heatsinking.\nVBAT_GDI_A comes from LM74800 protection sheet; external fuse and transient tests required."
     (at 266.7 83.82 0)
     (effects

Commit message: Redesign sport target as six DI/PI channels with two motors and one lambda
Parts:
- removed C227: 4700p, Power8GDI_GDI:REF_C50, symbol Power8GDI_GDI:hellen_one_common_Cap
- removed C237: 1000pF, Power8GDI_GDI:REF_C61, symbol Power8GDI_GDI:Device_C
- removed D206: STPS2H100UY, Power8GDI_GDI:REF_D14, symbol Power8GDI_GDI:Device_D_Schottky_Small
- removed Q210: BUK9230-100B, Power8GDI_GDI:REF_Q10, symbol Power8GDI_GDI:Device_Q_NMOS_GDS
- removed R209: 10, Power8GDI_GDI:REF_R18, symbol Power8GDI_GDI:Device_R
- removed TP204: TestPoint, Power8GDI_GDI:REF_S4, symbol Power8GDI_GDI:Connector_TestPoint
- added R297: 10k 1%, Power8GDI_GDI:REF_R123, symbol Power8GDI_GDI:Device_R
Connections:
- net GND: now also R297.2
- net PTA_VCCIO: now reaches C235.2, R221.4, U201.17 (VCCIO)
- net DI4 renamed PTA_UNUSED_START4
- net PTA_UNUSED_START4: now also R297.1
- net PTA_L4: no longer names the net of U201.35 (D_LS4)
- no-connect marks 3 -> 5
Other:
- title: Power8GDI Stage A - reference draft -> Power6GDI Stage A - 3 DI + 1 HPFP candidate

Commit message: Review B58 injector power stage and bind selected GDI6 BOM
Parts:
- C201: Hardware_Qualification (none) -> BOARD_QUALIFICATION_PENDING; LCSC C15849 -> (none); MPN (none) -> C0603C105K3RACTU; Manufacturer (none) -> KEMET; Procurement_Status (none) -> SELECTED_CATALOG_ITEM; Purchase_Released (none) -> false; Selection_Gaps (none) -> []; Selection_ID (none) -> SEL-4bca20b134b8; Selection_Ratings (none) -> {"capacitance_pf": 1000000, "dc_bias_qualification": "PENDI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; Selection_Source_URLs (none) -> https://search.kemet.com/download/specsheet/C0603C105K3RACTU; Source_LCSC (none) -> C15849
- C202, C203, C204, C211, C236, C244: Hardware_Qualification (none) -> BOARD_QUALIFICATION_PENDING; LCSC C576850 -> (none); MPN (none) -> C0603C331J1GACTU; Manufacturer (none) -> KEMET; Procurement_Status (none) -> SELECTED_CATALOG_ITEM; Purchase_Released (none) -> false; Selection_Gaps (none) -> []; Selection_ID (none) -> SEL-fcb87b627c08; Selection_Ratings (none) -> {"capacitance_pf": 330, "dielectric": "C0G", "rated_voltage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; Selection_Source_URLs (none) -> https://search.kemet.com/download/specsheet/C0603C331J1GACTU; Source_LCSC (none) -> C576850
- C205, C206: value 1200uF -> 1300uF 50V; Hardware_Qualification (none) -> INPUT_INRUSH_AND_TRANSIENT_REVIEW_REQUIRED; LCSC C5111952 -> (none); MPN (none) -> UBY1H132MHL6; Manufacturer (none) -> Nichicon; Procurement_Status (none) -> SELECTED_CONDITIONAL; Purchase_Released (none) -> false; Selection_Gaps (none) -> ["1300uF replaces1200uF input bulk; +8.3% capacitance/inrus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; Selection_ID (none) -> SEL-7599e2dc5064; Selection_Ratings (none) -> {"body_height_mm": 25, "capacitance_pf": 1300000000, "diame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; Selection_Source_URLs (none) -> https://www.nichicon.com/getmedia/640b351d-ceef-400c-b016-3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; Source_LCSC_previous_value (none) -> C5111952
- C207, C209: Hardware_Qualification (none) -> BOOST_RIPPLE_AND_VOLTAGE_MARGIN_REVIEW_REQUIRED; LCSC C5110766 -> (none); MPN (none) -> UBY1K471MHL; Manufacturer (none) -> Nichicon; Procurement_Status (none) -> SELECTED_CONDITIONAL; Purchase_Released (none) -> false; Selection_Gaps (none) -> ["80V rating on nominal65V boost requires measured overshoo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; Selection_ID (none) -> SEL-37b09fd0533a; Selection_Ratings (none) -> {"body_height_mm": 20, "capacitance_pf": 470000000, "diamet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; Selection_Source_URLs (none) -> https://www.nichicon.com/getmedia/640b351d-ceef-400c-b016-3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; Source_LCSC (none) -> C5110766
- C208, C246, C247, C248: Hardware_Qualification (none) -> BOARD_QUALIFICATION_PENDING; LCSC C342873 -> (none); MPN (none) -> C0805C224K1RACTU; Manufacturer (none) -> KEMET; Procurement_Status (none) -> SELECTED_CATALOG_ITEM; Purchase_Released (none) -> false; Selection_Gaps (none) -> []; Selection_ID (none) -> SEL-1427fa3d6f1a; Selection_Ratings (none) -> {"capacitance_pf": 220000, "dielectric": "X7R", "rated_volt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; Selection_Source_URLs (none) -> https://content.kemet.com/datasheets/CER_ENG_KIT_30.pdf; Source_LCSC (none) -> C342873
- C210, C213, C214, C215, C235: Hardware_Qualification (none) -> BOARD_QUALIFICATION_PENDING; LCSC C14663 -> (none); MPN (none) -> C0603C104K5RACTU; Manufacturer (none) -> KEMET; Procurement_Status (none) -> SELECTED_CATALOG_ITEM; Purchase_Released (none) -> false; Selection_Gaps (none) -> []; Selection_ID (none) -> SEL-6bf9727c4e40; Selection_Ratings (none) -> {"capacitance_pf": 100000, "dielectric": "X7R", "rated_volt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; Selection_Source_URLs (none) -> https://search.kemet.com/download/specsheet/C0603C104K5RACTU; Source_LCSC (none) -> C14663
- C212: Hardware_Qualification (none) -> BOARD_QUALIFICATION_PENDING; LCSC C19666 -> (none); MPN (none) -> GMC10X7R475K16NT; Manufacturer (none) -> Cal-Chip Electronics; Procurement_Status (none) -> SELECTED_CATALOG_ITEM; Purchase_Released (none) -> false; Selection_Gaps (none) -> []; Selection_ID (none) -> SEL-541f7eb877a5; Selection_Ratings (none) -> {"capacitance_pf": 4700000, "dc_bias_qualification": "PENDI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; Selection_Source_URLs (none) -> https://www.digikey.com/en/products/detail/cal-chip-electro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; Source_LCSC (none) -> C19666
- C216, C217, C218, C219, C240: Hardware_Qualification (none) -> BOARD_QUALIFICATION_PENDING; LCSC C1615 -> (none); MPN (none) -> 0603B334K250NT; Manufacturer (none) -> FH; Procurement_Status (none) -> SELECTED_CATALOG_ITEM; Purchase_Released (none) -> false; Selection_Gaps (none) -> []; Selection_ID (none) -> SEL-a2a1a7d509a7; Selection_Ratings (none) -> {"capacitance_pf": 330000, "dielectric": "X7R", "rated_volt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; Selection_Source_URLs (none) -> https://www.lcsc.com/product-detail/C1615.html; Source_LCSC (none) -> C1615
- C220, C221, C222, C223, C224, C225, C226, C241, C242, C249, C250, C251, C253: Hardware_Qualification (none) -> BOARD_QUALIFICATION_PENDING; LCSC C342899 -> (none); MPN (none) -> C0603C472J1GACTU; Manufacturer (none) -> KEMET; Procurement_Status (none) -> SELECTED_CATALOG_ITEM; Purchase_Released (none) -> false; Selection_Gaps (none) -> []; Selection_ID (none) -> SEL-d949ccbf136e; Selection_Ratings (none) -> {"capacitance_pf": 4700, "dielectric": "C0G", "rated_voltag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; Selection_Source_URLs (none) -> https://www.digikey.com/en/products/detail/kemet/C0603C472J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; Source_LCSC (none) -> C342899
- C228, C229, C230, C231, C232, C233, C234, C238, C239, C243, C252, C254: Hardware_Qualification (none) -> BOARD_QUALIFICATION_PENDING; LCSC C106247 -> (none); MPN (none) -> C0603C102J1GACTU; Manufacturer (none) -> KEMET; Procurement_Status (none) -> SELECTED_CATALOG_ITEM; Purchase_Released (none) -> false; Selection_Gaps (none) -> []; Selection_ID (none) -> SEL-ec742f39ec1f; Selection_Ratings (none) -> {"capacitance_pf": 1000, "dielectric": "C0G", "rated_voltag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; Selection_Source_URLs (none) -> https://search.kemet.com/download/specsheet/C0603C102J1GACTU; Source_LCSC (none) -> C106247
- C245: Hardware_Qualification (none) -> BOARD_QUALIFICATION_PENDING; LCSC C525649 -> (none); MPN (none) -> C0603C471J1GACTU; Manufacturer (none) -> KEMET; Procurement_Status (none) -> SELECTED_CATALOG_ITEM; Purchase_Released (none) -> false; Selection_Gaps (none) -> []; Selection_ID (none) -> SEL-1e0888f0acc7; Selection_Ratings (none) -> {"capacitance_pf": 470, "dielectric": "C0G", "rated_voltage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; Selection_Source_URLs (none) -> https://www.digikey.com/en/products/detail/kemet/C0603C471J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; Source_LCSC (none) -> C525649
- C298: Hardware_Qualification (none) -> BOARD_QUALIFICATION_PENDING; MPN (none) -> C0805C334K5RACTU; Manufacturer (none) -> KEMET; Procurement_Status (none) -> SELECTED_CATALOG_ITEM; Purchase_Released (none) -> false; Selection_Gaps (none) -> []; Selection_ID (none) -> SEL-02d268337ca5; Selection_Ratings (none) -> {"capacitance_pf": 330000, "dielectric": "X7R", "rated_volt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; Selection_Source_URLs (none) -> https://www.digikey.com/en/products/detail/kemet/C0805C334K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
- C299: Hardware_Qualification (none) -> BOARD_QUALIFICATION_PENDING; MPN (none) -> C0805C104K1RACTU; Manufacturer (none) -> KEMET; Procurement_Status (none) -> SELECTED_CATALOG_ITEM; Purchase_Released (none) -> false; Selection_Gaps (none) -> []; Selection_ID (none) -> SEL-50b208aec5b1; Selection_Ratings (none) -> {"capacitance_pf": 100000, "dielectric": "X7R", "rated_volt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; Selection_Source_URLs (none) -> https://www.mouser.com/datasheet/3/72/1/C0805C104K1RACTU.pdf
- D201, D204, D205, D207, D208, D209, D210: Hardware_Qualification (none) -> PINOUT_RATINGS_AND_DELIVERY_SUFFIX_REVIEW_PENDING; LCSC C163541 -> (none); MPN (none) -> STPS2H100UY; Manufacturer (none) -> STMicroelectronics; Procurement_Status (none) -> REFERENCE_MPN_RETAINED; Purchase_Released (none) -> false; Selection_Gaps (none) -> ["Existing schematic MPN retained. Complete circuit rating/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; Selection_ID (none) -> SEL-2af9fd635e9e; Selection_Ratings (none) -> {}; Selection_Source_URLs (none) -> https://www.st.com/en/search.html#q=STPS2H100UY; Source_LCSC (none) -> C163541
- D202, D203: Hardware_Qualification (none) -> REPETITIVE_PULSE_REVIEW_REQUIRED; LCSC C135494 -> (none); MPN (none) -> SBR10200CTL-13; Manufacturer (none) -> Diodes Incorporated; Procurement_Status (none) -> SELECTED_CONDITIONAL; Purchase_Released (none) -> false; Selection_Gaps (none) -> ["Qrr/commutation and actual diode temperature at DI duty n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; Selection_ID (none) -> SEL-64bdec054294; Selection_Ratings (none) -> {"configuration": "dual common cathode", "if_average_total_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; Selection_Source_URLs (none) -> https://www.diodes.com/part/view/SBR10200CTL https://www.di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; Source_LCSC (none) -> C135494
- D211: Hardware_Qualification (none) -> LED_CURRENT_AND_VISIBILITY_REVIEW_REQUIRED; LCSC C2296 -> (none); MPN (none) -> KT-0805Y; Manufacturer (none) -> Hubei KENTO Electronics; Procurement_Status (none) -> SELECTED_CONDITIONAL; Purchase_Released (none) -> false; Selection_Gaps (none) -> ["Source identity retained; forward current, temperature an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; Selection_ID (none) -> SEL-7f6b4dbc5098; Selection_Ratings (none) -> {"color": "yellow", "package": "0805"}; Selection_Source_URLs (none) -> https://www.lcsc.com/product-detail/C2296.html; Source_LCSC (none) -> C2296
- D212: Hardware_Qualification (none) -> PULSE_AND_THERMAL_REVIEW_REQUIRED; LCSC C260365 -> (none); MPN (none) -> SDURB1020CT; Manufacturer (none) -> SMC Diode Solutions; Procurement_Status (none) -> SELECTED_CONDITIONAL; Purchase_Released (none) -> false; Selection_Gaps (none) -> ["DigiKey source only offered MOQ800 full reel in price rev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; Selection_ID (none) -> SEL-1770aa2aa0fe; Selection_Ratings (none) -> {"configuration": "dual common cathode", "if_average_total_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; Selection_Source_URLs (none) -> https://www.digikey.com/en/products/detail/smc-diode-soluti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; Source_LCSC (none) -> C260365
- L201: Hardware_Qualification (none) -> MAGNETIC_THERMAL_AND_LAND_PATTERN_REVIEW_REQUIRED; LCSC C380073 -> (none); MPN (none) -> MS1350-6R8M; Manufacturer (none) -> COILMX; Procurement_Status (none) -> SELECTED_CONDITIONAL; Purchase_Released (none) -> false; Selection_Gaps (none) -> ["Original vendor identity recovered. Saturation drop perce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; Selection_ID (none) -> SEL-024e29fce0f3; Selection_Ratings (none) -> {"body_mm": [13.8, 12.6], "catalog_current_a": 10, "catalog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; Selection_Source_URLs (none) -> https://jlcpcb.com/partdetail/COILMX-MS13506R8M/C380073; Source_LCSC (none) -> C380073
- L202: Hardware_Qualification (none) -> MAGNETIC_THERMAL_AND_LAND_PATTERN_REVIEW_REQUIRED; LCSC C237980 -> (none); MPN (none) -> BCIHP1770-100M; Manufacturer (none) -> BaoCheng; Procurement_Status (none) -> SELECTED_CONDITIONAL; Purchase_Released (none) -> false; Selection_Gaps (none) -> ["Original vendor identity recovered. Saturation definition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; Selection_ID (none) -> SEL-00d67cd6f28d; Selection_Ratings (none) -> {"catalog_current_a": 17, "catalog_saturation_current_a": 1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; Selection_Source_URLs (none) -> https://www.lcsc.com/pt/product-detail/C237980.html; Source_LCSC (none) -> C237980
- Q201, Q202, Q203, Q204, Q205, Q206, Q207, Q208, Q209, Q211, Q212, Q213: value BUK9230-100B -> IPD60N10S4L12ATMA1; Hardware_Qualification (none) -> CONDITIONAL_HW_REVIEW; LCSC C89735 -> (none); MFG,MFG# Nexperia,BUK9230-100B -> (none); MPN (none) -> IPD60N10S4L12ATMA1; Manufacturer (none) -> Infineon Technologies; Procurement_Status (none) -> SELECTED_CONDITIONAL; Purchase_Released (none) -> false; Selection_Gaps (none) -> ["Hardware engineer approved candidate and matched DPAK geo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; Selection_ID (none) -> SEL-29d58d042c3c; Selection_Ratings (none) -> {"manufacturer_package": "PG-TO252-3-313", "minimum_gate_dr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; Selection_Source_URLs (none) -> https://www.infineon.com/assets/row/public/documents/10/49/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; Source_LCSC_obsolete_BUK (none) -> C89735; Source_MFG,MFG# (none) -> Nexperia,BUK9230-100B; Source_VEND1,VEND1# (none) -> DIGI,1727-4708-1-ND; Source_VEND2,VEND2# (none) -> ,; VEND1,VEND1# DIGI,1727-4708-1-ND -> (none); VEND2,VEND2# , -> (none)
- R201, R202, R204, R205, R206, R207, R208, R210, R211, R214, R226: Hardware_Qualification (none) -> BOARD_QUALIFICATION_PENDING; LCSC C22859 -> (none); MPN (none) -> CRCW060310R0FKEA; Manufacturer (none) -> Vishay; Procurement_Status (none) -> SELECTED_FAMILY_CODE; Purchase_Released (none) -> false; Selection_Gaps (none) -> []; Selection_ID (none) -> SEL-887dce68fe1a; Selection_Ratings (none) -> {"aec_q200": true, "derating": "Use manufacturer power vers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; Selection_Source_URLs (none) -> https://www.vishay.com/docs/20035/dcrcwe3.pdf; Source_LCSC (none) -> C22859
- R203, R212, R213, R215, R221: Hardware_Qualification (none) -> PULSE_THERMAL_AND_KELVIN_LAYOUT_REVIEW_REQUIRED; LCSC C309628 -> (none); MPN (none) -> WSLP1206R0100FEA; Manufacturer (none) -> Vishay; Procurement_Status (none) -> SELECTED_CONDITIONAL; Purchase_Released (none) -> false; Selection_Gaps (none) -> ["Original C309628 thick-film1500ppm/K rejected for precisi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; Selection_ID (none) -> SEL-618c5b25d6ed; Selection_Ratings (none) -> {"derating": "Use manufacturer power versus ambient/termina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; Selection_Source_URLs (none) -> https://www.vishay.com/docs/30122/wslp.pdf https://www.digi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; Source_LCSC (none) -> C309628
- R216: Hardware_Qualification (none) -> BOARD_QUALIFICATION_PENDING; LCSC C17477 -> (none); MPN (none) -> CRCW08050000Z0EA; Manufacturer (none) -> Vishay; Procurement_Status (none) -> SELECTED_FAMILY_CODE; Purchase_Released (none) -> false; Selection_Gaps (none) -> []; Selection_ID (none) -> SEL-0d6eae76dd7d; Selection_Ratings (none) -> {"aec_q200": true, "current_a": 2.5, "power_reference_tempe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; Selection_Source_URLs (none) -> https://www.vishay.com/docs/20035/dcrcwe3.pdf; Source_LCSC (none) -> C17477
- R217: Hardware_Qualification (none) -> BOARD_QUALIFICATION_PENDING; LCSC C22962 -> (none); MPN (none) -> CRCW0603220RFKEA; Manufacturer (none) -> Vishay; Procurement_Status (none) -> SELECTED_FAMILY_CODE; Purchase_Released (none) -> false; Selection_Gaps (none) -> []; Selection_ID (none) -> SEL-da2bcd5c4b94; Selection_Ratings (none) -> {"aec_q200": true, "derating": "Use manufacturer power vers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; Selection_Source_URLs (none) -> https://www.vishay.com/docs/20035/dcrcwe3.pdf; Source_LCSC (none) -> C22962
- R219: Hardware_Qualification (none) -> BOARD_QUALIFICATION_PENDING; LCSC C25197 -> (none); MPN (none) -> CRCW06035R10FKEA; Manufacturer (none) -> Vishay; Procurement_Status (none) -> SELECTED_FAMILY_CODE; Purchase_Released (none) -> false; Selection_Gaps (none) -> []; Selection_ID (none) -> SEL-cb8e07313c84; Selection_Ratings (none) -> {"aec_q200": true, "derating": "Use manufacturer power vers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; Selection_Source_URLs (none) -> https://www.vishay.com/docs/20035/dcrcwe3.pdf; Source_LCSC (none) -> C25197
- R220: Hardware_Qualification (none) -> BOARD_QUALIFICATION_PENDING; LCSC C23242 -> (none); MPN (none) -> CRCW060375K0FKEA; Manufacturer (none) -> Vishay; Procurement_Status (none) -> SELECTED_FAMILY_CODE; Purchase_Released (none) -> false; Selection_Gaps (none) -> []; Selection_ID (none) -> SEL-4f9f93b34738; Selection_Ratings (none) -> {"aec_q200": true, "derating": "Use manufacturer power vers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; Selection_Source_URLs (none) -> https://www.vishay.com/docs/20035/dcrcwe3.pdf; Source_LCSC (none) -> C23242
- R227, R228, R229: Hardware_Qualification (none) -> BOARD_QUALIFICATION_PENDING; LCSC C21190 -> (none); MPN (none) -> CRCW06031K00FKEA; Manufacturer (none) -> Vishay; Procurement_Status (none) -> SELECTED_FAMILY_CODE; Purchase_Released (none) -> false; Selection_Gaps (none) -> []; Selection_ID (none) -> SEL-38197231a947; Selection_Ratings (none) -> {"aec_q200": true, "derating": "Use manufacturer power vers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; Selection_Source_URLs (none) -> https://www.vishay.com/docs/20035/dcrcwe3.pdf; Source_LCSC (none) -> C21190
- R230, R231: Hardware_Qualification (none) -> BOARD_QUALIFICATION_PENDING; LCSC C17944 -> (none); MPN (none) -> CRCW12062K00FKEA; Manufacturer (none) -> Vishay; Procurement_Status (none) -> SELECTED_FAMILY_CODE; Purchase_Released (none) -> false; Selection_Gaps (none) -> []; Selection_ID (none) -> SEL-db0fa18c585f; Selection_Ratings (none) -> {"aec_q200": true, "derating": "Use manufacturer power vers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; Selection_Source_URLs (none) -> https://www.vishay.com/docs/20035/dcrcwe3.pdf; Source_LCSC (none) -> C17944
- R232, R233, R234, R235, R236, R237, R238, R239, R240: Hardware_Qualification (none) -> BOARD_QUALIFICATION_PENDING; LCSC C17756 -> (none); MPN (none) -> CRCW080556K0FKEA; Manufacturer (none) -> Vishay; Procurement_Status (none) -> SELECTED_FAMILY_CODE; Purchase_Released (none) -> false; Selection_Gaps (none) -> []; Selection_ID (none) -> SEL-d8cdbc522903; Selection_Ratings (none) -> {"aec_q200": true, "derating": "Use manufacturer power vers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; Selection_Source_URLs (none) -> https://www.vishay.com/docs/20035/dcrcwe3.pdf; Source_LCSC (none) -> C17756
- R297: Hardware_Qualification (none) -> BOARD_QUALIFICATION_PENDING; MPN (none) -> CRCW060310K0FKEA; Manufacturer (none) -> Vishay; Procurement_Status (none) -> SELECTED_FAMILY_CODE; Purchase_Released (none) -> false; Selection_Gaps (none) -> []; Selection_ID (none) -> SEL-9c0806476875; Selection_Ratings (none) -> {"aec_q200": true, "derating": "Use manufacturer power vers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; Selection_Source_URLs (none) -> https://www.vishay.com/docs/20035/dcrcwe3.pdf
- R298: Hardware_Qualification (none) -> BOARD_QUALIFICATION_PENDING; MPN (none) -> CRCW0603910RFKEA; Manufacturer (none) -> Vishay; Procurement_Status (none) -> SELECTED_FAMILY_CODE; Purchase_Released (none) -> false; Selection_Gaps (none) -> []; Selection_ID (none) -> SEL-73b716f91ac6; Selection_Ratings (none) -> {"aec_q200": true, "derating": "Use manufacturer power vers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; Selection_Source_URLs (none) -> https://www.vishay.com/docs/20035/dcrcwe3.pdf
- U201: Hardware_Qualification (none) -> GATE_DRIVE_AND_HIGH_ENERGY_REVIEW_REQUIRED; MPN (none) -> MC33PT2001AE; Manufacturer (none) -> NXP Semiconductors; Procurement_Status (none) -> SELECTED_CONDITIONAL; Purchase_Released (none) -> false; Selection_Gaps (none) -> ["AE72V version retained. Do not infer HAE80V limits. Valid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; Selection_ID (none) -> SEL-43c7059ab190; Selection_Ratings (none) -> {"body_mm": [10, 10, 1.4], "end_of_injection_detection": fa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; Selection_Source_URLs (none) -> https://www.nxp.com/docs/en/data-sheet/MC33PT2001_SDS.pdf
- U249: Hardware_Qualification (none) -> PINOUT_RATINGS_AND_DELIVERY_SUFFIX_REVIEW_PENDING; MPN (none) -> NCV78M05ABDTRKG; Manufacturer (none) -> onsemi; Procurement_Status (none) -> REFERENCE_MPN_RETAINED; Purchase_Released (none) -> false; Selection_Gaps (none) -> ["Existing schematic MPN retained. Complete circuit rating/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; Selection_ID (none) -> SEL-017b10d65e0f; Selection_Ratings (none) -> {}; Selection_Source_URLs (none) -> https://www.onsemi.com/pdf/datasheet/mc78m00-d.pdf
- Y201: Hardware_Qualification (none) -> CLOCK_AND_LAND_PATTERN_REVIEW_REQUIRED; LCSC C2901463 -> (none); MPN (none) -> SIT8924BM-81-33E-1.000000; Manufacturer (none) -> SiTime; Procurement_Status (none) -> SELECTED_CONDITIONAL; Purchase_Released (none) -> false; Selection_Gaps (none) -> ["Hardware found FN pad mismatch: source span5.08x4.4/pads1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; Selection_ID (none) -> SEL-da91e4c249ac; Selection_Ratings (none) -> {"aec_q100": true, "body_mm": [7, 5, 1], "current_supply_ma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; Selection_Source_URLs (none) -> https://www.sitime.com/support/resource-library/datasheets/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; Source_LCSC (none) -> C2901463
