File: Power8GDI/hardware/design/ignition/ignition_2.kicad_sch (KiCad schematic)
At the start: 16 parts, among them Q5440 STGB18N40LZT4, U5440 LTC6993HS6-1#WTRPBF, U5441 SN74LVC1G11BDCKRQ1, U5442 INA300AQDGSRQ1

Commit message: Review B58 injector power stage and bind selected GDI6 BOM
Parts:
- C5440, C5441, C5442: Hardware_Qualification (none) -> BOARD_QUALIFICATION_PENDING; MPN (none) -> C0603C104K5RACTU; Manufacturer (none) -> KEMET; Procurement_Status (none) -> SELECTED_CATALOG_ITEM; Purchase_Released (none) -> false; Selection_Gaps (none) -> []; Selection_ID (none) -> SEL-6bf9727c4e40; Selection_Ratings (none) -> {"capacitance_pf": 100000, "dielectric": "X7R", "rated_volt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; Selection_Source_URLs (none) -> https://search.kemet.com/download/specsheet/C0603C104K5RACTU
- Q5440: Hardware_Qualification (none) -> PINOUT_RATINGS_AND_DELIVERY_SUFFIX_REVIEW_PENDING; MPN (none) -> STGB18N40LZT4; Manufacturer (none) -> STMicroelectronics; Procurement_Status (none) -> REFERENCE_MPN_RETAINED; Purchase_Released (none) -> false; Selection_Gaps (none) -> ["Existing schematic MPN retained. Complete circuit rating/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; Selection_ID (none) -> SEL-c959c71ed77c; Selection_Ratings (none) -> {}; Selection_Source_URLs (none) -> https://www.st.com/en/search.html#q=STGB18N40LZT4
- R5440, R5442, R5444: Hardware_Qualification (none) -> BOARD_QUALIFICATION_PENDING; MPN (none) -> CRCW0603100KFKEA; Manufacturer (none) -> Vishay; Procurement_Status (none) -> SELECTED_FAMILY_CODE; Purchase_Released (none) -> false; Selection_Gaps (none) -> []; Selection_ID (none) -> SEL-4e3f06cba0aa; Selection_Ratings (none) -> {"aec_q200": true, "derating": "Use manufacturer power vers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; Selection_Source_URLs (none) -> https://www.vishay.com/docs/20035/dcrcwe3.pdf
- R5441: Hardware_Qualification (none) -> BOARD_QUALIFICATION_PENDING; MPN (none) -> TNPW0603147KBEEA; Manufacturer (none) -> Vishay; Procurement_Status (none) -> SELECTED_CATALOG_ITEM; Purchase_Released (none) -> false; Selection_Gaps (none) -> []; Selection_ID (none) -> SEL-b441cf204a6c; Selection_Ratings (none) -> {"aec_q200": true, "derating": "Use manufacturer power vers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; Selection_Source_URLs (none) -> https://www.digikey.com/en/products/detail/vishay-dale/TNPW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
- R5443: Hardware_Qualification (none) -> BOARD_QUALIFICATION_PENDING; MPN (none) -> CRCW060339K2FKEA; Manufacturer (none) -> Vishay; Procurement_Status (none) -> SELECTED_FAMILY_CODE; Purchase_Released (none) -> false; Selection_Gaps (none) -> []; Selection_ID (none) -> SEL-143cf3436985; Selection_Ratings (none) -> {"aec_q200": true, "derating": "Use manufacturer power vers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; Selection_Source_URLs (none) -> https://www.vishay.com/docs/20035/dcrcwe3.pdf
- R5445: Hardware_Qualification (none) -> BOARD_QUALIFICATION_PENDING; MPN (none) -> CRCW060310R0FKEA; Manufacturer (none) -> Vishay; Procurement_Status (none) -> SELECTED_FAMILY_CODE; Purchase_Released (none) -> false; Selection_Gaps (none) -> []; Selection_ID (none) -> SEL-887dce68fe1a; Selection_Ratings (none) -> {"aec_q200": true, "derating": "Use manufacturer power vers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; Selection_Source_URLs (none) -> https://www.vishay.com/docs/20035/dcrcwe3.pdf
- R5446: Hardware_Qualification (none) -> BOARD_QUALIFICATION_PENDING; MPN (none) -> CRCW060310K0FKEA; Manufacturer (none) -> Vishay; Procurement_Status (none) -> SELECTED_FAMILY_CODE; Purchase_Released (none) -> false; Selection_Gaps (none) -> []; Selection_ID (none) -> SEL-9c0806476875; Selection_Ratings (none) -> {"aec_q200": true, "derating": "Use manufacturer power vers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; Selection_Source_URLs (none) -> https://www.vishay.com/docs/20035/dcrcwe3.pdf
- R5447: Hardware_Qualification (none) -> PULSE_AND_KELVIN_LAYOUT_REVIEW_REQUIRED; MPN (none) -> WSLP2512R0100FEA; Manufacturer (none) -> Vishay; Procurement_Status (none) -> SELECTED_CONDITIONAL; Purchase_Released (none) -> false; Selection_Gaps (none) -> ["Repetitive pulse current, board heat flow and Kelvin rout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; Selection_ID (none) -> SEL-68c1815d8348; Selection_Ratings (none) -> {"derating": "Use manufacturer power versus ambient/termina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; Selection_Source_URLs (none) -> https://www.vishay.com/docs/30122/wslp.pdf
- R5448: Hardware_Qualification (none) -> BOARD_QUALIFICATION_PENDING; MPN (none) -> RNCF0603BTE4K99; Manufacturer (none) -> Stackpole Electronics; Procurement_Status (none) -> SELECTED_CATALOG_ITEM; Purchase_Released (none) -> false; Selection_Gaps (none) -> []; Selection_ID (none) -> SEL-d864a6215486; Selection_Ratings (none) -> {"aec_q200": true, "derating": "Use manufacturer power vers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; Selection_Source_URLs (none) -> https://www.digikey.com/en/products/detail/stackpole-electr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
- U5440: Hardware_Qualification (none) -> PINOUT_RATINGS_AND_DELIVERY_SUFFIX_REVIEW_PENDING; MPN (none) -> LTC6993HS6-1#WTRPBF; Manufacturer (none) -> Analog Devices; Procurement_Status (none) -> REFERENCE_MPN_RETAINED; Purchase_Released (none) -> false; Selection_Gaps (none) -> ["Existing schematic MPN retained. Complete circuit rating/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; Selection_ID (none) -> SEL-6e38c27363ea; Selection_Ratings (none) -> {}; Selection_Source_URLs (none) -> https://www.analog.com/en/search.html?q=LTC6993HS6-1#WTRPBF
- U5441: Hardware_Qualification (none) -> PINOUT_RATINGS_AND_DELIVERY_SUFFIX_REVIEW_PENDING; MPN (none) -> SN74LVC1G11BDCKRQ1; Manufacturer (none) -> Texas Instruments; Procurement_Status (none) -> REFERENCE_MPN_RETAINED; Purchase_Released (none) -> false; Selection_Gaps (none) -> ["Existing schematic MPN retained. Complete circuit rating/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; Selection_ID (none) -> SEL-af3da1e13ada; Selection_Ratings (none) -> {}; Selection_Source_URLs (none) -> https://www.ti.com/product/SN74LVC1G11B-Q1/part-details/SN7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
- U5442: Hardware_Qualification (none) -> BOARD_STRESS_AND_LAYOUT_REVIEW_REQUIRED; MPN (none) -> INA300AQDGSRQ1; Manufacturer (none) -> Texas Instruments; Procurement_Status (none) -> SELECTED_CONDITIONAL; Purchase_Released (none) -> false; Selection_Gaps (none) -> ["Catalog family limits verified; exact order suffix and ci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; Selection_ID (none) -> SEL-a097ea37f99e; Selection_Ratings (none) -> {"common_mode_max_v": 36, "common_mode_min_v": 0, "response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; Selection_Source_URLs (none) -> https://www.ti.com/product/INA300-Q1
