File: Power8GDI/hardware/design/interfaces/comms2.kicad_sch (KiCad schematic)
At the start: 16 parts, among them U1501 TCAN1042HGVDRQ1, U1502 TLIN1029ADRQ1

Commit message: Integrate protected GDI and CAN wideband nodes with Huge channel allocation
Parts:
- C1505: value 220p 100V C0G -> 1n 100V C0G; Design note (none) -> Commander bus capacitance; verify total cable/node capacita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
- D1502: value BAS21,215 DNP -> BAS21,215; Design note Optional commander pullup; anode toward VSUP. Both D1502/R1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 -> Commander assembly: anode toward VSUP. Remove BOTH D1502/R1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; now fitted
- R1507: value 1k DNP -> 1k 1% 0.5W; footprint Resistor_SMD:R_0603_1608Metric -> Resistor_SMD:R_1206_3216Metric; Design note (none) -> 0.256W upper bound at16V dominant; voltage/pulse derating r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; now fitted
Other:
- note added: "CAN2 default standby; LIN2 commander assembly, default sleep. MCU enables and schedules bus. Only one commander pullup per LIN bus. Remove BOTH D1502/R1507 for responder-only assembly. CAN2 uses PB5/PB6; SENT3 uses PE11 pad74. Shared timer, CAN filters and firmware remain pending. No automotive pulse/ESD/EMC or fault qualification is implied by this candidate."
- note removed: "CAN2 default standby; LIN2 default responder/sleep. MCU control required. Fit CAN termination only for an end node; fit BOTH commander parts only for a reviewed LIN commander. CAN2 uses PB5/PB6; SENT3 moves to PE11 pad74. Shared timer, CAN filters and firmware remain pending. No automotive pulse/ESD/EMC or fault qualification is implied by this candidate."
Changed lines of the file:
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@@
 (wire (pts (xy 500.38 228.6) (xy 500.38 236.22)) (stroke (width 0) (type default)))
 (global_label "GND" (shape bidirectional) (at 500.38 236.22 90) (effects (font (size 1.016 1.016)) (justify right bottom)))
-(symbol (lib_id "Power8GDI_Core:C") (at 444.5 224.79 0) (unit 1) (in_bom yes) (on_board yes) (dnp no) (property "Reference" "C1505" (at 448.5 223.52 0) (effects (font (size 1.27 1.27)) (justify left))) (property "Value" "220p 100V C0G" (at 448.5 226.06 0) (effects (font (size 1.27 1.27)) (justify left))) (property "Footprint" "Capacitor_SMD:C_0603_1608Metric" (at 444.5 224.79 0) (effects (font (size 1.27 1.27)) (hide yes))) (property "Design note" "" (at 444.5 224.79 0) (effects (font (size 1.27 1.27)) (hide yes))) (pin "1") (pin "2") (instances (project "Power8GDI_Core" (path "/f4d21065-0a5b-5086-a08e-1af9469f04bd/aef4a5ed-16a9-5635-82f1-5a0caf432873" (reference "C1505") (unit 1)))))
+(symbol (lib_id "Power8GDI_Core:C") (at 444.5 224.79 0) (unit 1) (in_bom yes) (on_board yes) (dnp no) (property "Reference" "C1505" (at 448.5 223.52 0) (effects (font (size 1.27 1.27)) (justify left))) (property "Value" "1n 100V C0G" (at 448.5 226.06 0) (effects (font (size 1.27 1.27)) (justify left))) (property "Footprint" "Capacitor_SMD:C_0603_1608Metric" (at 444.5 224.79 0) (effects (font (size 1.27 1.27)) (hide yes))) (property "Design note" "Commander bus capacitance; verify total cable/node capacitance" (at 444.5 224.79 0) (effects (font (size 1.27 1.27)) (hide yes))) (pin "1") (pin "2") (instances (project "Power8GDI_Core" (path "/f4d21065-0a5b-5086-a08e-1af9469f04bd/aef4a5ed-16a9-5635-82f1-5a0caf432873" (reference "C1505") (unit 1)))))
 (wire (pts (xy 444.5 220.98) (xy 444.5 213.36)) (stroke (width 0) (type default)))
 (global_label "LIN2_BUS" (shape bidirectional) (at 444.5 213.36 270) (effects (font (size 1.016 1.016)) (justify left bottom)))
 (wire (pts (xy 444.5 228.6) (xy 444.5 236.22)) (stroke (width 0) (type default)))
 (global_label "GND" (shape bidirectional) (at 444.5 236.22 90) (effects (font (size 1.016 1.016)) (justify right bottom)))
-(symbol (lib_id "Power8GDI_Core:Interface_BAS21") (at 355.6 229.87 0) (unit 1) (in_bom yes) (on_board yes) (dnp yes) (property "Reference" "D1502" (at 355.6 217.17 0) (effects (font (size 1.27 1.27)))) (property "Value" "BAS21,215 DNP" (at 375.92 242.57 0) (effects (font (size 1.27 1.27)) (justify left))) (property "Footprint" "Package_TO_SOT_SMD:SOT-23" (at 355.6 229.87 0) (effects (font (size 1.27 1.27)) (hide yes))) (property "Design note" "Optional commander pullup; anode toward VSUP. Both D1502/R1507 DNP in responder mode" (at 355.6 229.87 0) (effects (font (size 1.27 1.27)) (hide yes))) (pin "1") (pin "3") (pin "2") (instances (project "Power8GDI_Core" (path "/f4d21065-0a5b-5086-a08e-1af9469f04bd/aef4a5ed-16a9-5635-82f1-5a0caf432873" (reference "D1502") (unit 1)))))
+(symbol (lib_id "Power8GDI_Core:Interface_BAS21") (at 355.6 229.87 0) (unit 1) (in_bom yes) (on_board yes) (dnp no) (property "Reference" "D1502" (at 355.6 217.17 0) (effects (font (size 1.27 1.27)))) (property "Value" "BAS21,215" (at 375.92 242.57 0) (effects (font (size 1.27 1.27)) (justify left))) (property "Footprint" "Package_TO_SOT_SMD:SOT-23" (at 355.6 229.87 0) (effects (font (size 1.27 1.27)) (hide yes))) (property "Design note" "Commander assembly: anode toward VSUP. Remove BOTH D1502/R1507 for responder-only harness topology" (at 355.6 229.87 0) (effects (font (size 1.27 1.27)) (hide yes))) (pin "1") (pin "3") (pin "2") (instances (project "Power8GDI_Core" (path "/f4d21065-0a5b-5086-a08e-1af9469f04bd/aef4a5ed-16a9-5635-82f1-5a0caf432873" (reference "D1502") (unit 1)))))
 (wire (pts (xy 345.44 229.87) (xy 337.82 229.87)) (stroke (width 0) (type default)))
 (global_label "LIN2_VSUP" (shape bidirectional) (at 337.82 229.87 0) (effects (font (size 1.016 1.016)) (justify right bottom)))
@@
 (global_label "LIN2_COMMANDER_DIODE" (shape bidirectional) (at 373.38 229.87 180) (effects (font (size 1.016 1.016)) (justify left bottom)))
 (no_connect (at 355.6 240.03))
-(symbol (lib_id "Power8GDI_Core:R") (at 355.6 284.48 0) (unit 1) (in_bom yes) (on_board yes) (dnp yes) (property "Reference" "R1507" (at 359.6 283.21 0) (effects (font (size 1.27 1.27)) (justify left))) (property "Value" "1k DNP" (at 359.6 285.75 0) (effects (font (size 1.27 1.27)) (justify left))) (property "Footprint" "Resistor_SMD:R_0603_1608Metric" (at 355.6 284.48 0) (effects (font (size 1.27 1.27)) (hide yes))) (property "Design note" "" (at 355.6 284.48 0) (effects (font (size 1.27 1.27)) (hide yes))) (pin "1") (pin "2") (instances (project "Power8GDI_Core" (path "/f4d21065-0a5b-5086-a08e-1af9469f04bd/aef4a5ed-16a9-5635-82f1-5a0caf432873" (reference "R1507") (unit 1)))))
+(symbol (lib_id "Power8GDI_Core:R") (at 355.6 284.48 0) (unit 1) (in_bom yes) (on_board yes) (dnp no) (property "Reference" "R1507" (at 359.6 283.21 0) (effects (font (size 1.27 1.27)) (justify left))) (property "Value" "1k 1% 0.5W" (at 359.6 285.75 0) (effects (font (size 1.27 1.27)) (justify left))) (property "Footprint" "Resistor_SMD:R_1206_3216Metric" (at 355.6 284.48 0) (effects (font (size 1.27 1.27)) (hide yes))) (property "Design note" "0.256W upper bound at16V dominant; voltage/pulse derating remains required" (at 355.6 284.48 0) (effects (font (size 1.27 1.27)) (hide yes))) (pin "1") (pin "2") (instances (project "Power8GDI_Core" (path "/f4d21065-0a5b-5086-a08e-1af9469f04bd/aef4a5ed-16a9-5635-82f1-5a0caf432873" (reference "R1507") (unit 1)))))
 (wire (pts (xy 355.6 280.67) (xy 355.6 273.05)) (stroke (width 0) (type default)))
 (global_label "LIN2_COMMANDER_DIODE" (shape bidirectional) (at 355.6 273.05 270) (effects (font (size 1.016 1.016)) (justify left bottom)))
 (wire (pts (xy 355.6 288.29) (xy 355.6 295.91)) (stroke (width 0) (type default)))
 (global_label "LIN2_BUS" (shape bidirectional) (at 355.6 295.91 90) (effects (font (size 1.016 1.016)) (justify right bottom)))
-(text "CAN2 default standby; LIN2 default responder/sleep. MCU control required.\nFit CAN termination only for an end node; fit BOTH commander parts only for a reviewed LIN commander.\nCAN2 uses PB5/PB6; SENT3 moves to PE11 pad74. Shared timer, CAN filters and firmware remain pending.\nNo automotive pulse/ESD/EMC or fault qualification is implied by this candidate." (at 25.4 335 0) (effects (font (size 1.27 1.27)) (justify left top)))
+(text "CAN2 default standby; LIN2 commander assembly, default sleep. MCU enables and schedules bus.\nOnly one commander pullup per LIN bus. Remove BOTH D1502/R1507 for responder-only assembly.\nCAN2 uses PB5/PB6; SENT3 uses PE11 pad74. Shared timer, CAN filters and firmware remain pending.\nNo automotive pulse/ESD/EMC or fault qualification is implied by this candidate." (at 25.4 335 0) (effects (font (size 1.27 1.27)) (justify left top)))
 (sheet_instances (path "/" (page "1"))))

Commit message: Review B58 injector power stage and bind selected GDI6 BOM
Parts:
- C1501, C1502, C1503: Hardware_Qualification (none) -> BOARD_QUALIFICATION_PENDING; MPN (none) -> C0603C104K5RACTU; Manufacturer (none) -> KEMET; Procurement_Status (none) -> SELECTED_CATALOG_ITEM; Purchase_Released (none) -> false; Selection_Gaps (none) -> []; Selection_ID (none) -> SEL-6bf9727c4e40; Selection_Ratings (none) -> {"capacitance_pf": 100000, "dielectric": "X7R", "rated_volt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; Selection_Source_URLs (none) -> https://search.kemet.com/download/specsheet/C0603C104K5RACTU
- C1504: Hardware_Qualification (none) -> BOARD_QUALIFICATION_PENDING; MPN (none) -> C0805C105K5RACTU; Manufacturer (none) -> KEMET; Procurement_Status (none) -> SELECTED_CATALOG_ITEM; Purchase_Released (none) -> false; Selection_Gaps (none) -> []; Selection_ID (none) -> SEL-838906dbfe60; Selection_Ratings (none) -> {"capacitance_pf": 1000000, "dc_bias_qualification": "PENDI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; Selection_Source_URLs (none) -> https://search.kemet.com/component-documentation/download/s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
- C1505: Hardware_Qualification (none) -> BOARD_QUALIFICATION_PENDING; MPN (none) -> C0603C102J1GACTU; Manufacturer (none) -> KEMET; Procurement_Status (none) -> SELECTED_CATALOG_ITEM; Purchase_Released (none) -> false; Selection_Gaps (none) -> []; Selection_ID (none) -> SEL-ec742f39ec1f; Selection_Ratings (none) -> {"capacitance_pf": 1000, "dielectric": "C0G", "rated_voltag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; Selection_Source_URLs (none) -> https://search.kemet.com/download/specsheet/C0603C102J1GACTU
- D1501: Hardware_Qualification (none) -> PINOUT_RATINGS_AND_DELIVERY_SUFFIX_REVIEW_PENDING; MPN (none) -> PESD2CAN,215; Manufacturer (none) -> Nexperia; Procurement_Status (none) -> REFERENCE_MPN_RETAINED; Purchase_Released (none) -> false; Selection_Gaps (none) -> ["Existing schematic MPN retained. Complete circuit rating/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; Selection_ID (none) -> SEL-397878b612f9; Selection_Ratings (none) -> {}; Selection_Source_URLs (none) -> https://www.nexperia.com/product/PESD2CAN
- D1502: Hardware_Qualification (none) -> PINOUT_RATINGS_AND_DELIVERY_SUFFIX_REVIEW_PENDING; MPN (none) -> BAS21,215; Manufacturer (none) -> Nexperia; Procurement_Status (none) -> REFERENCE_MPN_RETAINED; Purchase_Released (none) -> false; Selection_Gaps (none) -> ["Existing schematic MPN retained. Complete circuit rating/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; Selection_ID (none) -> SEL-3ac3f96db10b; Selection_Ratings (none) -> {}; Selection_Source_URLs (none) -> https://www.nexperia.com/product/BAS21
- R1501, R1504, R1505: Hardware_Qualification (none) -> BOARD_QUALIFICATION_PENDING; MPN (none) -> CRCW060310K0FKEA; Manufacturer (none) -> Vishay; Procurement_Status (none) -> SELECTED_FAMILY_CODE; Purchase_Released (none) -> false; Selection_Gaps (none) -> []; Selection_ID (none) -> SEL-9c0806476875; Selection_Ratings (none) -> {"aec_q200": true, "derating": "Use manufacturer power vers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; Selection_Source_URLs (none) -> https://www.vishay.com/docs/20035/dcrcwe3.pdf
- R1503: Hardware_Qualification (none) -> BOARD_QUALIFICATION_PENDING; MPN (none) -> CRCW06034K70FKEA; Manufacturer (none) -> Vishay; Procurement_Status (none) -> SELECTED_FAMILY_CODE; Purchase_Released (none) -> false; Selection_Gaps (none) -> []; Selection_ID (none) -> SEL-1f010ac9622d; Selection_Ratings (none) -> {"aec_q200": true, "derating": "Use manufacturer power vers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; Selection_Source_URLs (none) -> https://www.vishay.com/docs/20035/dcrcwe3.pdf
- R1506: Hardware_Qualification (none) -> BOARD_QUALIFICATION_PENDING; MPN (none) -> CRCW06030000Z0EA; Manufacturer (none) -> Vishay; Procurement_Status (none) -> SELECTED_FAMILY_CODE; Purchase_Released (none) -> false; Selection_Gaps (none) -> []; Selection_ID (none) -> SEL-8473f02313b2; Selection_Ratings (none) -> {"aec_q200": true, "current_a": 2, "power_reference_tempera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; Selection_Source_URLs (none) -> https://www.vishay.com/docs/20035/dcrcwe3.pdf
- R1507: Hardware_Qualification (none) -> BOARD_QUALIFICATION_PENDING; MPN (none) -> CRCW12061K00FKEAHP; Manufacturer (none) -> Vishay; Procurement_Status (none) -> SELECTED_CATALOG_ITEM; Purchase_Released (none) -> false; Selection_Gaps (none) -> []; Selection_ID (none) -> SEL-515f600e0ec3; Selection_Ratings (none) -> {"aec_q200": true, "derating": "Use manufacturer power vers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; Selection_Source_URLs (none) -> https://www.vishay.com/docs/20043/crcwhpe3.pdf https://www.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
- U1501: Hardware_Qualification (none) -> PINOUT_RATINGS_AND_DELIVERY_SUFFIX_REVIEW_PENDING; MPN (none) -> TCAN1042HGVDRQ1; Manufacturer (none) -> Texas Instruments; Procurement_Status (none) -> REFERENCE_MPN_RETAINED; Purchase_Released (none) -> false; Selection_Gaps (none) -> ["Existing schematic MPN retained. Complete circuit rating/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; Selection_ID (none) -> SEL-c86778911c36; Selection_Ratings (none) -> {}; Selection_Source_URLs (none) -> https://www.ti.com/product/TCAN1042H-Q1/part-details/TCAN10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
- U1502: Hardware_Qualification (none) -> PINOUT_RATINGS_AND_DELIVERY_SUFFIX_REVIEW_PENDING; MPN (none) -> TLIN1029ADRQ1; Manufacturer (none) -> Texas Instruments; Procurement_Status (none) -> REFERENCE_MPN_RETAINED; Purchase_Released (none) -> false; Selection_Gaps (none) -> ["Existing schematic MPN retained. Complete circuit rating/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; Selection_ID (none) -> SEL-d38cf124d61a; Selection_Ratings (none) -> {}; Selection_Source_URLs (none) -> https://www.ti.com/product/TLIN1029A-Q1/part-details/TLIN10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
