File: Power8GDI/hardware/design/interfaces/sd_spi.kicad_sch (KiCad schematic)
At the start: 15 parts, among them J1502 Molex 1040310811

Commit message: Review B58 injector power stage and bind selected GDI6 BOM
Parts:
- C1520: Hardware_Qualification (none) -> BOARD_QUALIFICATION_PENDING; MPN (none) -> C0603C104K5RACTU; Manufacturer (none) -> KEMET; Procurement_Status (none) -> SELECTED_CATALOG_ITEM; Purchase_Released (none) -> false; Selection_Gaps (none) -> []; Selection_ID (none) -> SEL-6bf9727c4e40; Selection_Ratings (none) -> {"capacitance_pf": 100000, "dielectric": "X7R", "rated_volt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; Selection_Source_URLs (none) -> https://search.kemet.com/download/specsheet/C0603C104K5RACTU
- C1521: Hardware_Qualification (none) -> BOARD_QUALIFICATION_PENDING; MPN (none) -> GMC21X7R106K25NT; Manufacturer (none) -> Cal-Chip Electronics; Procurement_Status (none) -> SELECTED_CATALOG_ITEM; Purchase_Released (none) -> false; Selection_Gaps (none) -> []; Selection_ID (none) -> SEL-1f2219112d7d; Selection_Ratings (none) -> {"capacitance_pf": 10000000, "dc_bias_qualification": "PEND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; Selection_Source_URLs (none) -> https://www.digikey.com/en/products/detail/cal-chip-electro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
- C1522: Hardware_Qualification (none) -> BOARD_QUALIFICATION_PENDING; MPN (none) -> C0603C102K5RACTU; Manufacturer (none) -> KEMET; Procurement_Status (none) -> SELECTED_CATALOG_ITEM; Purchase_Released (none) -> false; Selection_Gaps (none) -> []; Selection_ID (none) -> SEL-84498dfd21b1; Selection_Ratings (none) -> {"capacitance_pf": 1000, "dielectric": "X7R", "rated_voltag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; Selection_Source_URLs (none) -> https://www.digikey.com/en/products/detail/kemet/C0603C102K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
- D1520, D1521: Hardware_Qualification (none) -> PINOUT_RATINGS_AND_DELIVERY_SUFFIX_REVIEW_PENDING; MPN (none) -> USBLC6-2SC6; Manufacturer (none) -> STMicroelectronics; Procurement_Status (none) -> REFERENCE_MPN_RETAINED; Purchase_Released (none) -> false; Selection_Gaps (none) -> ["Existing schematic MPN retained. Complete circuit rating/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; Selection_ID (none) -> SEL-ceeac0a83c9b; Selection_Ratings (none) -> {}; Selection_Source_URLs (none) -> https://www.st.com/en/search.html#q=USBLC6-2SC6
- J1502: Hardware_Qualification (none) -> PINOUT_RATINGS_AND_DELIVERY_SUFFIX_REVIEW_PENDING; MPN (none) -> 1040310811; Manufacturer (none) -> Molex; Procurement_Status (none) -> REFERENCE_MPN_RETAINED; Purchase_Released (none) -> false; Selection_Gaps (none) -> ["Existing schematic MPN retained. Complete circuit rating/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; Selection_ID (none) -> SEL-7925eaf8b85b; Selection_Ratings (none) -> {}; Selection_Source_URLs (none) -> https://www.molex.com/en-us/products/part-detail/1040310811
- R1520: Hardware_Qualification (none) -> BOARD_QUALIFICATION_PENDING; MPN (none) -> CRCW06030000Z0EA; Manufacturer (none) -> Vishay; Procurement_Status (none) -> SELECTED_FAMILY_CODE; Purchase_Released (none) -> false; Selection_Gaps (none) -> []; Selection_ID (none) -> SEL-8473f02313b2; Selection_Ratings (none) -> {"aec_q200": true, "current_a": 2, "power_reference_tempera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; Selection_Source_URLs (none) -> https://www.vishay.com/docs/20035/dcrcwe3.pdf
- R1521, R1522: Hardware_Qualification (none) -> BOARD_QUALIFICATION_PENDING; MPN (none) -> CRCW060322R0FKEA; Manufacturer (none) -> Vishay; Procurement_Status (none) -> SELECTED_FAMILY_CODE; Purchase_Released (none) -> false; Selection_Gaps (none) -> []; Selection_ID (none) -> SEL-829683b28581; Selection_Ratings (none) -> {"aec_q200": true, "derating": "Use manufacturer power vers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; Selection_Source_URLs (none) -> https://www.vishay.com/docs/20035/dcrcwe3.pdf
- R1523, R1524, R1525, R1526, R1527, R1528: Hardware_Qualification (none) -> BOARD_QUALIFICATION_PENDING; MPN (none) -> CRCW060347K0FKEA; Manufacturer (none) -> Vishay; Procurement_Status (none) -> SELECTED_FAMILY_CODE; Purchase_Released (none) -> false; Selection_Gaps (none) -> []; Selection_ID (none) -> SEL-8ba99d730f8b; Selection_Ratings (none) -> {"aec_q200": true, "derating": "Use manufacturer power vers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; Selection_Source_URLs (none) -> https://www.vishay.com/docs/20035/dcrcwe3.pdf
