File: Power8GDI/hardware/design/interfaces/sensor_power.kicad_sch (KiCad schematic)
At the start: 17 parts, among them U1530 TPS7B4253QDDARQ1, U1531 TPS7B4253QDDARQ1

Commit message: Review B58 injector power stage and bind selected GDI6 BOM
Parts:
- C1530, C1535: Hardware_Qualification (none) -> BOARD_QUALIFICATION_PENDING; MPN (none) -> C0805C105K5RACTU; Manufacturer (none) -> KEMET; Procurement_Status (none) -> SELECTED_CATALOG_ITEM; Purchase_Released (none) -> false; Selection_Gaps (none) -> []; Selection_ID (none) -> SEL-838906dbfe60; Selection_Ratings (none) -> {"capacitance_pf": 1000000, "dc_bias_qualification": "PENDI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; Selection_Source_URLs (none) -> https://search.kemet.com/component-documentation/download/s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
- C1531, C1532, C1534, C1536, C1537, C1539: Hardware_Qualification (none) -> BOARD_QUALIFICATION_PENDING; MPN (none) -> C0603C104K5RACTU; Manufacturer (none) -> KEMET; Procurement_Status (none) -> SELECTED_CATALOG_ITEM; Purchase_Released (none) -> false; Selection_Gaps (none) -> []; Selection_ID (none) -> SEL-6bf9727c4e40; Selection_Ratings (none) -> {"capacitance_pf": 100000, "dielectric": "X7R", "rated_volt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; Selection_Source_URLs (none) -> https://search.kemet.com/download/specsheet/C0603C104K5RACTU
- C1533, C1538: footprint Capacitor_SMD:C_1210_3225Metric -> Power8GDI_Interfaces:CGA9P3_2220; Design note Require effective >=10uF at voltage/temp/tolerance, ESR1moh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 -> CGA9P3X7R1H226M250KB candidate; effective >=10uF and ESR1mo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; Hardware_Qualification (none) -> LAND_PATTERN_AND_EFFECTIVE_CAPACITANCE_REVIEW_REQUIRED; MPN (none) -> CGA9P3X7R1H226M250KB; Manufacturer (none) -> TDK; Procurement_Status (none) -> SELECTED_CONDITIONAL; Purchase_Released (none) -> false; Selection_Gaps (none) -> ["Source1210 footprint must become2220. Typical manufacture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; Selection_ID (none) -> SEL-09e313605b32; Selection_Ratings (none) -> {"aec_q200": true, "capacitance_pf": 22000000, "dc_bias_qua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; Selection_Source_URLs (none) -> https://product.tdk.com/en/search/capacitor/ceramic/mlcc/in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
- D1530, D1531: Hardware_Qualification (none) -> PINOUT_RATINGS_AND_DELIVERY_SUFFIX_REVIEW_PENDING; MPN (none) -> STPS2H100UY; Manufacturer (none) -> STMicroelectronics; Procurement_Status (none) -> REFERENCE_MPN_RETAINED; Purchase_Released (none) -> false; Selection_Gaps (none) -> ["Existing schematic MPN retained. Complete circuit rating/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; Selection_ID (none) -> SEL-2af9fd635e9e; Selection_Ratings (none) -> {}; Selection_Source_URLs (none) -> https://www.st.com/en/search.html#q=STPS2H100UY
- R1530, R1531, R1532: Hardware_Qualification (none) -> BOARD_QUALIFICATION_PENDING; MPN (none) -> CRCW08050000Z0EA; Manufacturer (none) -> Vishay; Procurement_Status (none) -> SELECTED_FAMILY_CODE; Purchase_Released (none) -> false; Selection_Gaps (none) -> []; Selection_ID (none) -> SEL-49a75d3b142a; Selection_Ratings (none) -> {"aec_q200": true, "current_a": 2.5, "power_reference_tempe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; Selection_Source_URLs (none) -> https://www.vishay.com/docs/20035/dcrcwe3.pdf
- U1530, U1531: Hardware_Qualification (none) -> PINOUT_RATINGS_AND_DELIVERY_SUFFIX_REVIEW_PENDING; MPN (none) -> TPS7B4253QDDARQ1; Manufacturer (none) -> Texas Instruments; Procurement_Status (none) -> REFERENCE_MPN_RETAINED; Purchase_Released (none) -> false; Selection_Gaps (none) -> ["Existing schematic MPN retained. Complete circuit rating/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; Selection_ID (none) -> SEL-009e4917c633; Selection_Ratings (none) -> {}; Selection_Source_URLs (none) -> https://www.ti.com/product/TPS7B4253-Q1/part-details/TPS7B4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
