File: Power8GDI/hardware/design/io/analog_1.kicad_sch (KiCad schematic)
At the start: 27 parts, among them U701 TLV9004QPWRQ1

Commit message: Review B58 injector power stage and bind selected GDI6 BOM
Parts:
- C700, C702, C704, C706: Hardware_Qualification (none) -> BOARD_QUALIFICATION_PENDING; MPN (none) -> C0603C102J1GACTU; Manufacturer (none) -> KEMET; Procurement_Status (none) -> SELECTED_CATALOG_ITEM; Purchase_Released (none) -> false; Selection_Gaps (none) -> []; Selection_ID (none) -> SEL-ec742f39ec1f; Selection_Ratings (none) -> {"capacitance_pf": 1000, "dielectric": "C0G", "rated_voltag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; Selection_Source_URLs (none) -> https://search.kemet.com/download/specsheet/C0603C102J1GACTU
- C701, C703, C705, C707: Hardware_Qualification (none) -> BOARD_QUALIFICATION_PENDING; MPN (none) -> C0603C103K5RACTU; Manufacturer (none) -> KEMET; Procurement_Status (none) -> SELECTED_CATALOG_ITEM; Purchase_Released (none) -> false; Selection_Gaps (none) -> []; Selection_ID (none) -> SEL-003cf16db818; Selection_Ratings (none) -> {"capacitance_pf": 10000, "dielectric": "X7R", "rated_volta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; Selection_Source_URLs (none) -> https://www.digikey.com/en/products/detail/kemet/C0603C103K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
- C740: Hardware_Qualification (none) -> BOARD_QUALIFICATION_PENDING; MPN (none) -> C0603C104K5RACTU; Manufacturer (none) -> KEMET; Procurement_Status (none) -> SELECTED_CATALOG_ITEM; Purchase_Released (none) -> false; Selection_Gaps (none) -> []; Selection_ID (none) -> SEL-6bf9727c4e40; Selection_Ratings (none) -> {"capacitance_pf": 100000, "dielectric": "X7R", "rated_volt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; Selection_Source_URLs (none) -> https://search.kemet.com/download/specsheet/C0603C104K5RACTU
- C741: Hardware_Qualification (none) -> BOARD_QUALIFICATION_PENDING; MPN (none) -> C0603C105K3RACTU; Manufacturer (none) -> KEMET; Procurement_Status (none) -> SELECTED_CATALOG_ITEM; Purchase_Released (none) -> false; Selection_Gaps (none) -> []; Selection_ID (none) -> SEL-4bca20b134b8; Selection_Ratings (none) -> {"capacitance_pf": 1000000, "dc_bias_qualification": "PENDI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; Selection_Source_URLs (none) -> https://search.kemet.com/download/specsheet/C0603C105K3RACTU
- D701, D702, D703, D704: Hardware_Qualification (none) -> PINOUT_RATINGS_AND_DELIVERY_SUFFIX_REVIEW_PENDING; MPN (none) -> BAT54S,215; Manufacturer (none) -> Nexperia; Procurement_Status (none) -> REFERENCE_MPN_RETAINED; Purchase_Released (none) -> false; Selection_Gaps (none) -> ["Existing schematic MPN retained. Complete circuit rating/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; Selection_ID (none) -> SEL-b62e273620d3; Selection_Ratings (none) -> {}; Selection_Source_URLs (none) -> https://www.nexperia.com/product/BAT54S
- R700, R701, R703, R704, R706, R707, R709, R710: Hardware_Qualification (none) -> BOARD_QUALIFICATION_PENDING; MPN (none) -> RNCF0603BTE100K; Manufacturer (none) -> Stackpole Electronics; Procurement_Status (none) -> SELECTED_CATALOG_ITEM; Purchase_Released (none) -> false; Selection_Gaps (none) -> []; Selection_ID (none) -> SEL-c5cdfb61a2a3; Selection_Ratings (none) -> {"aec_q200": true, "derating": "Use manufacturer power vers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; Selection_Source_URLs (none) -> https://www.digikey.com/en/products/detail/stackpole-electr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
- R702, R705, R708, R711: Hardware_Qualification (none) -> BOARD_QUALIFICATION_PENDING; MPN (none) -> CRCW06031K00FKEA; Manufacturer (none) -> Vishay; Procurement_Status (none) -> SELECTED_FAMILY_CODE; Purchase_Released (none) -> false; Selection_Gaps (none) -> []; Selection_ID (none) -> SEL-38197231a947; Selection_Ratings (none) -> {"aec_q200": true, "derating": "Use manufacturer power vers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; Selection_Source_URLs (none) -> https://www.vishay.com/docs/20035/dcrcwe3.pdf
- U701: Hardware_Qualification (none) -> PINOUT_RATINGS_AND_DELIVERY_SUFFIX_REVIEW_PENDING; MPN (none) -> TLV9004QPWRQ1; Manufacturer (none) -> Texas Instruments; Procurement_Status (none) -> REFERENCE_MPN_RETAINED; Purchase_Released (none) -> false; Selection_Gaps (none) -> ["Existing schematic MPN retained. Complete circuit rating/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; Selection_ID (none) -> SEL-75e8c7fc6566; Selection_Ratings (none) -> {}; Selection_Source_URLs (none) -> https://www.ti.com/product/TLV9004-Q1/part-details/TLV9004Q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
