File: Power8GDI/hardware/design/logic_power/logic_3v3.kicad_sch (KiCad schematic)
At the start: 10 parts, among them U5300 TPS62130AQRGTRQ1

Commit message: Review B58 injector power stage and bind selected GDI6 BOM
Parts:
- C5300: Hardware_Qualification (none) -> BOARD_QUALIFICATION_PENDING; MPN (none) -> GMC21X7R106K25NT; Manufacturer (none) -> Cal-Chip Electronics; Procurement_Status (none) -> SELECTED_CATALOG_ITEM; Purchase_Released (none) -> false; Selection_Gaps (none) -> ["Required effective capacitance not yet verified with supp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; Selection_ID (none) -> SEL-072e01fa6b90; Selection_Ratings (none) -> {"capacitance_pf": 10000000, "dc_bias_qualification": "PEND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; Selection_Source_URLs (none) -> https://www.digikey.com/en/products/detail/cal-chip-electro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
- C5301: Hardware_Qualification (none) -> BOARD_QUALIFICATION_PENDING; MPN (none) -> C0805C104K1RACTU; Manufacturer (none) -> KEMET; Procurement_Status (none) -> SELECTED_CATALOG_ITEM; Purchase_Released (none) -> false; Selection_Gaps (none) -> []; Selection_ID (none) -> SEL-50b208aec5b1; Selection_Ratings (none) -> {"capacitance_pf": 100000, "dielectric": "X7R", "rated_volt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; Selection_Source_URLs (none) -> https://www.mouser.com/datasheet/3/72/1/C0805C104K1RACTU.pdf
- C5302: Hardware_Qualification (none) -> BOARD_QUALIFICATION_PENDING; MPN (none) -> C1210C226K4RACTU; Manufacturer (none) -> KEMET; Procurement_Status (none) -> SELECTED_CATALOG_ITEM; Purchase_Released (none) -> false; Selection_Gaps (none) -> ["Required effective capacitance not yet verified with supp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; Selection_ID (none) -> SEL-402dd3bcb9f5; Selection_Ratings (none) -> {"capacitance_pf": 22000000, "dc_bias_qualification": "PEND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; Selection_Source_URLs (none) -> https://www.digikey.com/en/products/detail/kemet/C1210C226K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
- C5303: Hardware_Qualification (none) -> BOARD_QUALIFICATION_PENDING; MPN (none) -> C0805C332J5GACTU; Manufacturer (none) -> KEMET; Procurement_Status (none) -> SELECTED_CATALOG_ITEM; Purchase_Released (none) -> false; Selection_Gaps (none) -> []; Selection_ID (none) -> SEL-0d91b403f861; Selection_Ratings (none) -> {"capacitance_pf": 3300, "dielectric": "C0G", "rated_voltag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; Selection_Source_URLs (none) -> https://www.digikey.com/en/products/detail/kemet/C0805C332J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
- L5300: Hardware_Qualification (none) -> PINOUT_RATINGS_AND_DELIVERY_SUFFIX_REVIEW_PENDING; MPN (none) -> XAL5030-222MEC; Manufacturer (none) -> Coilcraft; Procurement_Status (none) -> REFERENCE_MPN_RETAINED; Purchase_Released (none) -> false; Selection_Gaps (none) -> ["Existing schematic MPN retained. Complete circuit rating/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; Selection_ID (none) -> SEL-4a14a5c9b81a; Selection_Ratings (none) -> {}; Selection_Source_URLs (none) -> https://www.coilcraft.com/en-us/products/power/shielded-ind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
- R5300: Hardware_Qualification (none) -> BOARD_QUALIFICATION_PENDING; MPN (none) -> RNCF0603BTE100K; Manufacturer (none) -> Stackpole Electronics; Procurement_Status (none) -> SELECTED_CATALOG_ITEM; Purchase_Released (none) -> false; Selection_Gaps (none) -> []; Selection_ID (none) -> SEL-c5cdfb61a2a3; Selection_Ratings (none) -> {"aec_q200": true, "derating": "Use manufacturer power vers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; Selection_Source_URLs (none) -> https://www.digikey.com/en/products/detail/stackpole-electr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
- R5301: Hardware_Qualification (none) -> BOARD_QUALIFICATION_PENDING; MPN (none) -> RNCF0603BTE32K0; Manufacturer (none) -> Stackpole Electronics; Procurement_Status (none) -> SELECTED_CATALOG_ITEM; Purchase_Released (none) -> false; Selection_Gaps (none) -> []; Selection_ID (none) -> SEL-fd24b7608546; Selection_Ratings (none) -> {"power_w": 0.167, "resistance_ohm": 32000, "tcr_ppm_c": 25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; Selection_Source_URLs (none) -> https://www.digikey.com/en/products/detail/stackpole-electr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
- R5302: Hardware_Qualification (none) -> BOARD_QUALIFICATION_PENDING; MPN (none) -> CRCW0603100KFKEA; Manufacturer (none) -> Vishay; Procurement_Status (none) -> SELECTED_FAMILY_CODE; Purchase_Released (none) -> false; Selection_Gaps (none) -> []; Selection_ID (none) -> SEL-4e3f06cba0aa; Selection_Ratings (none) -> {"aec_q200": true, "derating": "Use manufacturer power vers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; Selection_Source_URLs (none) -> https://www.vishay.com/docs/20035/dcrcwe3.pdf
- R5303: Hardware_Qualification (none) -> BOARD_QUALIFICATION_PENDING; MPN (none) -> CRCW060310K0FKEA; Manufacturer (none) -> Vishay; Procurement_Status (none) -> SELECTED_FAMILY_CODE; Purchase_Released (none) -> false; Selection_Gaps (none) -> []; Selection_ID (none) -> SEL-9c0806476875; Selection_Ratings (none) -> {"aec_q200": true, "derating": "Use manufacturer power vers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; Selection_Source_URLs (none) -> https://www.vishay.com/docs/20035/dcrcwe3.pdf
- U5300: Hardware_Qualification (none) -> BOARD_STRESS_AND_LAYOUT_REVIEW_REQUIRED; MPN (none) -> TPS62130AQRGTRQ1; Manufacturer (none) -> Texas Instruments; Procurement_Status (none) -> SELECTED_CONDITIONAL; Purchase_Released (none) -> false; Selection_Gaps (none) -> ["Catalog family limits verified; exact order suffix and ci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; Selection_ID (none) -> SEL-758eea3267d5; Selection_Ratings (none) -> {"output_current_catalog_a": 3, "output_max_v": 6, "supply_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; Selection_Source_URLs (none) -> https://www.ti.com/product/TPS62130A-Q1
