File: Power8GDI/hardware/design/logic_power/logic_5v.kicad_sch (KiCad schematic)
At the start: 22 parts, among them U5200 LM76003QRNPRQ1

Commit message: Review B58 injector power stage and bind selected GDI6 BOM
Parts:
- C5200: Hardware_Qualification (none) -> BOARD_QUALIFICATION_PENDING; MPN (none) -> C3225X7R2A106K250AC; Manufacturer (none) -> TDK; Procurement_Status (none) -> SELECTED_CATALOG_ITEM; Purchase_Released (none) -> false; Selection_Gaps (none) -> ["Required effective capacitance not yet verified with supp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; Selection_ID (none) -> SEL-0dd94486aade; Selection_Ratings (none) -> {"capacitance_pf": 10000000, "dc_bias_qualification": "PEND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; Selection_Source_URLs (none) -> https://www.digikey.com/en/products/detail/tdk/C3225X7R2A10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
- C5201: Hardware_Qualification (none) -> BOARD_QUALIFICATION_PENDING; MPN (none) -> C3225X7R2A106K250AC; Manufacturer (none) -> TDK; Procurement_Status (none) -> SELECTED_CATALOG_ITEM; Purchase_Released (none) -> false; Selection_Gaps (none) -> []; Selection_ID (none) -> SEL-3a565b360a05; Selection_Ratings (none) -> {"capacitance_pf": 10000000, "dc_bias_qualification": "PEND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; Selection_Source_URLs (none) -> https://www.digikey.com/en/products/detail/tdk/C3225X7R2A10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
- C5202: Hardware_Qualification (none) -> BOARD_QUALIFICATION_PENDING; MPN (none) -> C0805C473K1RACTU; Manufacturer (none) -> KEMET; Procurement_Status (none) -> SELECTED_CATALOG_ITEM; Purchase_Released (none) -> false; Selection_Gaps (none) -> []; Selection_ID (none) -> SEL-03610c33d4d8; Selection_Ratings (none) -> {"capacitance_pf": 47000, "dielectric": "X7R", "rated_volta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; Selection_Source_URLs (none) -> https://www.digikey.com/en/products/detail/kemet/C0805C473K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
- C5203: Hardware_Qualification (none) -> BOARD_QUALIFICATION_PENDING; MPN (none) -> C0805C474K5RACTU; Manufacturer (none) -> KEMET; Procurement_Status (none) -> SELECTED_CATALOG_ITEM; Purchase_Released (none) -> false; Selection_Gaps (none) -> []; Selection_ID (none) -> SEL-a95f291e32fb; Selection_Ratings (none) -> {"capacitance_pf": 470000, "dielectric": "X7R", "rated_volt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; Selection_Source_URLs (none) -> https://content.kemet.com/datasheets/CER_ENG_KIT_30.pdf
- C5204: Hardware_Qualification (none) -> BOARD_QUALIFICATION_PENDING; MPN (none) -> C0805C225K4RACTU; Manufacturer (none) -> KEMET; Procurement_Status (none) -> SELECTED_CATALOG_ITEM; Purchase_Released (none) -> false; Selection_Gaps (none) -> []; Selection_ID (none) -> SEL-c39b16fde8b4; Selection_Ratings (none) -> {"capacitance_pf": 2200000, "dc_bias_qualification": "PENDI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; Selection_Source_URLs (none) -> https://search.kemet.com/download/specsheet/C0805C225K4RACTU
- C5205: Hardware_Qualification (none) -> BOARD_QUALIFICATION_PENDING; MPN (none) -> C0805C105K5RACTU; Manufacturer (none) -> KEMET; Procurement_Status (none) -> SELECTED_CATALOG_ITEM; Purchase_Released (none) -> false; Selection_Gaps (none) -> []; Selection_ID (none) -> SEL-838906dbfe60; Selection_Ratings (none) -> {"capacitance_pf": 1000000, "dc_bias_qualification": "PENDI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; Selection_Source_URLs (none) -> https://search.kemet.com/component-documentation/download/s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
- C5206: Hardware_Qualification (none) -> BOARD_QUALIFICATION_PENDING; MPN (none) -> C0805C223K1RACTU; Manufacturer (none) -> KEMET; Procurement_Status (none) -> SELECTED_CATALOG_ITEM; Purchase_Released (none) -> false; Selection_Gaps (none) -> []; Selection_ID (none) -> SEL-514923e6d12b; Selection_Ratings (none) -> {"capacitance_pf": 22000, "dielectric": "X7R", "rated_volta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; Selection_Source_URLs (none) -> https://www.tme.com/Document/1eb495a6db632c9d0f71cb50aeea42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
- C5207: Hardware_Qualification (none) -> BOARD_QUALIFICATION_PENDING; MPN (none) -> C0805C181J5GACTU; Manufacturer (none) -> KEMET; Procurement_Status (none) -> SELECTED_CATALOG_ITEM; Purchase_Released (none) -> false; Selection_Gaps (none) -> ["Required effective capacitance not yet verified with supp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; Selection_ID (none) -> SEL-68451c148484; Selection_Ratings (none) -> {"capacitance_pf": 180, "dielectric": "C0G", "rated_voltage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; Selection_Source_URLs (none) -> https://www.digikey.com/en/products/detail/kemet/C0805C181J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
- C5208, C5209, C5210, C5211: value 47u 25V X7R -> 47u 16V X7R; Design note 4 output ceramics nominal188uF. Require >=100uF effective l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 -> CS3225X7R476K160NRL candidate at5V;4 ceramics nominal188uF.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; Hardware_Qualification (none) -> LAND_PATTERN_AND_EFFECTIVE_CAPACITANCE_REVIEW_REQUIRED; MPN (none) -> CS3225X7R476K160NRL; Manufacturer (none) -> Samwha Capacitor; Procurement_Status (none) -> SELECTED_CONDITIONAL; Purchase_Released (none) -> false; Selection_Gaps (none) -> ["Four capacitors must jointly retain>=100uF effective at5V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; Selection_ID (none) -> SEL-738eb3c0631c; Selection_Ratings (none) -> {"bank_refs": ["C5208", "C5209", "C5210", "C5211"], "capaci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; Selection_Source_URLs (none) -> https://jlcpcb.com/partdetail/6321105-CS3225X7R476K160NRL/C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
- D5200: Hardware_Qualification (none) -> PINOUT_RATINGS_AND_DELIVERY_SUFFIX_REVIEW_PENDING; MPN (none) -> STPS5H100BY-TR; Manufacturer (none) -> STMicroelectronics; Procurement_Status (none) -> REFERENCE_MPN_RETAINED; Purchase_Released (none) -> false; Selection_Gaps (none) -> ["Existing schematic MPN retained. Complete circuit rating/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; Selection_ID (none) -> SEL-474c4e2ea71d; Selection_Ratings (none) -> {}; Selection_Source_URLs (none) -> https://www.st.com/en/search.html#q=STPS5H100BY-TR
- D5201: Hardware_Qualification (none) -> PINOUT_RATINGS_AND_DELIVERY_SUFFIX_REVIEW_PENDING; MPN (none) -> SMBJ24CA; Manufacturer (none) -> Littelfuse; Procurement_Status (none) -> REFERENCE_MPN_RETAINED; Purchase_Released (none) -> false; Selection_Gaps (none) -> ["Existing schematic MPN retained. Complete circuit rating/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; Selection_ID (none) -> SEL-9a26101f9da7; Selection_Ratings (none) -> {}; Selection_Source_URLs (none) -> https://www.littelfuse.com/products/tvs-diodes/surface-moun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
- L5200: Hardware_Qualification (none) -> PINOUT_RATINGS_AND_DELIVERY_SUFFIX_REVIEW_PENDING; MPN (none) -> XAL7070-682MEC; Manufacturer (none) -> Coilcraft; Procurement_Status (none) -> REFERENCE_MPN_RETAINED; Purchase_Released (none) -> false; Selection_Gaps (none) -> ["Existing schematic MPN retained. Complete circuit rating/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; Selection_ID (none) -> SEL-12eeb84d8118; Selection_Ratings (none) -> {}; Selection_Source_URLs (none) -> https://www.coilcraft.com/en-us/products/power/shielded-ind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
- R5200, R5203: Hardware_Qualification (none) -> BOARD_QUALIFICATION_PENDING; MPN (none) -> RNCF0603BTE100K; Manufacturer (none) -> Stackpole Electronics; Procurement_Status (none) -> SELECTED_CATALOG_ITEM; Purchase_Released (none) -> false; Selection_Gaps (none) -> []; Selection_ID (none) -> SEL-c5cdfb61a2a3; Selection_Ratings (none) -> {"aec_q200": true, "derating": "Use manufacturer power vers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; Selection_Source_URLs (none) -> https://www.digikey.com/en/products/detail/stackpole-electr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
- R5201: Hardware_Qualification (none) -> BOARD_QUALIFICATION_PENDING; MPN (none) -> PNM0603E2502BST5; Manufacturer (none) -> Vishay; Procurement_Status (none) -> SELECTED_CATALOG_ITEM; Purchase_Released (none) -> false; Selection_Gaps (none) -> []; Selection_ID (none) -> SEL-84ab17abcd9d; Selection_Ratings (none) -> {"power_w": 0.1, "resistance_ohm": 25000, "tcr_ppm_c": 25, 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; Selection_Source_URLs (none) -> https://www.ti.com.cn/cn/lit/df/tidrav4/tidrav4.pdf
- R5202: Hardware_Qualification (none) -> BOARD_QUALIFICATION_PENDING; MPN (none) -> RNCF0805BTE470K; Manufacturer (none) -> Stackpole Electronics; Procurement_Status (none) -> SELECTED_CATALOG_ITEM; Purchase_Released (none) -> false; Selection_Gaps (none) -> []; Selection_ID (none) -> SEL-bf41e3f1a439; Selection_Ratings (none) -> {"aec_q200": true, "derating": "Use manufacturer power vers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; Selection_Source_URLs (none) -> https://www.digikey.com/en/products/detail/stackpole-electr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
- R5204: Hardware_Qualification (none) -> BOARD_QUALIFICATION_PENDING; MPN (none) -> CRCW0603100KFKEA; Manufacturer (none) -> Vishay; Procurement_Status (none) -> SELECTED_FAMILY_CODE; Purchase_Released (none) -> false; Selection_Gaps (none) -> []; Selection_ID (none) -> SEL-4e3f06cba0aa; Selection_Ratings (none) -> {"aec_q200": true, "derating": "Use manufacturer power vers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; Selection_Source_URLs (none) -> https://www.vishay.com/docs/20035/dcrcwe3.pdf
- R5205: Hardware_Qualification (none) -> BOARD_QUALIFICATION_PENDING; MPN (none) -> CRCW06031M00FKEA; Manufacturer (none) -> Vishay; Procurement_Status (none) -> SELECTED_FAMILY_CODE; Purchase_Released (none) -> false; Selection_Gaps (none) -> []; Selection_ID (none) -> SEL-0d98ae3ae719; Selection_Ratings (none) -> {"aec_q200": true, "derating": "Use manufacturer power vers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; Selection_Source_URLs (none) -> https://www.vishay.com/docs/20035/dcrcwe3.pdf
- U5200: Hardware_Qualification (none) -> BOARD_STRESS_AND_LAYOUT_REVIEW_REQUIRED; MPN (none) -> LM76003QRNPRQ1; Manufacturer (none) -> Texas Instruments; Procurement_Status (none) -> SELECTED_CONDITIONAL; Purchase_Released (none) -> false; Selection_Gaps (none) -> ["Catalog family limits verified; exact order suffix and ci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; Selection_ID (none) -> SEL-4575c1966305; Selection_Ratings (none) -> {"output_current_catalog_a": 3.5, "supply_absolute_max_v": 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; Selection_Source_URLs (none) -> https://www.ti.com/product/LM76003-Q1
