File: Power8GDI/hardware/design/outputs/ls_bank_1.kicad_sch (KiCad schematic)
At the start: 23 parts, among them U1101 TLE9104SHXUMA1, U1121 SN74LVC14AQPWRQ1

Commit message: Redesign sport target as six DI/PI channels with two motors and one lambda
Parts:
- U1121: Design note TI SCAS705B. Used gates1..4 invert MCU commands; inputs5/6 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 -> TI SCAS705B. Only assigned gates invert MCU commands; all u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
Changed lines of the file:
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@@
 (wire (pts (xy 165.1 288.29) (xy 165.1 295.91)) (stroke (width 0) (type default)))
 (global_label "PI4_IN_N" (shape bidirectional) (at 165.1 295.91 90) (effects (font (size 1.016 1.016)) (justify right bottom)))
-(symbol (lib_id "Power8GDI_Core:SN74LVC14A_Q1") (at 260.35 100.33 0) (unit 1) (in_bom yes) (on_board yes) (dnp no) (property "Reference" "U1121" (at 260.35 72.39 0) (effects (font (size 1.27 1.27)))) (property "Value" "SN74LVC14AQPWRQ1" (at 260.35 128.27 0) (effects (font (size 1.27 1.27)))) (property "Footprint" "Package_SO:TSSOP-14_4.4x5mm_P0.65mm" (at 260.35 100.33 0) (effects (font (size 1.27 1.27)) (hide yes))) (property "Design note" "TI SCAS705B. Used gates1..4 invert MCU commands; inputs5/6 tied low and outputs no-connect." (at 260.35 100.33 0) (effects (font (size 1.27 1.27)) (hide yes))) (pin "14") (pin "7") (pin "1") (pin "2") (pin "3") (pin "4") (pin "5") (pin "6") (pin "9") (pin "8") (pin "11") (pin "10") (pin "13") (pin "12") (instances (project "Power8GDI_Core" (path "/f4d21065-0a5b-5086-a08e-1af9469f04bd/0600f9f6-675b-5097-9f87-65bf79110ac0" (reference "U1121") (unit 1)))))
+(symbol (lib_id "Power8GDI_Core:SN74LVC14A_Q1") (at 260.35 100.33 0) (unit 1) (in_bom yes) (on_board yes) (dnp no) (property "Reference" "U1121" (at 260.35 72.39 0) (effects (font (size 1.27 1.27)))) (property "Value" "SN74LVC14AQPWRQ1" (at 260.35 128.27 0) (effects (font (size 1.27 1.27)))) (property "Footprint" "Package_SO:TSSOP-14_4.4x5mm_P0.65mm" (at 260.35 100.33 0) (effects (font (size 1.27 1.27)) (hide yes))) (property "Design note" "TI SCAS705B. Only assigned gates invert MCU commands; all unused inputs tied low and outputs no-connect." (at 260.35 100.33 0) (effects (font (size 1.27 1.27)) (hide yes))) (pin "14") (pin "7") (pin "1") (pin "2") (pin "3") (pin "4") (pin "5") (pin "6") (pin "9") (pin "8") (pin "11") (pin "10") (pin "13") (pin "12") (instances (project "Power8GDI_Core" (path "/f4d21065-0a5b-5086-a08e-1af9469f04bd/0600f9f6-675b-5097-9f87-65bf79110ac0" (reference "U1121") (unit 1)))))
 (wire (pts (xy 260.35 74.93) (xy 260.35 67.31)) (stroke (width 0) (type default)))
 (global_label "+3V3" (shape bidirectional) (at 260.35 67.31 270) (effects (font (size 1.016 1.016)) (justify left bottom)))

Commit message: Review B58 injector power stage and bind selected GDI6 BOM
Parts:
- C1101, C1102, C1103: Hardware_Qualification (none) -> BOARD_QUALIFICATION_PENDING; MPN (none) -> C0603C104K5RACTU; Manufacturer (none) -> KEMET; Procurement_Status (none) -> SELECTED_CATALOG_ITEM; Purchase_Released (none) -> false; Selection_Gaps (none) -> []; Selection_ID (none) -> SEL-6bf9727c4e40; Selection_Ratings (none) -> {"capacitance_pf": 100000, "dielectric": "X7R", "rated_volt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; Selection_Source_URLs (none) -> https://search.kemet.com/download/specsheet/C0603C104K5RACTU
- C1104: Hardware_Qualification (none) -> BOARD_QUALIFICATION_PENDING; MPN (none) -> C0603C105K3RACTU; Manufacturer (none) -> KEMET; Procurement_Status (none) -> SELECTED_CATALOG_ITEM; Purchase_Released (none) -> false; Selection_Gaps (none) -> []; Selection_ID (none) -> SEL-4bca20b134b8; Selection_Ratings (none) -> {"capacitance_pf": 1000000, "dc_bias_qualification": "PENDI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; Selection_Source_URLs (none) -> https://search.kemet.com/download/specsheet/C0603C105K3RACTU
- R1101, R1104, R1107, R1110: Hardware_Qualification (none) -> BOARD_QUALIFICATION_PENDING; MPN (none) -> CRCW0603100KFKEA; Manufacturer (none) -> Vishay; Procurement_Status (none) -> SELECTED_FAMILY_CODE; Purchase_Released (none) -> false; Selection_Gaps (none) -> []; Selection_ID (none) -> SEL-4e3f06cba0aa; Selection_Ratings (none) -> {"aec_q200": true, "derating": "Use manufacturer power vers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; Selection_Source_URLs (none) -> https://www.vishay.com/docs/20035/dcrcwe3.pdf
- R1102, R1105, R1108, R1111, R1115, R1116: Hardware_Qualification (none) -> BOARD_QUALIFICATION_PENDING; MPN (none) -> CRCW0603100RFKEA; Manufacturer (none) -> Vishay; Procurement_Status (none) -> SELECTED_FAMILY_CODE; Purchase_Released (none) -> false; Selection_Gaps (none) -> []; Selection_ID (none) -> SEL-319468e4af3f; Selection_Ratings (none) -> {"aec_q200": true, "derating": "Use manufacturer power vers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; Selection_Source_URLs (none) -> https://www.vishay.com/docs/20035/dcrcwe3.pdf
- R1103, R1106, R1109, R1112, R1114, R1117: Hardware_Qualification (none) -> BOARD_QUALIFICATION_PENDING; MPN (none) -> CRCW060310K0FKEA; Manufacturer (none) -> Vishay; Procurement_Status (none) -> SELECTED_FAMILY_CODE; Purchase_Released (none) -> false; Selection_Gaps (none) -> []; Selection_ID (none) -> SEL-9c0806476875; Selection_Ratings (none) -> {"aec_q200": true, "derating": "Use manufacturer power vers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; Selection_Source_URLs (none) -> https://www.vishay.com/docs/20035/dcrcwe3.pdf
- R1113: Hardware_Qualification (none) -> BOARD_QUALIFICATION_PENDING; MPN (none) -> CRCW060347R0FKEA; Manufacturer (none) -> Vishay; Procurement_Status (none) -> SELECTED_FAMILY_CODE; Purchase_Released (none) -> false; Selection_Gaps (none) -> []; Selection_ID (none) -> SEL-092784c899c7; Selection_Ratings (none) -> {"aec_q200": true, "derating": "Use manufacturer power vers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; Selection_Source_URLs (none) -> https://www.vishay.com/docs/20035/dcrcwe3.pdf
- U1101: Hardware_Qualification (none) -> PINOUT_RATINGS_AND_DELIVERY_SUFFIX_REVIEW_PENDING; MPN (none) -> TLE9104SHXUMA1; Manufacturer (none) -> Infineon Technologies; Procurement_Status (none) -> REFERENCE_MPN_RETAINED; Purchase_Released (none) -> false; Selection_Gaps (none) -> ["Existing schematic MPN retained. Complete circuit rating/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; Selection_ID (none) -> SEL-05b4f44d8450; Selection_Ratings (none) -> {}; Selection_Source_URLs (none) -> https://www.infineon.com/part/TLE9104SHXUMA1
- U1121: Hardware_Qualification (none) -> PINOUT_RATINGS_AND_DELIVERY_SUFFIX_REVIEW_PENDING; MPN (none) -> SN74LVC14AQPWRQ1; Manufacturer (none) -> Texas Instruments; Procurement_Status (none) -> REFERENCE_MPN_RETAINED; Purchase_Released (none) -> false; Selection_Gaps (none) -> ["Existing schematic MPN retained. Complete circuit rating/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; Selection_ID (none) -> SEL-90b5d0e9725e; Selection_Ratings (none) -> {}; Selection_Source_URLs (none) -> https://www.ti.com/product/SN74LVC14A-Q1/part-details/SN74L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
