File: Power8GDI/hardware/design/outputs/ls_bank_2.kicad_sch (KiCad schematic)
At the start: 23 parts, among them U1102 TLE9104SHXUMA1, U1122 SN74LVC14AQPWRQ1

Commit message: Redesign sport target as six DI/PI channels with two motors and one lambda
Parts:
- U1122: Design note TI SCAS705B. Used gates1..4 invert MCU commands; inputs5/6 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 -> TI SCAS705B. Only assigned gates invert MCU commands; all u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
Connections:
- net HARNESS_PI7 renamed HARNESS_VVT1
- net HARNESS_PI8 renamed HARNESS_VVT2
- net PI7 renamed VVT1
- net PI7_INV renamed VVT1_INV
- net PI7_IN_N renamed VVT1_IN_N
- net PI8 renamed VVT2
- net PI8_INV renamed VVT2_INV
- net PI8_IN_N renamed VVT2_IN_N
Other:
- title: Direct protected low-side PI5, PI6, PI7, PI8 -> Direct protected low-side PI5, PI6, VVT1, VVT2

Commit message: Review B58 injector power stage and bind selected GDI6 BOM
Parts:
- C1121, C1122, C1123: Hardware_Qualification (none) -> BOARD_QUALIFICATION_PENDING; MPN (none) -> C0603C104K5RACTU; Manufacturer (none) -> KEMET; Procurement_Status (none) -> SELECTED_CATALOG_ITEM; Purchase_Released (none) -> false; Selection_Gaps (none) -> []; Selection_ID (none) -> SEL-6bf9727c4e40; Selection_Ratings (none) -> {"capacitance_pf": 100000, "dielectric": "X7R", "rated_volt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; Selection_Source_URLs (none) -> https://search.kemet.com/download/specsheet/C0603C104K5RACTU
- C1124: Hardware_Qualification (none) -> BOARD_QUALIFICATION_PENDING; MPN (none) -> C0603C105K3RACTU; Manufacturer (none) -> KEMET; Procurement_Status (none) -> SELECTED_CATALOG_ITEM; Purchase_Released (none) -> false; Selection_Gaps (none) -> []; Selection_ID (none) -> SEL-4bca20b134b8; Selection_Ratings (none) -> {"capacitance_pf": 1000000, "dc_bias_qualification": "PENDI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; Selection_Source_URLs (none) -> https://search.kemet.com/download/specsheet/C0603C105K3RACTU
- R1121, R1124, R1127, R1130: Hardware_Qualification (none) -> BOARD_QUALIFICATION_PENDING; MPN (none) -> CRCW0603100KFKEA; Manufacturer (none) -> Vishay; Procurement_Status (none) -> SELECTED_FAMILY_CODE; Purchase_Released (none) -> false; Selection_Gaps (none) -> []; Selection_ID (none) -> SEL-4e3f06cba0aa; Selection_Ratings (none) -> {"aec_q200": true, "derating": "Use manufacturer power vers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; Selection_Source_URLs (none) -> https://www.vishay.com/docs/20035/dcrcwe3.pdf
- R1122, R1125, R1128, R1131, R1135, R1136: Hardware_Qualification (none) -> BOARD_QUALIFICATION_PENDING; MPN (none) -> CRCW0603100RFKEA; Manufacturer (none) -> Vishay; Procurement_Status (none) -> SELECTED_FAMILY_CODE; Purchase_Released (none) -> false; Selection_Gaps (none) -> []; Selection_ID (none) -> SEL-319468e4af3f; Selection_Ratings (none) -> {"aec_q200": true, "derating": "Use manufacturer power vers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; Selection_Source_URLs (none) -> https://www.vishay.com/docs/20035/dcrcwe3.pdf
- R1123, R1126, R1129, R1132, R1134, R1137: Hardware_Qualification (none) -> BOARD_QUALIFICATION_PENDING; MPN (none) -> CRCW060310K0FKEA; Manufacturer (none) -> Vishay; Procurement_Status (none) -> SELECTED_FAMILY_CODE; Purchase_Released (none) -> false; Selection_Gaps (none) -> []; Selection_ID (none) -> SEL-9c0806476875; Selection_Ratings (none) -> {"aec_q200": true, "derating": "Use manufacturer power vers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; Selection_Source_URLs (none) -> https://www.vishay.com/docs/20035/dcrcwe3.pdf
- R1133: Hardware_Qualification (none) -> BOARD_QUALIFICATION_PENDING; MPN (none) -> CRCW060347R0FKEA; Manufacturer (none) -> Vishay; Procurement_Status (none) -> SELECTED_FAMILY_CODE; Purchase_Released (none) -> false; Selection_Gaps (none) -> []; Selection_ID (none) -> SEL-092784c899c7; Selection_Ratings (none) -> {"aec_q200": true, "derating": "Use manufacturer power vers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; Selection_Source_URLs (none) -> https://www.vishay.com/docs/20035/dcrcwe3.pdf
- U1102: Hardware_Qualification (none) -> PINOUT_RATINGS_AND_DELIVERY_SUFFIX_REVIEW_PENDING; MPN (none) -> TLE9104SHXUMA1; Manufacturer (none) -> Infineon Technologies; Procurement_Status (none) -> REFERENCE_MPN_RETAINED; Purchase_Released (none) -> false; Selection_Gaps (none) -> ["Existing schematic MPN retained. Complete circuit rating/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; Selection_ID (none) -> SEL-05b4f44d8450; Selection_Ratings (none) -> {}; Selection_Source_URLs (none) -> https://www.infineon.com/part/TLE9104SHXUMA1
- U1122: Hardware_Qualification (none) -> PINOUT_RATINGS_AND_DELIVERY_SUFFIX_REVIEW_PENDING; MPN (none) -> SN74LVC14AQPWRQ1; Manufacturer (none) -> Texas Instruments; Procurement_Status (none) -> REFERENCE_MPN_RETAINED; Purchase_Released (none) -> false; Selection_Gaps (none) -> ["Existing schematic MPN retained. Complete circuit rating/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; Selection_ID (none) -> SEL-90b5d0e9725e; Selection_Ratings (none) -> {}; Selection_Source_URLs (none) -> https://www.ti.com/product/SN74LVC14A-Q1/part-details/SN74L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
