File: Power8GDI/hardware/design/outputs/ls_bank_3.kicad_sch (KiCad schematic)
At the start: 23 parts, among them U1103 TLE9104SHXUMA1, U1123 SN74LVC14AQPWRQ1

Commit message: Redesign sport target as six DI/PI channels with two motors and one lambda
Parts:
- U1123: Design note TI SCAS705B. Used gates1..4 invert MCU commands; inputs5/6 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 -> TI SCAS705B. Only assigned gates invert MCU commands; all u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
Connections:
- net HARNESS_VVT1 is gone; now on net HARNESS_VVT3: U1103.1 (OUT1)
- net HARNESS_VVT2 is gone; now on net HARNESS_VVT4: U1103.20 (OUT2)
- net VVT1 is gone; now on net VVT3: R1141.1, U1123.1 (1A)
- net VVT1_INV is gone; now on net VVT3_INV: R1142.1, U1123.2 (1Y_INV)
- net VVT1_IN_N is gone; now on net VVT3_IN_N: R1142.2, R1143.2, U1103.3 (IN1_N)
- net VVT2 is gone; now on net VVT4: R1144.1, U1123.3 (2A)
- net VVT2_INV is gone; now on net VVT4_INV: R1145.1, U1123.4 (2Y_INV)
- net VVT2_IN_N is gone; now on net VVT4_IN_N: R1145.2, R1146.2, U1103.18 (IN2_N)
- net HARNESS_VVT3: no longer U1103.10 (OUT3)
- net HARNESS_VVT4: no longer U1103.11 (OUT4)
- net VVT3: no longer R1147.1, U1123.5 (3A)
- net VVT3_INV: no longer R1148.1, U1123.6 (3Y_INV)
- net VVT3_IN_N: no longer R1148.2, R1149.2, U1103.4 (IN3_N)
- net VVT4: no longer R1150.1, U1123.9 (4A)
- net VVT4_INV: no longer R1151.1, U1123.8 (4Y_INV)
- net VVT4_IN_N: no longer R1151.2, R1152.2, U1103.17 (IN4_N)
- new net AUX_PWM1: R1147.1, U1123.5 (3A)
- new net AUX_PWM1_INV: R1148.1, U1123.6 (3Y_INV)
- new net AUX_PWM1_IN_N: R1148.2, R1149.2, U1103.4 (IN3_N)
- new net AUX_PWM2: R1150.1, U1123.9 (4A)
- new net AUX_PWM2_INV: R1151.1, U1123.8 (4Y_INV)
- new net AUX_PWM2_IN_N: R1151.2, R1152.2, U1103.17 (IN4_N)
- new net HARNESS_AUX_PWM1: U1103.10 (OUT3)
- new net HARNESS_AUX_PWM2: U1103.11 (OUT4)
Other:
- title: Direct protected low-side VVT1, VVT2, VVT3, VVT4 -> Direct protected low-side VVT3, VVT4, AUX_PWM1, AUX_PWM2

Commit message: Review B58 injector power stage and bind selected GDI6 BOM
Parts:
- C1141, C1142, C1143: Hardware_Qualification (none) -> BOARD_QUALIFICATION_PENDING; MPN (none) -> C0603C104K5RACTU; Manufacturer (none) -> KEMET; Procurement_Status (none) -> SELECTED_CATALOG_ITEM; Purchase_Released (none) -> false; Selection_Gaps (none) -> []; Selection_ID (none) -> SEL-6bf9727c4e40; Selection_Ratings (none) -> {"capacitance_pf": 100000, "dielectric": "X7R", "rated_volt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; Selection_Source_URLs (none) -> https://search.kemet.com/download/specsheet/C0603C104K5RACTU
- C1144: Hardware_Qualification (none) -> BOARD_QUALIFICATION_PENDING; MPN (none) -> C0603C105K3RACTU; Manufacturer (none) -> KEMET; Procurement_Status (none) -> SELECTED_CATALOG_ITEM; Purchase_Released (none) -> false; Selection_Gaps (none) -> []; Selection_ID (none) -> SEL-4bca20b134b8; Selection_Ratings (none) -> {"capacitance_pf": 1000000, "dc_bias_qualification": "PENDI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; Selection_Source_URLs (none) -> https://search.kemet.com/download/specsheet/C0603C105K3RACTU
- R1141, R1144, R1147, R1150: Hardware_Qualification (none) -> BOARD_QUALIFICATION_PENDING; MPN (none) -> CRCW0603100KFKEA; Manufacturer (none) -> Vishay; Procurement_Status (none) -> SELECTED_FAMILY_CODE; Purchase_Released (none) -> false; Selection_Gaps (none) -> []; Selection_ID (none) -> SEL-4e3f06cba0aa; Selection_Ratings (none) -> {"aec_q200": true, "derating": "Use manufacturer power vers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; Selection_Source_URLs (none) -> https://www.vishay.com/docs/20035/dcrcwe3.pdf
- R1142, R1145, R1148, R1151, R1155, R1156: Hardware_Qualification (none) -> BOARD_QUALIFICATION_PENDING; MPN (none) -> CRCW0603100RFKEA; Manufacturer (none) -> Vishay; Procurement_Status (none) -> SELECTED_FAMILY_CODE; Purchase_Released (none) -> false; Selection_Gaps (none) -> []; Selection_ID (none) -> SEL-319468e4af3f; Selection_Ratings (none) -> {"aec_q200": true, "derating": "Use manufacturer power vers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; Selection_Source_URLs (none) -> https://www.vishay.com/docs/20035/dcrcwe3.pdf
- R1143, R1146, R1149, R1152, R1154, R1157: Hardware_Qualification (none) -> BOARD_QUALIFICATION_PENDING; MPN (none) -> CRCW060310K0FKEA; Manufacturer (none) -> Vishay; Procurement_Status (none) -> SELECTED_FAMILY_CODE; Purchase_Released (none) -> false; Selection_Gaps (none) -> []; Selection_ID (none) -> SEL-9c0806476875; Selection_Ratings (none) -> {"aec_q200": true, "derating": "Use manufacturer power vers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; Selection_Source_URLs (none) -> https://www.vishay.com/docs/20035/dcrcwe3.pdf
- R1153: Hardware_Qualification (none) -> BOARD_QUALIFICATION_PENDING; MPN (none) -> CRCW060347R0FKEA; Manufacturer (none) -> Vishay; Procurement_Status (none) -> SELECTED_FAMILY_CODE; Purchase_Released (none) -> false; Selection_Gaps (none) -> []; Selection_ID (none) -> SEL-092784c899c7; Selection_Ratings (none) -> {"aec_q200": true, "derating": "Use manufacturer power vers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; Selection_Source_URLs (none) -> https://www.vishay.com/docs/20035/dcrcwe3.pdf
- U1103: Hardware_Qualification (none) -> PINOUT_RATINGS_AND_DELIVERY_SUFFIX_REVIEW_PENDING; MPN (none) -> TLE9104SHXUMA1; Manufacturer (none) -> Infineon Technologies; Procurement_Status (none) -> REFERENCE_MPN_RETAINED; Purchase_Released (none) -> false; Selection_Gaps (none) -> ["Existing schematic MPN retained. Complete circuit rating/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; Selection_ID (none) -> SEL-05b4f44d8450; Selection_Ratings (none) -> {}; Selection_Source_URLs (none) -> https://www.infineon.com/part/TLE9104SHXUMA1
- U1123: Hardware_Qualification (none) -> PINOUT_RATINGS_AND_DELIVERY_SUFFIX_REVIEW_PENDING; MPN (none) -> SN74LVC14AQPWRQ1; Manufacturer (none) -> Texas Instruments; Procurement_Status (none) -> REFERENCE_MPN_RETAINED; Purchase_Released (none) -> false; Selection_Gaps (none) -> ["Existing schematic MPN retained. Complete circuit rating/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; Selection_ID (none) -> SEL-90b5d0e9725e; Selection_Ratings (none) -> {}; Selection_Source_URLs (none) -> https://www.ti.com/product/SN74LVC14A-Q1/part-details/SN74L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
