File: Power8GDI/hardware/design/outputs/ls_bank_4.kicad_sch (KiCad schematic)
At the start: 23 parts, among them U1104 TLE9104SHXUMA1, U1124 SN74LVC14AQPWRQ1

Commit message: Redesign sport target as six DI/PI channels with two motors and one lambda
Parts:
- U1124: Design note TI SCAS705B. Used gates1..4 invert MCU commands; inputs5/6 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 -> TI SCAS705B. Only assigned gates invert MCU commands; all u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
Connections:
- net AUX_PWM1 is gone; now on net AUX_PWM3: R1161.1, U1124.1 (1A)
- net AUX_PWM1_INV is gone; now on net AUX_PWM3_INV: R1162.1, U1124.2 (1Y_INV)
- net AUX_PWM1_IN_N is gone; now on net AUX_PWM3_IN_N: R1162.2, R1163.2, U1104.3 (IN1_N)
- net AUX_PWM2 is gone; now on net AUX_PWM4: R1164.1, U1124.3 (2A)
- net AUX_PWM2_INV is gone; now on net AUX_PWM4_INV: R1165.1, U1124.4 (2Y_INV)
- net AUX_PWM2_IN_N is gone; now on net AUX_PWM4_IN_N: R1165.2, R1166.2, U1104.18 (IN2_N)
- net HARNESS_AUX_PWM1 is gone; now on net HARNESS_AUX_PWM3: U1104.1 (OUT1)
- net HARNESS_AUX_PWM2 is gone; now on net HARNESS_AUX_PWM4: U1104.20 (OUT2)
- net AUX_PWM3: no longer R1167.1, U1124.5 (3A)
- net AUX_PWM3_INV: no longer R1168.1, U1124.6 (3Y_INV)
- net AUX_PWM3_IN_N: no longer R1168.2, R1169.2, U1104.4 (IN3_N)
- net AUX_PWM4: no longer R1170.1, U1124.9 (4A)
- net AUX_PWM4_INV: no longer R1171.1, U1124.8 (4Y_INV)
- net AUX_PWM4_IN_N: no longer R1171.2, R1172.2, U1104.17 (IN4_N)
- net HARNESS_AUX_PWM3: no longer U1104.10 (OUT3)
- net HARNESS_AUX_PWM4: no longer U1104.11 (OUT4)
- new net AUX_PWM5: R1167.1, U1124.5 (3A)
- new net AUX_PWM5_INV: R1168.1, U1124.6 (3Y_INV)
- new net AUX_PWM5_IN_N: R1168.2, R1169.2, U1104.4 (IN3_N)
- new net AUX_PWM6: R1170.1, U1124.9 (4A)
- new net AUX_PWM6_INV: R1171.1, U1124.8 (4Y_INV)
- new net AUX_PWM6_IN_N: R1171.2, R1172.2, U1104.17 (IN4_N)
- new net HARNESS_AUX_PWM5: U1104.10 (OUT3)
- new net HARNESS_AUX_PWM6: U1104.11 (OUT4)
Other:
- title: Direct protected low-side AUX_PWM1, AUX_PWM2, AUX_PWM3, AUX_PWM4 -> Direct protected low-side AUX_PWM3, AUX_PWM4, AUX_PWM5, AUX_PWM6

Commit message: Review B58 injector power stage and bind selected GDI6 BOM
Parts:
- C1161, C1162, C1163: Hardware_Qualification (none) -> BOARD_QUALIFICATION_PENDING; MPN (none) -> C0603C104K5RACTU; Manufacturer (none) -> KEMET; Procurement_Status (none) -> SELECTED_CATALOG_ITEM; Purchase_Released (none) -> false; Selection_Gaps (none) -> []; Selection_ID (none) -> SEL-6bf9727c4e40; Selection_Ratings (none) -> {"capacitance_pf": 100000, "dielectric": "X7R", "rated_volt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; Selection_Source_URLs (none) -> https://search.kemet.com/download/specsheet/C0603C104K5RACTU
- C1164: Hardware_Qualification (none) -> BOARD_QUALIFICATION_PENDING; MPN (none) -> C0603C105K3RACTU; Manufacturer (none) -> KEMET; Procurement_Status (none) -> SELECTED_CATALOG_ITEM; Purchase_Released (none) -> false; Selection_Gaps (none) -> []; Selection_ID (none) -> SEL-4bca20b134b8; Selection_Ratings (none) -> {"capacitance_pf": 1000000, "dc_bias_qualification": "PENDI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; Selection_Source_URLs (none) -> https://search.kemet.com/download/specsheet/C0603C105K3RACTU
- R1161, R1164, R1167, R1170: Hardware_Qualification (none) -> BOARD_QUALIFICATION_PENDING; MPN (none) -> CRCW0603100KFKEA; Manufacturer (none) -> Vishay; Procurement_Status (none) -> SELECTED_FAMILY_CODE; Purchase_Released (none) -> false; Selection_Gaps (none) -> []; Selection_ID (none) -> SEL-4e3f06cba0aa; Selection_Ratings (none) -> {"aec_q200": true, "derating": "Use manufacturer power vers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; Selection_Source_URLs (none) -> https://www.vishay.com/docs/20035/dcrcwe3.pdf
- R1162, R1165, R1168, R1171, R1175, R1176: Hardware_Qualification (none) -> BOARD_QUALIFICATION_PENDING; MPN (none) -> CRCW0603100RFKEA; Manufacturer (none) -> Vishay; Procurement_Status (none) -> SELECTED_FAMILY_CODE; Purchase_Released (none) -> false; Selection_Gaps (none) -> []; Selection_ID (none) -> SEL-319468e4af3f; Selection_Ratings (none) -> {"aec_q200": true, "derating": "Use manufacturer power vers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; Selection_Source_URLs (none) -> https://www.vishay.com/docs/20035/dcrcwe3.pdf
- R1163, R1166, R1169, R1172, R1174, R1177: Hardware_Qualification (none) -> BOARD_QUALIFICATION_PENDING; MPN (none) -> CRCW060310K0FKEA; Manufacturer (none) -> Vishay; Procurement_Status (none) -> SELECTED_FAMILY_CODE; Purchase_Released (none) -> false; Selection_Gaps (none) -> []; Selection_ID (none) -> SEL-9c0806476875; Selection_Ratings (none) -> {"aec_q200": true, "derating": "Use manufacturer power vers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; Selection_Source_URLs (none) -> https://www.vishay.com/docs/20035/dcrcwe3.pdf
- R1173: Hardware_Qualification (none) -> BOARD_QUALIFICATION_PENDING; MPN (none) -> CRCW060347R0FKEA; Manufacturer (none) -> Vishay; Procurement_Status (none) -> SELECTED_FAMILY_CODE; Purchase_Released (none) -> false; Selection_Gaps (none) -> []; Selection_ID (none) -> SEL-092784c899c7; Selection_Ratings (none) -> {"aec_q200": true, "derating": "Use manufacturer power vers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; Selection_Source_URLs (none) -> https://www.vishay.com/docs/20035/dcrcwe3.pdf
- U1104: Hardware_Qualification (none) -> PINOUT_RATINGS_AND_DELIVERY_SUFFIX_REVIEW_PENDING; MPN (none) -> TLE9104SHXUMA1; Manufacturer (none) -> Infineon Technologies; Procurement_Status (none) -> REFERENCE_MPN_RETAINED; Purchase_Released (none) -> false; Selection_Gaps (none) -> ["Existing schematic MPN retained. Complete circuit rating/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; Selection_ID (none) -> SEL-05b4f44d8450; Selection_Ratings (none) -> {}; Selection_Source_URLs (none) -> https://www.infineon.com/part/TLE9104SHXUMA1
- U1124: Hardware_Qualification (none) -> PINOUT_RATINGS_AND_DELIVERY_SUFFIX_REVIEW_PENDING; MPN (none) -> SN74LVC14AQPWRQ1; Manufacturer (none) -> Texas Instruments; Procurement_Status (none) -> REFERENCE_MPN_RETAINED; Purchase_Released (none) -> false; Selection_Gaps (none) -> ["Existing schematic MPN retained. Complete circuit rating/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; Selection_ID (none) -> SEL-90b5d0e9725e; Selection_Ratings (none) -> {}; Selection_Source_URLs (none) -> https://www.ti.com/product/SN74LVC14A-Q1/part-details/SN74L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
