File: Power8GDI/hardware/design/outputs/ls_bank_5.kicad_sch (KiCad schematic)
At the start: 23 parts, among them U1105 TLE9104SHXUMA1, U1125 SN74LVC14AQPWRQ1

Commit message: Redesign sport target as six DI/PI channels with two motors and one lambda
Parts:
- U1125: Design note TI SCAS705B. Used gates1..4 invert MCU commands; inputs5/6 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 -> TI SCAS705B. Only assigned gates invert MCU commands; all u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
Connections:
- net AUX_PWM5 is gone; now on net AUX_PWM7: R1181.1, U1125.1 (1A)
- net AUX_PWM5_INV is gone; now on net AUX_PWM7_INV: R1182.1, U1125.2 (1Y_INV)
- net AUX_PWM5_IN_N is gone; now on net AUX_PWM7_IN_N: R1182.2, R1183.2, U1105.3 (IN1_N)
- net AUX_PWM6 is gone; now on net AUX_PWM8: R1184.1, U1125.3 (2A)
- net AUX_PWM6_INV is gone; now on net AUX_PWM8_INV: R1185.1, U1125.4 (2Y_INV)
- net AUX_PWM6_IN_N is gone; now on net AUX_PWM8_IN_N: R1185.2, R1186.2, U1105.18 (IN2_N)
- net HARNESS_AUX_PWM5 is gone; now on net HARNESS_AUX_PWM7: U1105.1 (OUT1)
- net HARNESS_AUX_PWM6 is gone; now on net HARNESS_AUX_PWM8: U1105.20 (OUT2)
- net AUX_PWM7: no longer R1187.1, U1125.5 (3A)
- net AUX_PWM7_INV: no longer R1188.1, U1125.6 (3Y_INV)
- net AUX_PWM7_IN_N: no longer R1188.2, R1189.2, U1105.4 (IN3_N)
- net AUX_PWM8: no longer R1190.1, U1125.9 (4A)
- net AUX_PWM8_INV: no longer R1191.1, U1125.8 (4Y_INV)
- net AUX_PWM8_IN_N: no longer R1191.2, R1192.2, U1105.17 (IN4_N)
- net HARNESS_AUX_PWM7: no longer U1105.10 (OUT3)
- net HARNESS_AUX_PWM8: no longer U1105.11 (OUT4)
- new net HARNESS_LS_AUX1: U1105.10 (OUT3)
- new net HARNESS_LS_AUX2: U1105.11 (OUT4)
- new net LS_AUX1: R1187.1, U1125.5 (3A)
- new net LS_AUX1_INV: R1188.1, U1125.6 (3Y_INV)
- new net LS_AUX1_IN_N: R1188.2, R1189.2, U1105.4 (IN3_N)
- new net LS_AUX2: R1190.1, U1125.9 (4A)
- new net LS_AUX2_INV: R1191.1, U1125.8 (4Y_INV)
- new net LS_AUX2_IN_N: R1191.2, R1192.2, U1105.17 (IN4_N)
Other:
- title: Direct protected low-side AUX_PWM5, AUX_PWM6, AUX_PWM7, AUX_PWM8 -> Direct protected low-side AUX_PWM7, AUX_PWM8, LS_AUX1, LS_AUX2

Commit message: Review B58 injector power stage and bind selected GDI6 BOM
Parts:
- C1181, C1182, C1183: Hardware_Qualification (none) -> BOARD_QUALIFICATION_PENDING; MPN (none) -> C0603C104K5RACTU; Manufacturer (none) -> KEMET; Procurement_Status (none) -> SELECTED_CATALOG_ITEM; Purchase_Released (none) -> false; Selection_Gaps (none) -> []; Selection_ID (none) -> SEL-6bf9727c4e40; Selection_Ratings (none) -> {"capacitance_pf": 100000, "dielectric": "X7R", "rated_volt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; Selection_Source_URLs (none) -> https://search.kemet.com/download/specsheet/C0603C104K5RACTU
- C1184: Hardware_Qualification (none) -> BOARD_QUALIFICATION_PENDING; MPN (none) -> C0603C105K3RACTU; Manufacturer (none) -> KEMET; Procurement_Status (none) -> SELECTED_CATALOG_ITEM; Purchase_Released (none) -> false; Selection_Gaps (none) -> []; Selection_ID (none) -> SEL-4bca20b134b8; Selection_Ratings (none) -> {"capacitance_pf": 1000000, "dc_bias_qualification": "PENDI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; Selection_Source_URLs (none) -> https://search.kemet.com/download/specsheet/C0603C105K3RACTU
- R1181, R1184, R1187, R1190: Hardware_Qualification (none) -> BOARD_QUALIFICATION_PENDING; MPN (none) -> CRCW0603100KFKEA; Manufacturer (none) -> Vishay; Procurement_Status (none) -> SELECTED_FAMILY_CODE; Purchase_Released (none) -> false; Selection_Gaps (none) -> []; Selection_ID (none) -> SEL-4e3f06cba0aa; Selection_Ratings (none) -> {"aec_q200": true, "derating": "Use manufacturer power vers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; Selection_Source_URLs (none) -> https://www.vishay.com/docs/20035/dcrcwe3.pdf
- R1182, R1185, R1188, R1191, R1195, R1196: Hardware_Qualification (none) -> BOARD_QUALIFICATION_PENDING; MPN (none) -> CRCW0603100RFKEA; Manufacturer (none) -> Vishay; Procurement_Status (none) -> SELECTED_FAMILY_CODE; Purchase_Released (none) -> false; Selection_Gaps (none) -> []; Selection_ID (none) -> SEL-319468e4af3f; Selection_Ratings (none) -> {"aec_q200": true, "derating": "Use manufacturer power vers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; Selection_Source_URLs (none) -> https://www.vishay.com/docs/20035/dcrcwe3.pdf
- R1183, R1186, R1189, R1192, R1194, R1197: Hardware_Qualification (none) -> BOARD_QUALIFICATION_PENDING; MPN (none) -> CRCW060310K0FKEA; Manufacturer (none) -> Vishay; Procurement_Status (none) -> SELECTED_FAMILY_CODE; Purchase_Released (none) -> false; Selection_Gaps (none) -> []; Selection_ID (none) -> SEL-9c0806476875; Selection_Ratings (none) -> {"aec_q200": true, "derating": "Use manufacturer power vers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; Selection_Source_URLs (none) -> https://www.vishay.com/docs/20035/dcrcwe3.pdf
- R1193: Hardware_Qualification (none) -> BOARD_QUALIFICATION_PENDING; MPN (none) -> CRCW060347R0FKEA; Manufacturer (none) -> Vishay; Procurement_Status (none) -> SELECTED_FAMILY_CODE; Purchase_Released (none) -> false; Selection_Gaps (none) -> []; Selection_ID (none) -> SEL-092784c899c7; Selection_Ratings (none) -> {"aec_q200": true, "derating": "Use manufacturer power vers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; Selection_Source_URLs (none) -> https://www.vishay.com/docs/20035/dcrcwe3.pdf
- U1105: Hardware_Qualification (none) -> PINOUT_RATINGS_AND_DELIVERY_SUFFIX_REVIEW_PENDING; MPN (none) -> TLE9104SHXUMA1; Manufacturer (none) -> Infineon Technologies; Procurement_Status (none) -> REFERENCE_MPN_RETAINED; Purchase_Released (none) -> false; Selection_Gaps (none) -> ["Existing schematic MPN retained. Complete circuit rating/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; Selection_ID (none) -> SEL-05b4f44d8450; Selection_Ratings (none) -> {}; Selection_Source_URLs (none) -> https://www.infineon.com/part/TLE9104SHXUMA1
- U1125: Hardware_Qualification (none) -> PINOUT_RATINGS_AND_DELIVERY_SUFFIX_REVIEW_PENDING; MPN (none) -> SN74LVC14AQPWRQ1; Manufacturer (none) -> Texas Instruments; Procurement_Status (none) -> REFERENCE_MPN_RETAINED; Purchase_Released (none) -> false; Selection_Gaps (none) -> ["Existing schematic MPN retained. Complete circuit rating/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; Selection_ID (none) -> SEL-90b5d0e9725e; Selection_Ratings (none) -> {}; Selection_Source_URLs (none) -> https://www.ti.com/product/SN74LVC14A-Q1/part-details/SN74L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
