File: Power8GDI/hardware/design/outputs/ls_bank_6.kicad_sch (KiCad schematic)
At the start: 23 parts, among them U1106 TLE9104SHXUMA1, U1126 SN74LVC14AQPWRQ1

Commit message: Redesign sport target as six DI/PI channels with two motors and one lambda
Parts:
- removed R1207, R1210: 100k, Resistor_SMD:R_0603_1608Metric, symbol Power8GDI_Core:R
- removed R1208, R1211: 100R, Resistor_SMD:R_0603_1608Metric, symbol Power8GDI_Core:R
- removed R1209, R1212: 10k, Resistor_SMD:R_0603_1608Metric, symbol Power8GDI_Core:R
- U1126: Design note TI SCAS705B. Used gates1..4 invert MCU commands; inputs5/6 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 -> TI SCAS705B. Only assigned gates invert MCU commands; all u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
Connections:
- net HARNESS_LS_AUX1 is gone; now on net HARNESS_LS_AUX3: U1106.1 (OUT1)
- net HARNESS_LS_AUX2 is gone; now on net HARNESS_LS_AUX4: U1106.20 (OUT2)
- net LS_AUX1 is gone; now on net LS_AUX3: R1201.1, U1126.1 (1A)
- net LS_AUX1_INV is gone; now on net LS_AUX3_INV: R1202.1, U1126.2 (1Y_INV)
- net LS_AUX1_IN_N is gone; now on net LS_AUX3_IN_N: R1202.2, R1203.2, U1106.3 (IN1_N)
- net LS_AUX2 is gone; now on net LS_AUX4: R1204.1, U1126.3 (2A)
- net LS_AUX2_INV is gone; now on net LS_AUX4_INV: R1205.1, U1126.4 (2Y_INV)
- net LS_AUX2_IN_N is gone; now on net LS_AUX4_IN_N: R1205.2, R1206.2, U1106.18 (IN2_N)
- net +3V3: now also U1106.17 (IN4_N), U1106.4 (IN3_N)
- net GND: now also U1126.5 (3A), U1126.9 (4A)
- net HARNESS_LS_AUX3: no longer U1106.10 (OUT3)
- net HARNESS_LS_AUX4: no longer U1106.11 (OUT4)
- net LS_AUX3: no longer U1126.5 (3A)
- net LS_AUX3_INV: no longer U1126.6 (3Y_INV)
- net LS_AUX3_IN_N: no longer U1106.4 (IN3_N)
- net LS_AUX4: no longer U1126.9 (4A)
- net LS_AUX4_INV: no longer U1126.8 (4Y_INV)
- net LS_AUX4_IN_N: no longer U1106.17 (IN4_N)
- no-connect marks 2 -> 6
Other:
- title: Direct protected low-side LS_AUX1, LS_AUX2, LS_AUX3, LS_AUX4 -> Direct protected low-side LS_AUX3, LS_AUX4

Commit message: Review B58 injector power stage and bind selected GDI6 BOM
Parts:
- C1201, C1202, C1203: Hardware_Qualification (none) -> BOARD_QUALIFICATION_PENDING; MPN (none) -> C0603C104K5RACTU; Manufacturer (none) -> KEMET; Procurement_Status (none) -> SELECTED_CATALOG_ITEM; Purchase_Released (none) -> false; Selection_Gaps (none) -> []; Selection_ID (none) -> SEL-6bf9727c4e40; Selection_Ratings (none) -> {"capacitance_pf": 100000, "dielectric": "X7R", "rated_volt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; Selection_Source_URLs (none) -> https://search.kemet.com/download/specsheet/C0603C104K5RACTU
- C1204: Hardware_Qualification (none) -> BOARD_QUALIFICATION_PENDING; MPN (none) -> C0603C105K3RACTU; Manufacturer (none) -> KEMET; Procurement_Status (none) -> SELECTED_CATALOG_ITEM; Purchase_Released (none) -> false; Selection_Gaps (none) -> []; Selection_ID (none) -> SEL-4bca20b134b8; Selection_Ratings (none) -> {"capacitance_pf": 1000000, "dc_bias_qualification": "PENDI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; Selection_Source_URLs (none) -> https://search.kemet.com/download/specsheet/C0603C105K3RACTU
- R1201, R1204: Hardware_Qualification (none) -> BOARD_QUALIFICATION_PENDING; MPN (none) -> CRCW0603100KFKEA; Manufacturer (none) -> Vishay; Procurement_Status (none) -> SELECTED_FAMILY_CODE; Purchase_Released (none) -> false; Selection_Gaps (none) -> []; Selection_ID (none) -> SEL-4e3f06cba0aa; Selection_Ratings (none) -> {"aec_q200": true, "derating": "Use manufacturer power vers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; Selection_Source_URLs (none) -> https://www.vishay.com/docs/20035/dcrcwe3.pdf
- R1202, R1205, R1215, R1216: Hardware_Qualification (none) -> BOARD_QUALIFICATION_PENDING; MPN (none) -> CRCW0603100RFKEA; Manufacturer (none) -> Vishay; Procurement_Status (none) -> SELECTED_FAMILY_CODE; Purchase_Released (none) -> false; Selection_Gaps (none) -> []; Selection_ID (none) -> SEL-319468e4af3f; Selection_Ratings (none) -> {"aec_q200": true, "derating": "Use manufacturer power vers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; Selection_Source_URLs (none) -> https://www.vishay.com/docs/20035/dcrcwe3.pdf
- R1203, R1206, R1214, R1217: Hardware_Qualification (none) -> BOARD_QUALIFICATION_PENDING; MPN (none) -> CRCW060310K0FKEA; Manufacturer (none) -> Vishay; Procurement_Status (none) -> SELECTED_FAMILY_CODE; Purchase_Released (none) -> false; Selection_Gaps (none) -> []; Selection_ID (none) -> SEL-9c0806476875; Selection_Ratings (none) -> {"aec_q200": true, "derating": "Use manufacturer power vers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; Selection_Source_URLs (none) -> https://www.vishay.com/docs/20035/dcrcwe3.pdf
- R1213: Hardware_Qualification (none) -> BOARD_QUALIFICATION_PENDING; MPN (none) -> CRCW060347R0FKEA; Manufacturer (none) -> Vishay; Procurement_Status (none) -> SELECTED_FAMILY_CODE; Purchase_Released (none) -> false; Selection_Gaps (none) -> []; Selection_ID (none) -> SEL-092784c899c7; Selection_Ratings (none) -> {"aec_q200": true, "derating": "Use manufacturer power vers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; Selection_Source_URLs (none) -> https://www.vishay.com/docs/20035/dcrcwe3.pdf
- U1106: Hardware_Qualification (none) -> PINOUT_RATINGS_AND_DELIVERY_SUFFIX_REVIEW_PENDING; MPN (none) -> TLE9104SHXUMA1; Manufacturer (none) -> Infineon Technologies; Procurement_Status (none) -> REFERENCE_MPN_RETAINED; Purchase_Released (none) -> false; Selection_Gaps (none) -> ["Existing schematic MPN retained. Complete circuit rating/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; Selection_ID (none) -> SEL-05b4f44d8450; Selection_Ratings (none) -> {}; Selection_Source_URLs (none) -> https://www.infineon.com/part/TLE9104SHXUMA1
- U1126: Hardware_Qualification (none) -> PINOUT_RATINGS_AND_DELIVERY_SUFFIX_REVIEW_PENDING; MPN (none) -> SN74LVC14AQPWRQ1; Manufacturer (none) -> Texas Instruments; Procurement_Status (none) -> REFERENCE_MPN_RETAINED; Purchase_Released (none) -> false; Selection_Gaps (none) -> ["Existing schematic MPN retained. Complete circuit rating/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; Selection_ID (none) -> SEL-90b5d0e9725e; Selection_Ratings (none) -> {}; Selection_Source_URLs (none) -> https://www.ti.com/product/SN74LVC14A-Q1/part-details/SN74L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
