File: Power8GDI/hardware/design/safety/safety_gate.kicad_sch (KiCad schematic)
At the start: 33 parts, among them U801 TPS3431SQDRBRQ1, U802 TPS3808G33QDBVRQ1, U803 SN74LVC1G17QDBVRQ1, U804 SN74LVC2G74QDCURQ1, U805 SN74LVC244AQPWRQ1

Commit message: Connect eight passive-coil stages to global fault latch and validate revised hierarchy
Parts:
- removed C805: 100nF 25V X7R, Capacitor_SMD:C_0603_1608Metric, symbol Power8GDI_Safety:C
- removed R811, R812, R813, R814, R815, R816, R817, R818, R821, R822, R823, R824, R825, R826, R827, R828: 10k 1%, Resistor_SMD:R_0603_1608Metric, symbol Power8GDI_Safety:R
- removed U805: SN74LVC244AQPWRQ1, Package_SO:Texas_PW0020A_TSSOP-20_4.4x6.5mm_P0.65mm, symbol Power8GDI_Safety:SN74LVC244AQPWRQ1
- added R6500: 0R, Resistor_SMD:R_0603_1608Metric, symbol Power8GDI_Safety:R
Connections:
- net HW_KILL_N: now also R6500.2
- new net IGN_OC_OK: R6500.1
Other:
- note added: "3.3 V logic only. Hardware faults asynchronously clear enable; recovery requires a fresh ARM rising edge. Ignition OC joins HW_KILL_N through R6500. Per-load inhibition lives on driver sheets. 64.288 ms nominal watchdog is a backup CPU monitor, NOT a coil dwell/current limiter."
- note added: "HW_KILL_N: local 3.3 V open-drain/contact-to-ground boundary only; no harness/12 V direct connection. Local ignition timers and latched OC detectors are on ignition sheets. ARM/power-sequence tests remain required. IC decoupling capacitors C801..C804 must be placed at U801..U804 respectively."
- note removed: "3.3 V logic only. Hardware faults asynchronously clear enable; recovery requires a fresh ARM rising edge. MIC output isolation remains DNP. No PT2001 DRVEN connection or assumed polarity. 64.288 ms nominal watchdog is a backup CPU monitor, NOT a coil dwell/current limiter."
- note removed: "HW_KILL_N: local 3.3 V open-drain/contact-to-ground boundary only; no harness/12 V direct connection. No independent max-dwell/current limiter exists yet. ARM timing and power-sequence fault injection remain required. IC decoupling capacitors C801..C805 must be placed at U801..U805 respectively."
- title: Watchdog, latched inhibit and eight ignition gates -> Watchdog and latched global actuator inhibit
- moved on the sheet: C801, C802, C803, C804, C806

Commit message: Latch actuator inhibit on independent 5V undervoltage detection
Parts:
- added C807: 100nF 25V X7R, Capacitor_SMD:C_0603_1608Metric, symbol Power8GDI_Safety:C
- added C808: 1nF 50V C0G 5%, Capacitor_SMD:C_0603_1608Metric, symbol Power8GDI_Safety:C
- added R807: 102k 0.1% 25ppm, Resistor_SMD:R_0603_1608Metric, symbol Power8GDI_Safety:R
- added R808: 9.76k 0.1% 25ppm, Resistor_SMD:R_0603_1608Metric, symbol Power8GDI_Safety:R
- added U806: TPS3808G01QDBVRQ1, Package_TO_SOT_SMD:SOT-23-6, symbol Power8GDI_Safety:TPS3808G01QDBVRQ1
Connections:
- net +3V3: now also C807.1, U806.3 (~{MR}), U806.6 (VDD)
- net GND: now also C807.2, C808.2, R808.2, U806.2 (GND)
- net SAFETY_FAULT_N: now also U806.1 (~{RESET})
- new net +5V_CORE: R807.1
- new net SAFETY_5V_SENSE: C808.1, R807.2, R808.1, U806.5 (SENSE)
- no-connect marks 2 -> 3
Other:
- note added: "HW_KILL_N: local 3.3 V open-drain/contact-to-ground boundary only; no harness/12 V direct connection. U806 monitors divided 5V independently of regulator PG. Fault release never substitutes for a fresh ARM edge. C801..C804 at U801..U804; C807 at U806. Dynamic brownout/partial-power tests remain required."
- note removed: "HW_KILL_N: local 3.3 V open-drain/contact-to-ground boundary only; no harness/12 V direct connection. Local ignition timers and latched OC detectors are on ignition sheets. ARM/power-sequence tests remain required. IC decoupling capacitors C801..C804 must be placed at U801..U804 respectively."
Changed lines of the file:
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@@
 (wire (pts (xy 95.25 139.7) (xy 102.87 139.7)) (stroke (width 0) (type default)))
 (global_label "GND" (shape bidirectional) (at 102.87 139.7 180) (effects (font (size 1.016 1.016)) (justify left bottom)))
+(symbol (lib_id "Power8GDI_Safety:TPS3808G01QDBVRQ1") (at 219.71 139.7 0) (unit 1) (in_bom yes) (on_board yes) (dnp no) (property "Reference" "U806" (at 219.71 130.81 0) (effects (font (size 1.27 1.27)))) (property "Value" "TPS3808G01QDBVRQ1" (at 219.71 148.59 0) (effects (font (size 1.27 1.27)))) (property "Footprint" "Package_TO_SOT_SMD:SOT-23-6" (at 219.71 139.7 0) (effects (font (size 1.27 1.27)) (hide yes))) (property "Design note" "Independent 5V undervoltage fault while 3V3 remains alive; CT open 12..28ms recovery. TI SBVS085J." (at 219.71 139.7 0) (effects (font (size 1.27 1.27)) (hide yes))) (pin "6") (pin "5") (pin "3") (pin "4") (pin "1") (pin "2") (instances (project "Power8GDI_Core" (path "/f4d21065-0a5b-5086-a08e-1af9469f04bd/d3688535-de83-5779-ad3b-0e54c99cc6b1" (reference "U806") (unit 1))) (project "safety_gate" (path "/eded34d9-2614-5eea-9c99-f04c697d2107" (reference "U806") (unit 1)))))
+(wire (pts (xy 204.47 135.89) (xy 196.85 135.89)) (stroke (width 0) (type default)))
+(global_label "+3V3" (shape bidirectional) (at 196.85 135.89 0) (effects (font (size 1.016 1.016)) (justify right bottom)))
+(wire (pts (xy 204.47 138.43) (xy 196.85 138.43)) (stroke (width 0) (type default)))
+(global_label "SAFETY_5V_SENSE" (shape bidirectional) (at 196.85 138.43 0) (effects (font (size 1.016 1.016)) (justify right bottom)))
+(wire (pts (xy 204.47 140.97) (xy 196.85 140.97)) (stroke (width 0) (type default)))
+(global_label "+3V3" (shape bidirectional) (at 196.85 140.97 0) (effects (font (size 1.016 1.016)) (justify right bottom)))
+(no_connect (at 204.47 143.51))
+(wire (pts (xy 234.95 135.89) (xy 242.57 135.89)) (stroke (width 0) (type default)))
+(global_label "SAFETY_FAULT_N" (shape bidirectional) (at 242.57 135.89 180) (effects (font (size 1.016 1.016)) (justify left bottom)))
+(wire (pts (xy 234.95 138.43) (xy 242.57 138.43)) (stroke (width 0) (type default)))
+(global_label "GND" (shape bidirectional) (at 242.57 138.43 180) (effects (font (size 1.016 1.016)) (justify left bottom)))
 (symbol (lib_id "Power8GDI_Safety:R") (at 74.93 204.47 0) (unit 1) (in_bom yes) (on_board yes) (dnp no) (property "Reference" "R801" (at 78.93 203.2 0) (effects (font (size 1.27 1.27)) (justify left))) (property "Value" "10k 1%" (at 78.93 205.74 0) (effects (font (size 1.27 1.27)) (justify left))) (property "Footprint" "Resistor_SMD:R_0603_1608Metric" (at 74.93 204.47 0) (effects (font (size 1.27 1.27)) (hide yes))) (property "Design note" "" (at 74.93 204.47 0) (effects (font (size 1.27 1.27)) (hide yes))) (pin "1") (pin "2") (instances (project "Power8GDI_Core" (path "/f4d21065-0a5b-5086-a08e-1af9469f04bd/d3688535-de83-5779-ad3b-0e54c99cc6b1" (reference "R801") (unit 1))) (project "safety_gate" (path "/eded34d9-2614-5eea-9c99-f04c697d2107" (reference "R801") (unit 1)))))
 (wire (pts (xy 69.85 204.47) (xy 62.23 204.47)) (stroke (width 0) (type default)))
@@
 (wire (pts (xy 485.14 245.11) (xy 492.76 245.11)) (stroke (width 0) (type default)))
 (global_label "GND" (shape bidirectional) (at 492.76 245.11 180) (effects (font (size 1.016 1.016)) (justify left bottom)))
-(text "HW_KILL_N: local 3.3 V open-drain/contact-to-ground boundary only; no harness/12 V direct connection.\nLocal ignition timers and latched OC detectors are on ignition sheets. ARM/power-sequence tests remain required.\nIC decoupling capacitors C801..C804 must be placed at U801..U804 respectively." (at 20 370 0) (effects (font (size 1.27 1.27)) (justify left top)))
+(symbol (lib_id "Power8GDI_Safety:R") (at 74.93 265.43 0) (unit 1) (in_bom yes) (on_board yes) (dnp no) (property "Reference" "R807" (at 78.93 264.16 0) (effects (font (size 1.27 1.27)) (justify left))) (property "Value" "102k 0.1% 25ppm" (at 78.93 266.7 0) (effects (font (size 1.27 1.27)) (justify left))) (property "Footprint" "Resistor_SMD:R_0603_1608Metric" (at 74.93 265.43 0) (effects (font (size 1.27 1.27)) (hide yes))) (property "Design note" "" (at 74.93 265.43 0) (effects (font (size 1.27 1.27)) (hide yes))) (pin "1") (pin "2") (instances (project "Power8GDI_Core" (path "/f4d21065-0a5b-5086-a08e-1af9469f04bd/d3688535-de83-5779-ad3b-0e54c99cc6b1" (reference "R807") (unit 1))) (project "safety_gate" (path "/eded34d9-2614-5eea-9c99-f04c697d2107" (reference "R807") (unit 1)))))
+(wire (pts (xy 69.85 265.43) (xy 62.23 265.43)) (stroke (width 0) (type default)))
+(global_label "+5V_CORE" (shape bidirectional) (at 62.23 265.43 0) (effects (font (size 1.016 1.016)) (justify right bottom)))
+(wire (pts (xy 80.01 265.43) (xy 87.63 265.43)) (stroke (width 0) (type default)))
+(global_label "SAFETY_5V_SENSE" (shape bidirectional) (at 87.63 265.43 180) (effects (font (size 1.016 1.016)) (justify left bottom)))
+(symbol (lib_id "Power8GDI_Safety:R") (at 209.55 265.43 0) (unit 1) (in_bom yes) (on_board yes) (dnp no) (property "Reference" "R808" (at 213.55 264.16 0) (effects (font (size 1.27 1.27)) (justify left))) (property "Value" "9.76k 0.1% 25ppm" (at 213.55 266.7 0) (effects (font (size 1.27 1.27)) (justify left))) (property "Footprint" "Resistor_SMD:R_0603_1608Metric" (at 209.55 265.43 0) (effects (font (size 1.27 1.27)) (hide yes))) (property "Design note" "" (at 209.55 265.43 0) (effects (font (size 1.27 1.27)) (hide yes))) (pin "1") (pin "2") (instances (project "Power8GDI_Core" (path "/f4d21065-0a5b-5086-a08e-1af9469f04bd/d3688535-de83-5779-ad3b-0e54c99cc6b1" (reference "R808") (unit 1))) (project "safety_gate" (path "/eded34d9-2614-5eea-9c99-f04c697d2107" (reference "R808") (unit 1)))))
+(wire (pts (xy 204.47 265.43) (xy 196.85 265.43)) (stroke (width 0) (type default)))
+(global_label "SAFETY_5V_SENSE" (shape bidirectional) (at 196.85 265.43 0) (effects (font (size 1.016 1.016)) (justify right bottom)))
+(wire (pts (xy 214.63 265.43) (xy 222.25 265.43)) (stroke (width 0) (type default)))
+(global_label "GND" (shape bidirectional) (at 222.25 265.43 180) (effects (font (size 1.016 1.016)) (justify left bottom)))
+(symbol (lib_id "Power8GDI_Safety:C") (at 345.44 265.43 0) (unit 1) (in_bom yes) (on_board yes) (dnp no) (property "Reference" "C807" (at 349.44 264.16 0) (effects (font (size 1.27 1.27)) (justify left))) (property "Value" "100nF 25V X7R" (at 349.44 266.7 0) (effects (font (size 1.27 1.27)) (justify left))) (property "Footprint" "Capacitor_SMD:C_0603_1608Metric" (at 345.44 265.43 0) (effects (font (size 1.27 1.27)) (hide yes))) (property "Design note" "" (at 345.44 265.43 0) (effects (font (size 1.27 1.27)) (hide yes))) (pin "1") (pin "2") (instances (project "Power8GDI_Core" (path "/f4d21065-0a5b-5086-a08e-1af9469f04bd/d3688535-de83-5779-ad3b-0e54c99cc6b1" (reference "C807") (unit 1))) (project "safety_gate" (path "/eded34d9-2614-5eea-9c99-f04c697d2107" (reference "C807") (unit 1)))))
+(wire (pts (xy 340.36 265.43) (xy 332.74 265.43)) (stroke (width 0) (type default)))
+(global_label "+3V3" (shape bidirectional) (at 332.74 265.43 0) (effects (font (size 1.016 1.016)) (justify right bottom)))
+(wire (pts (xy 350.52 265.43) (xy 358.14 265.43)) (stroke (width 0) (type default)))
+(global_label "GND" (shape bidirectional) (at 358.14 265.43 180) (effects (font (size 1.016 1.016)) (justify left bottom)))
+(symbol (lib_id "Power8GDI_Safety:C") (at 480.06 265.43 0) (unit 1) (in_bom yes) (on_board yes) (dnp no) (property "Reference" "C808" (at 484.06 264.16 0) (effects (font (size 1.27 1.27)) (justify left))) (property "Value" "1nF 50V C0G 5%" (at 484.06 266.7 0) (effects (font (size 1.27 1.27)) (justify left))) (property "Footprint" "Capacitor_SMD:C_0603_1608Metric" (at 480.06 265.43 0) (effects (font (size 1.27 1.27)) (hide yes))) (property "Design note" "" (at 480.06 265.43 0) (effects (font (size 1.27 1.27)) (hide yes))) (pin "1") (pin "2") (instances (project "Power8GDI_Core" (path "/f4d21065-0a5b-5086-a08e-1af9469f04bd/d3688535-de83-5779-ad3b-0e54c99cc6b1" (reference "C808") (unit 1))) (project "safety_gate" (path "/eded34d9-2614-5eea-9c99-f04c697d2107" (reference "C808") (unit 1)))))
+(wire (pts (xy 474.98 265.43) (xy 467.36 265.43)) (stroke (width 0) (type default)))
+(global_label "SAFETY_5V_SENSE" (shape bidirectional) (at 467.36 265.43 0) (effects (font (size 1.016 1.016)) (justify right bottom)))
+(wire (pts (xy 485.14 265.43) (xy 492.76 265.43)) (stroke (width 0) (type default)))
+(global_label "GND" (shape bidirectional) (at 492.76 265.43 180) (effects (font (size 1.016 1.016)) (justify left bottom)))
+(text "HW_KILL_N: local 3.3 V open-drain/contact-to-ground boundary only; no harness/12 V direct connection.\nU806 monitors divided 5V independently of regulator PG. Fault release never substitutes for a fresh ARM edge.\nC801..C804 at U801..U804; C807 at U806. Dynamic brownout/partial-power tests remain required." (at 20 370 0) (effects (font (size 1.27 1.27)) (justify left top)))
 (sheet_instances (path "/" (page "1"))))

Commit message: Review B58 injector power stage and bind selected GDI6 BOM
Parts:
- C801, C802, C803, C804, C807: Hardware_Qualification (none) -> BOARD_QUALIFICATION_PENDING; MPN (none) -> C0603C104K5RACTU; Manufacturer (none) -> KEMET; Procurement_Status (none) -> SELECTED_CATALOG_ITEM; Purchase_Released (none) -> false; Selection_Gaps (none) -> []; Selection_ID (none) -> SEL-6bf9727c4e40; Selection_Ratings (none) -> {"capacitance_pf": 100000, "dielectric": "X7R", "rated_volt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; Selection_Source_URLs (none) -> https://search.kemet.com/download/specsheet/C0603C104K5RACTU
- C806: Hardware_Qualification (none) -> BOARD_QUALIFICATION_PENDING; MPN (none) -> C0603C121F5GACTU; Manufacturer (none) -> KEMET; Procurement_Status (none) -> SELECTED_CATALOG_ITEM; Purchase_Released (none) -> false; Selection_Gaps (none) -> []; Selection_ID (none) -> SEL-9d485d08899c; Selection_Ratings (none) -> {"capacitance_pf": 120, "dielectric": "C0G", "rated_voltage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; Selection_Source_URLs (none) -> https://www.digikey.com/en/products/detail/kemet/C0603C121F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
- C808: Hardware_Qualification (none) -> BOARD_QUALIFICATION_PENDING; MPN (none) -> C0603C102J1GACTU; Manufacturer (none) -> KEMET; Procurement_Status (none) -> SELECTED_CATALOG_ITEM; Purchase_Released (none) -> false; Selection_Gaps (none) -> []; Selection_ID (none) -> SEL-ec742f39ec1f; Selection_Ratings (none) -> {"capacitance_pf": 1000, "dielectric": "C0G", "rated_voltag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; Selection_Source_URLs (none) -> https://search.kemet.com/download/specsheet/C0603C102J1GACTU
- R6500: Hardware_Qualification (none) -> BOARD_QUALIFICATION_PENDING; MPN (none) -> CRCW06030000Z0EA; Manufacturer (none) -> Vishay; Procurement_Status (none) -> SELECTED_FAMILY_CODE; Purchase_Released (none) -> false; Selection_Gaps (none) -> []; Selection_ID (none) -> SEL-8473f02313b2; Selection_Ratings (none) -> {"aec_q200": true, "current_a": 2, "power_reference_tempera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; Selection_Source_URLs (none) -> https://www.vishay.com/docs/20035/dcrcwe3.pdf
- R801, R802, R803, R804, R805, R806: Hardware_Qualification (none) -> BOARD_QUALIFICATION_PENDING; MPN (none) -> CRCW060310K0FKEA; Manufacturer (none) -> Vishay; Procurement_Status (none) -> SELECTED_FAMILY_CODE; Purchase_Released (none) -> false; Selection_Gaps (none) -> []; Selection_ID (none) -> SEL-9c0806476875; Selection_Ratings (none) -> {"aec_q200": true, "derating": "Use manufacturer power vers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; Selection_Source_URLs (none) -> https://www.vishay.com/docs/20035/dcrcwe3.pdf
- R807: Hardware_Qualification (none) -> BOARD_QUALIFICATION_PENDING; MPN (none) -> TNPW0603102KBEEA; Manufacturer (none) -> Vishay; Procurement_Status (none) -> SELECTED_CATALOG_ITEM; Purchase_Released (none) -> false; Selection_Gaps (none) -> []; Selection_ID (none) -> SEL-3f87dfffdd40; Selection_Ratings (none) -> {"aec_q200": true, "derating": "Use manufacturer power vers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; Selection_Source_URLs (none) -> https://www.digikey.com/en/products/detail/vishay-dale/TNPW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
- R808: Hardware_Qualification (none) -> BOARD_QUALIFICATION_PENDING; MPN (none) -> TNPW06039K76BEEA; Manufacturer (none) -> Vishay; Procurement_Status (none) -> SELECTED_CATALOG_ITEM; Purchase_Released (none) -> false; Selection_Gaps (none) -> []; Selection_ID (none) -> SEL-2ea30ddc83cb; Selection_Ratings (none) -> {"aec_q200": true, "derating": "Use manufacturer power vers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; Selection_Source_URLs (none) -> https://www.digikey.com/en/products/detail/vishay-dale/TNPW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
- U801: Hardware_Qualification (none) -> PINOUT_RATINGS_AND_DELIVERY_SUFFIX_REVIEW_PENDING; MPN (none) -> TPS3431SQDRBRQ1; Manufacturer (none) -> Texas Instruments; Procurement_Status (none) -> REFERENCE_MPN_RETAINED; Purchase_Released (none) -> false; Selection_Gaps (none) -> ["Existing schematic MPN retained. Complete circuit rating/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; Selection_ID (none) -> SEL-ee816c604e28; Selection_Ratings (none) -> {}; Selection_Source_URLs (none) -> https://www.ti.com/product/TPS3431-Q1/part-details/TPS3431S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
- U802: Hardware_Qualification (none) -> PINOUT_RATINGS_AND_DELIVERY_SUFFIX_REVIEW_PENDING; MPN (none) -> TPS3808G33QDBVRQ1; Manufacturer (none) -> Texas Instruments; Procurement_Status (none) -> REFERENCE_MPN_RETAINED; Purchase_Released (none) -> false; Selection_Gaps (none) -> ["Existing schematic MPN retained. Complete circuit rating/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; Selection_ID (none) -> SEL-36c2480848bd; Selection_Ratings (none) -> {}; Selection_Source_URLs (none) -> https://www.ti.com/product/TPS3808-Q1/part-details/TPS3808G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
- U803: Hardware_Qualification (none) -> PINOUT_RATINGS_AND_DELIVERY_SUFFIX_REVIEW_PENDING; MPN (none) -> SN74LVC1G17QDBVRQ1; Manufacturer (none) -> Texas Instruments; Procurement_Status (none) -> REFERENCE_MPN_RETAINED; Purchase_Released (none) -> false; Selection_Gaps (none) -> ["Existing schematic MPN retained. Complete circuit rating/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; Selection_ID (none) -> SEL-ecf3e6662afb; Selection_Ratings (none) -> {}; Selection_Source_URLs (none) -> https://www.ti.com/product/SN74LVC1G17-Q1/part-details/SN74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
- U804: Hardware_Qualification (none) -> PINOUT_RATINGS_AND_DELIVERY_SUFFIX_REVIEW_PENDING; MPN (none) -> SN74LVC2G74QDCURQ1; Manufacturer (none) -> Texas Instruments; Procurement_Status (none) -> REFERENCE_MPN_RETAINED; Purchase_Released (none) -> false; Selection_Gaps (none) -> ["Existing schematic MPN retained. Complete circuit rating/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; Selection_ID (none) -> SEL-776f81deb4dc; Selection_Ratings (none) -> {}; Selection_Source_URLs (none) -> https://www.ti.com/product/SN74LVC2G74-Q1/part-details/SN74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
- U806: Hardware_Qualification (none) -> PINOUT_RATINGS_AND_DELIVERY_SUFFIX_REVIEW_PENDING; MPN (none) -> TPS3808G01QDBVRQ1; Manufacturer (none) -> Texas Instruments; Procurement_Status (none) -> REFERENCE_MPN_RETAINED; Purchase_Released (none) -> false; Selection_Gaps (none) -> ["Existing schematic MPN retained. Complete circuit rating/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; Selection_ID (none) -> SEL-3a6da169e9be; Selection_Ratings (none) -> {}; Selection_Source_URLs (none) -> https://www.ti.com/product/TPS3808-Q1/part-details/TPS3808G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
