File: Power8GDI/hardware/design/board/gdi6_candidate/Power8GDI_Review.kicad_pcb (KiCad board)
At the start: 4 copper layers, 245 x 165 mm, 1092 parts, among them J101 SWD 3V3 target reference, J1501 Molex 1050170001, J1502 Molex 1040310811, J5600 Conn_02x03_Odd_Even, J601 6437288-1 / KEY1 CANDIDATE, J602 6437288-1 / KEY1 CANDIDATE, J603 6437288-1 / KEY1 CANDIDATE, J604 6437288-1 / KEY1 CANDIDATE, Q1510 2N7002,215, Q201 IPD60N10S4L12ATMA1, Q202 IPD60N10S4L12ATMA1, Q203 IPD60N10S4L12ATMA1, Q204 IPD60N10S4L12ATMA1, Q205 IPD60N10S4L12ATMA1, Q206 IPD60N10S4L12ATMA1, Q207 IPD60N10S4L12ATMA1, Q208 IPD60N10S4L12ATMA1, Q209 IPD60N10S4L12ATMA1, Q211 IPD60N10S4L12ATMA1, Q212 IPD60N10S4L12ATMA1, Q213 IPD60N10S4L12ATMA1, Q301 IPD60N10S4L12ATMA1, Q302 IPD60N10S4L12ATMA1, Q303 IPD60N10S4L12ATMA1, Q304 IPD60N10S4L12ATMA1, Q305 IPD60N10S4L12ATMA1, Q306 IPD60N10S4L12ATMA1, Q307 IPD60N10S4L12ATMA1, Q308 IPD60N10S4L12ATMA1, Q309 IPD60N10S4L12ATMA1, Q311 IPD60N10S4L12ATMA1, Q312 IPD60N10S4L12ATMA1, Q313 IPD60N10S4L12ATMA1, Q5001 IPD90N10S4-06, Q5002 IPD90N10S4-06, Q5051 IPD90N10S4-06, Q5052 IPD90N10S4-06, Q5420 STGB18N40LZT4, Q5440 STGB18N40LZT4, Q5460 STGB18N40LZT4, Q5480 STGB18N40LZT4, Q5500 STGB18N40LZT4, Q5520 STGB18N40LZT4, Q5600 VND7NV04TR-E, Q5620 BC847B-QR, Q6200 IPD90N10S4-06, Q6201 IPD90N10S4-06, Q6250 IPD90N10S4-06, Q6251 IPD90N10S4-06, U101 STM32F767IIT6, U103 TCAN1042HGVDRQ1, U104 TLIN1029ADRQ1, U1101 TLE9104SHXUMA1, U1102 TLE9104SHXUMA1, U1103 TLE9104SHXUMA1, U1104 TLE9104SHXUMA1, U1105 TLE9104SHXUMA1, U1106 TLE9104SHXUMA1, U1121 SN74LVC14AQPWRQ1, U1122 SN74LVC14AQPWRQ1, U1123 SN74LVC14AQPWRQ1, U1124 SN74LVC14AQPWRQ1, U1125 SN74LVC14AQPWRQ1, U1126 SN74LVC14AQPWRQ1, U1140 SN74LVC1G17QDBVRQ1, U1501 TCAN1042HGVDRQ1, U1502 TLIN1029ADRQ1, U1530 TPS7B4253QDDARQ1, U1531 TPS7B4253QDDARQ1, U1600 SN74LVC14AQPWRQ1, U1701 TPIC8101DWR, U1702 SN74AHCT244QPWRQ1, U1703 CLVC1G125QDBVRQ1, U201 MC33PT2001AE, U249 NCV78M05ABDTRKG, U301 MC33PT2001AE, U349 NCV78M05ABDTRKG, U5001 LM74800QDRRRQ1, U5051 LM74800QDRRRQ1, U5101 SN74LVC2G08QDCURQ1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

Commit message: Route WBO regulator feed and separate LT3042 Kelvin sense
Routing:
- net WBO1_3V3: track 16.1 -> 47.4 mm, vias 0 -> 1
Changed lines of the file:
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@@
+	)
+	(segment
+		(start 177.10295 68.975)
+		(end 178.60295 66.975)
+		(width 0.25)
+		(layer "F.Cu")
+		(net 632)
 	)
 	(segment
@@
 		(net 632)
 	)
+	(via
+		(at 177.10295 68.975)
+		(size 0.65)
+		(drill 0.3)
+		(layers "F.Cu" "B.Cu")
+		(net 632)
+	)
+	(segment
+		(start 164.2 88.078729)
+		(end 164.011038 88.078729)
+		(width 0.2)
+		(layer "B.Cu")
+		(net 632)
+	)
+	(segment
+		(start 173.761038 73.578729)
+		(end 176.011038 72.578729)
+		(width 0.4)
+		(layer "B.Cu")
+		(net 632)
+	)
 	(segment
 		(start 163.15 85.5)
-		(end 163.15 86)
+		(end 164.2 85.5)
 		(width 0.2)
+		(layer "B.Cu")
+		(net 632)
+	)
+	(segment
+		(start 168.011038 84.828729)
+		(end 168.011038 82.578729)
+		(width 0.4)
+		(layer "B.Cu")
+		(net 632)
+	)
+	(segment
+		(start 167.511038 85.328729)
+		(end 168.011038 84.828729)
+		(width 0.4)
 		(layer "B.Cu")
 		(net 632)
@@
 	)
 	(segment
+		(start 169.261038 81.078729)
+		(end 169.261038 79.828729)
+		(width 0.4)
+		(layer "B.Cu")
+		(net 632)
+	)
+	(segment
+		(start 170.511038 78.328729)
+		(end 170.511038 76.078729)
+		(width 0.4)
+		(layer "B.Cu")
+		(net 632)
+	)
+	(segment
 		(start 163.15 86)
 		(end 164.011038 88.078729)
 		(width 0.2)
+		(layer "B.Cu")
+		(net 632)
+	)
+	(segment
+		(start 169.261038 79.828729)
+		(end 170.511038 78.328729)
+		(width 0.4)
+		(layer "B.Cu")
+		(net 632)
+	)
+	(segment
+		(start 168.011038 82.578729)
+		(end 169.261038 81.078729)
+		(width 0.4)
+		(layer "B.Cu")
+		(net 632)
+	)
+	(segment
+		(start 173.011038 73.578729)
+		(end 173.761038 73.578729)
+		(width 0.4)
 		(layer "B.Cu")
 		(net 632)
@@
 		(layer "B.Cu")
 		(net 632)
+	)
+	(segment
+		(start 176.011038 72.578729)
+		(end 177.10295 68.975)
+		(width 0.4)
+		(layer "B.Cu")
+		(net 632)
+	)
+	(segment
+		(start 164.011038 88.078729)
+		(end 166.511038 85.578729)
+		(width 0.4)
+		(layer "B.Cu")
+		(net 632)
+	)
+	(segment
+		(start 170.511038 76.078729)
+		(end 173.011038 73.578729)
+		(width 0.4)
+		(layer "B.Cu")
+		(net 632)
+	)
+	(segment
+		(start 164.2 85.5)
+		(end 164.2 88.078729)
+		(width 0.2)
+		(layer "B.Cu")
+		(net 632)
+	)
+	(segment
+		(start 166.511038 85.578729)
+		(end 167.511038 85.328729)
+		(width 0.4)
+		(layer "B.Cu")
+		(net 632)

Commit message: Connect WBO regulator and output capacitor ground returns
Routing:
- net GND: track 116.3 -> 125.2 mm
Changed lines of the file:
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@@
+	)
+	(segment
+		(start 164.011038 91.028729)
+		(end 161 85)
+		(width 0.25)
+		(layer "B.Cu")
+		(net 133)
 	)
 	(segment
@@
 		(layer "B.Cu")
 		(net 133)
+	)
+	(segment
+		(start 163.15 85)
+		(end 161 85)
+		(width 0.25)
+		(layer "B.Cu")
+		(net 133)
